File: MiniLatte.kicad_pcb (KiCad board)
At the start: 2 copper layers, 1 part

Commit message: .
Parts:
- added C1: 100nF, Capacitor_SMD:C_0402_1005Metric, F.Cu at (41.6, 111.5)
- added C10: 100nF, Capacitor_SMD:C_0402_1005Metric, F.Cu at (44.4, 117.4)
- added C100: 120pF, Capacitor_SMD:C_0402_1005Metric, F.Cu at (23.3, 94.1)
- added C101: 120pF, Capacitor_SMD:C_0402_1005Metric, F.Cu at (23.3, 96.1)
- added C102: 100nF, Capacitor_SMD:C_0402_1005Metric, F.Cu at (41.6, 86.9)
- added C103: 100nF, Capacitor_SMD:C_0402_1005Metric, F.Cu at (41.6, 88.9)
- added C104: 100nF, Capacitor_SMD:C_0402_1005Metric, F.Cu at (41.6, 90.9)
- added C105: 100nF, Capacitor_SMD:C_0402_1005Metric, F.Cu at (41.6, 92.9)
- added C106: 100nF, Capacitor_SMD:C_0402_1005Metric, F.Cu at (41.6, 94.8)
- added C107: 100nF, Capacitor_SMD:C_0402_1005Metric, F.Cu at (41.6, 96.8)
- added C108: 100nF, Capacitor_SMD:C_0402_1005Metric, F.Cu at (44.5, 86.9)
- added C109: 100nF, Capacitor_SMD:C_0402_1005Metric, F.Cu at (44.5, 88.9)
- added C11: 18pF, Capacitor_SMD:C_0402_1005Metric, F.Cu at (44.4, 119.4)
- added C110: 100nF, Capacitor_SMD:C_0402_1005Metric, F.Cu at (44.5, 90.9)
- added C111: 100nF, Capacitor_SMD:C_0402_1005Metric, F.Cu at (44.5, 92.9)
- added C112: 18pF, Capacitor_SMD:C_0402_1005Metric, F.Cu at (44.5, 94.8)
- added C113: 100nF, Capacitor_SMD:C_0402_1005Metric, F.Cu at (44.5, 96.8)
- added C114: 100nF, Capacitor_SMD:C_0402_1005Metric, F.Cu at (47.4, 86.9)
- added C115: 100nF, Capacitor_SMD:C_0402_1005Metric, F.Cu at (47.4, 88.9)
- added C116: 100nF, Capacitor_SMD:C_0402_1005Metric, F.Cu at (47.4, 90.9)
- added C117: 18pF, Capacitor_SMD:C_0402_1005Metric, F.Cu at (47.4, 92.9)
- added C118: 10uF, Capacitor_SMD:C_0805_2012Metric, F.Cu at (57.3, 87.5)
- added C119: 100nF, Capacitor_SMD:C_0402_1005Metric, F.Cu at (47.4, 94.8)
- added C12: 100nF, Capacitor_SMD:C_0402_1005Metric, F.Cu at (44.4, 121.4)
- added C120: 100nF, Capacitor_SMD:C_0402_1005Metric, F.Cu at (36.7, 100.8)
- added C121: 100nF, Capacitor_SMD:C_0402_1005Metric, F.Cu at (36.7, 102.8)
- added C122: 100nF, Capacitor_SMD:C_0402_1005Metric, F.Cu at (36.7, 104.8)
- added C123: 100nF, Capacitor_SMD:C_0402_1005Metric, F.Cu at (36.7, 106.7)
- added C124: 100nF, Capacitor_SMD:C_0402_1005Metric, F.Cu at (36.7, 108.7)
- added C125: 100nF, Capacitor_SMD:C_0402_1005Metric, F.Cu at (36.7, 110.7)
- added C126: 100nF, Capacitor_SMD:C_0402_1005Metric, F.Cu at (36.7, 112.7)
- added C127: 100nF, Capacitor_SMD:C_0402_1005Metric, F.Cu at (36.7, 114.6)
- added C128: 100nF, Capacitor_SMD:C_0402_1005Metric, F.Cu at (47.4, 176.8)
- added C129: 10uF, Capacitor_SMD:C_0805_2012Metric, F.Cu at (48.7, 188.4)
- added C13: 100nF, Capacitor_SMD:C_0402_1005Metric, F.Cu at (47.3, 111.5)
- added C130: 10uF, Capacitor_SMD:C_0805_2012Metric, F.Cu at (48.7, 191.4)
- added C131: 100nF, Capacitor_SMD:C_0402_1005Metric, F.Cu at (47.4, 178.7)
- added C132: 1uF, Capacitor_SMD:C_0603_1608Metric, F.Cu at (52.9, 193.9)
- added C133: 100nF, Capacitor_SMD:C_0402_1005Metric, F.Cu at (47.4, 180.7)
- added C134: 1uF, Capacitor_SMD:C_0603_1608Metric, F.Cu at (52.9, 196.4)
- added C135: 10uF, Capacitor_SMD:C_0805_2012Metric, F.Cu at (48.7, 194.4)
- added C136: 100nF, Capacitor_SMD:C_0402_1005Metric, F.Cu at (47.4, 182.7)
- added C137: 10uF, Capacitor_SMD:C_0805_2012Metric, F.Cu at (48.7, 197.4)
- added C138: 100nF, Capacitor_SMD:C_0402_1005Metric, F.Cu at (21.7, 190.7)
- added C139: 100nF, Capacitor_SMD:C_0402_1005Metric, F.Cu at (21.7, 192.7)
- added C14: 100nF, Capacitor_SMD:C_0402_1005Metric, F.Cu at (47.3, 113.5)
- added C140: 100nF, Capacitor_SMD:C_0402_1005Metric, F.Cu at (21.7, 194.6)
- added C141: 100nF, Capacitor_SMD:C_0402_1005Metric, F.Cu at (21.7, 196.6)
- added C142: 100nF, Capacitor_SMD:C_0402_1005Metric, F.Cu at (24.6, 190.7)
- added C143: 100nF, Capacitor_SMD:C_0402_1005Metric, F.Cu at (24.6, 192.7)
- added C144: 100nF, Capacitor_SMD:C_0402_1005Metric, F.Cu at (24.6, 194.6)
- added C145: 100nF, Capacitor_SMD:C_0402_1005Metric, F.Cu at (24.6, 196.6)
- added C146: 100nF, Capacitor_SMD:C_0402_1005Metric, F.Cu at (27.5, 190.7)
- added C147: 100nF, Capacitor_SMD:C_0402_1005Metric, F.Cu at (27.5, 192.7)
- added C148: 100nF, Capacitor_SMD:C_0402_1005Metric, F.Cu at (27.5, 194.6)
- added C149: 100nF, Capacitor_SMD:C_0402_1005Metric, F.Cu at (27.5, 196.6)
- added C15: 100nF, Capacitor_SMD:C_0402_1005Metric, F.Cu at (47.3, 115.5)
- added C150: 100nF, Capacitor_SMD:C_0402_1005Metric, F.Cu at (30.4, 190.7)
- added C151: 100nF, Capacitor_SMD:C_0402_1005Metric, F.Cu at (30.4, 192.7)
- added C152: 100nF, Capacitor_SMD:C_0402_1005Metric, F.Cu at (30.4, 194.6)
- added C153: 100nF, Capacitor_SMD:C_0402_1005Metric, F.Cu at (30.4, 196.6)
- added C154: 220nF, Capacitor_SMD:C_0402_1005Metric, F.Cu at (50.3, 176.8)
- added C155: 220nF, Capacitor_SMD:C_0402_1005Metric, F.Cu at (50.3, 178.7)
- added C156: 330nF, Capacitor_SMD:C_0402_1005Metric, F.Cu at (50.3, 180.7)
- added C157: 330nF, Capacitor_SMD:C_0402_1005Metric, F.Cu at (50.3, 182.7)
- added C158: 220nF, Capacitor_SMD:C_0402_1005Metric, F.Cu at (53.1, 176.8)
- added C159: 220nF, Capacitor_SMD:C_0402_1005Metric, F.Cu at (53.1, 178.7)
- added C16: 18pF, Capacitor_SMD:C_0402_1005Metric, F.Cu at (47.3, 117.4)
- added C160: 330nF, Capacitor_SMD:C_0402_1005Metric, F.Cu at (53.1, 180.7)
- added C161: 330nF, Capacitor_SMD:C_0402_1005Metric, F.Cu at (53.1, 182.7)
- added C17: 10uF, Capacitor_SMD:C_0805_2012Metric, F.Cu at (57.3, 112.1)
- added C18: 100nF, Capacitor_SMD:C_0402_1005Metric, F.Cu at (47.3, 119.4)
- added C19: 100nF, Capacitor_SMD:C_0402_1005Metric, F.Cu at (56.4, 133.8)
- added C2: 100nF, Capacitor_SMD:C_0402_1005Metric, F.Cu at (41.6, 113.5)
- added C20: 100nF, Capacitor_SMD:C_0402_1005Metric, F.Cu at (56.4, 135.8)
- added C21: 100nF, Capacitor_SMD:C_0402_1005Metric, F.Cu at (56.4, 137.8)
- added C22: 100nF, Capacitor_SMD:C_0402_1005Metric, F.Cu at (56.4, 139.7)
- added C23: 100nF, Capacitor_SMD:C_0402_1005Metric, F.Cu at (56.4, 141.7)
- added C24: 100nF, Capacitor_SMD:C_0402_1005Metric, F.Cu at (56.4, 143.7)
- added C25: 100nF, Capacitor_SMD:C_0402_1005Metric, F.Cu at (56.4, 145.7)
- added C26: 100nF, Capacitor_SMD:C_0402_1005Metric, F.Cu at (56.4, 147.6)
- added C27: 100nF, Capacitor_SMD:C_0402_1005Metric, F.Cu at (0.80, 119.3)
- added C28: 100nF, Capacitor_SMD:C_0402_1005Metric, F.Cu at (0.80, 121.2)
- added C29: 18pF, Capacitor_SMD:C_0402_1005Metric, F.Cu at (0.80, 123.2)
- added C3: 100nF, Capacitor_SMD:C_0402_1005Metric, F.Cu at (41.6, 115.5)
- added C30: 18pF, Capacitor_SMD:C_0402_1005Metric, F.Cu at (0.80, 125.2)
- added C31: 100nF, Capacitor_SMD:C_0402_1005Metric, F.Cu at (0.80, 127.1)
- added C32: 100nF, Capacitor_SMD:C_0402_1005Metric, F.Cu at (0.80, 129.1)
- added C33: 100nF, Capacitor_SMD:C_0402_1005Metric, F.Cu at (3.67, 119.3)
- added C34: 22uF, Capacitor_SMD:C_0805_2012Metric, F.Cu at (1.59, 136.1)
- added C35: 10uF, Capacitor_SMD:C_0805_2012Metric, F.Cu at (1.59, 139.2)
- added C36: 10uF, Capacitor_SMD:C_0805_2012Metric, F.Cu at (1.59, 142.2)
- added C37: 100nF, Capacitor_SMD:C_0402_1005Metric, F.Cu at (3.67, 121.2)
- added C38: 100nF, Capacitor_SMD:C_0402_1005Metric, F.Cu at (3.67, 123.2)
- added C39: 100nF, Capacitor_SMD:C_0402_1005Metric, F.Cu at (3.67, 125.2)
- added C4: 100nF, Capacitor_SMD:C_0402_1005Metric, F.Cu at (41.6, 117.4)
- added C40: 100nF, Capacitor_SMD:C_0402_1005Metric, F.Cu at (3.67, 127.1)
- added C41: 220nF, Capacitor_SMD:C_0402_1005Metric, F.Cu at (-6.47, 95.9)
- added C42: 220nF, Capacitor_SMD:C_0402_1005Metric, F.Cu at (-6.47, 97.9)
- added C43: 18pF, Capacitor_SMD:C_0402_1005Metric, F.Cu at (-6.47, 99.8)
- added C44: 18pF, Capacitor_SMD:C_0402_1005Metric, F.Cu at (-6.47, 101.8)
- added C45: 10uF, Capacitor_SMD:C_0805_2012Metric, F.Cu at (-13.2, 107.2)
- added C46: 100nF, Capacitor_SMD:C_0402_1005Metric, F.Cu at (-6.47, 103.8)
- added C47: 100nF, Capacitor_SMD:C_0402_1005Metric, F.Cu at (-6.47, 105.7)
- added C48: 100nF, Capacitor_SMD:C_0402_1005Metric, F.Cu at (-6.47, 107.7)
- added C49: 100nF, Capacitor_SMD:C_0402_1005Metric, F.Cu at (-3.60, 95.9)
- added C5: 100nF, Capacitor_SMD:C_0402_1005Metric, F.Cu at (41.6, 119.4)
- added C50: 100nF, Capacitor_SMD:C_0402_1005Metric, F.Cu at (-3.60, 97.9)
- added C51: 100nF, Capacitor_SMD:C_0402_1005Metric, F.Cu at (-3.60, 99.8)
- added C52: 22pF, Capacitor_SMD:C_0402_1005Metric, F.Cu at (-3.60, 101.8)
- added C53: 10uF, Capacitor_SMD:C_0805_2012Metric, F.Cu at (-13.2, 110.2)
- added C54: 100nF, Capacitor_SMD:C_0402_1005Metric, F.Cu at (-3.60, 103.8)
- added C55: 100nF, Capacitor_SMD:C_0402_1005Metric, F.Cu at (-3.60, 105.7)
- added C56: 100nF, Capacitor_SMD:C_0402_1005Metric, F.Cu at (-3.60, 107.7)
- added C57: 100nF, Capacitor_SMD:C_0402_1005Metric, F.Cu at (-0.73, 95.9)
- added C58: 100nF, Capacitor_SMD:C_0402_1005Metric, F.Cu at (-0.73, 97.9)
- added C59: 100nF, Capacitor_SMD:C_0402_1005Metric, F.Cu at (-0.73, 99.8)
- added C6: 100nF, Capacitor_SMD:C_0402_1005Metric, F.Cu at (41.6, 121.4)
- added C60: 100nF, Capacitor_SMD:C_0402_1005Metric, F.Cu at (-0.73, 101.8)
- added C61: 100nF, Capacitor_SMD:C_0402_1005Metric, F.Cu at (-0.73, 103.8)
- added C62: 100nF, Capacitor_SMD:C_0402_1005Metric, F.Cu at (-0.73, 105.7)
- added C63: 100nF, Capacitor_SMD:C_0402_1005Metric, F.Cu at (-0.73, 107.7)
- added C64: 100nF, Capacitor_SMD:C_0402_1005Metric, F.Cu at (2.14, 95.9)
- added C65: 100nF, Capacitor_SMD:C_0402_1005Metric, F.Cu at (2.14, 97.9)
- added C66: 100nF, Capacitor_SMD:C_0402_1005Metric, F.Cu at (2.14, 99.8)
- added C67: 100nF, Capacitor_SMD:C_0402_1005Metric, F.Cu at (2.14, 101.8)
- added C68: 100nF, Capacitor_SMD:C_0402_1005Metric, F.Cu at (2.14, 103.8)
- added C69: 100nF, Capacitor_SMD:C_0402_1005Metric, F.Cu at (2.14, 105.7)
- added C7: 100nF, Capacitor_SMD:C_0402_1005Metric, F.Cu at (44.4, 111.5)
- added C70: 1nF 2kV, Capacitor_SMD:C_1210_3225Metric, F.Cu at (0.32, 110.8)
- added C71: 220nF, Capacitor_SMD:C_0402_1005Metric, F.Cu at (33.1, 133.8)
- added C72: 220nF, Capacitor_SMD:C_0402_1005Metric, F.Cu at (33.1, 135.8)
- added C73: 220nF, Capacitor_SMD:C_0402_1005Metric, F.Cu at (33.1, 137.8)
- added C74: 220nF, Capacitor_SMD:C_0402_1005Metric, F.Cu at (33.1, 139.7)
- added C75: 220nF, Capacitor_SMD:C_0402_1005Metric, F.Cu at (33.1, 141.7)
- added C76: 220nF, Capacitor_SMD:C_0402_1005Metric, F.Cu at (36.0, 133.8)
- added C77: 220nF, Capacitor_SMD:C_0402_1005Metric, F.Cu at (36.0, 135.8)
- added C78: 220nF, Capacitor_SMD:C_0402_1005Metric, F.Cu at (36.0, 137.8)
- added C79: 220nF, Capacitor_SMD:C_0402_1005Metric, F.Cu at (36.0, 139.7)
- added C8: 100nF, Capacitor_SMD:C_0402_1005Metric, F.Cu at (44.4, 113.5)
- added C80: 220nF, Capacitor_SMD:C_0402_1005Metric, F.Cu at (36.0, 141.7)
- added C81: 10uF, Capacitor_SMD:C_0805_2012Metric, F.Cu at (27.1, 76.8)
- added C82: 10uF, Capacitor_SMD:C_0805_2012Metric, F.Cu at (27.1, 79.8)
- added C83: 10uF, Capacitor_SMD:C_0805_2012Metric, F.Cu at (27.1, 82.8)
- added C84: 100nF, Capacitor_SMD:C_0402_1005Metric, F.Cu at (17.5, 90.2)
- added C85: 100nF, Capacitor_SMD:C_0402_1005Metric, F.Cu at (17.5, 92.1)
- added C86: 100nF, Capacitor_SMD:C_0402_1005Metric, F.Cu at (17.5, 94.1)
- added C87: 22uF, Capacitor_SMD:C_0805_2012Metric, F.Cu at (31.5, 76.8)
- added C88: 22uF, Capacitor_SMD:C_0805_2012Metric, F.Cu at (31.5, 79.8)
- added C89: 22uF, Capacitor_SMD:C_0805_2012Metric, F.Cu at (31.5, 82.8)
- added C9: 100nF, Capacitor_SMD:C_0402_1005Metric, F.Cu at (44.4, 115.5)
- added C90: 22uF, Capacitor_SMD:C_0805_2012Metric, F.Cu at (36.0, 76.8)
- added C91: 22uF, Capacitor_SMD:C_0805_2012Metric, F.Cu at (36.0, 79.8)
- added C92: 22uF, Capacitor_SMD:C_0805_2012Metric, F.Cu at (36.0, 82.8)
- added C93: 100nF, Capacitor_SMD:C_0402_1005Metric, F.Cu at (17.5, 96.1)
- added C94: 100nF, Capacitor_SMD:C_0402_1005Metric, F.Cu at (20.4, 90.2)
- added C95: 100nF, Capacitor_SMD:C_0402_1005Metric, F.Cu at (20.4, 92.1)
- added C96: 10nf, Capacitor_SMD:C_0402_1005Metric, F.Cu at (20.4, 94.1)
- added C97: 10nf, Capacitor_SMD:C_0402_1005Metric, F.Cu at (20.4, 96.1)
- added C98: 10nf, Capacitor_SMD:C_0402_1005Metric, F.Cu at (23.3, 90.2)
- added C99: 120pF, Capacitor_SMD:C_0402_1005Metric, F.Cu at (23.3, 92.1)
- added CN1: 2199230-4_C2977809, easyeda2kicad:PCIE-SMD_2199230-4, F.Cu at (-19.7, 100.7)
- added CN2: APCI0107-P001A, easyeda2kicad:CONN-SMD_APCI0107-P001A, F.Cu at (20.1, 137.9)
- added CN3: APCI0107-P001A, easyeda2kicad:CONN-SMD_APCI0107-P001A, F.Cu at (20.1, 148.0)
- added CN4: APCI0107-P001A, easyeda2kicad:CONN-SMD_APCI0107-P001A, F.Cu at (20.1, 158.1)
- added Card1: SD-006M, easyeda2kicad:SD-SMD_SD-006M, F.Cu at (-16.1, 130.9)
- added Card2: TF-01A, easyeda2kicad:TF-SMD_TF-01A, F.Cu at (-22.8, 156.6)
- added D1: RCLAMP0524P-N, easyeda2kicad:DFN-10L_L2.5-W1.0-P0.50-BL, F.Cu at (30.9, 177.0)
- added D2: RCLAMP0524P-N, easyeda2kicad:DFN-10L_L2.5-W1.0-P0.50-BL, F.Cu at (30.9, 179.9)
- added D3: RCLAMP0524P-N, easyeda2kicad:DFN-10L_L2.5-W1.0-P0.50-BL, F.Cu at (30.9, 182.8)
- added D4: RCLAMP0524P-N, easyeda2kicad:DFN-10L_L2.5-W1.0-P0.50-BL, F.Cu at (30.9, 185.7)
- added D5: RCLAMP0524P-N, easyeda2kicad:DFN-10L_L2.5-W1.0-P0.50-BL, F.Cu at (52.8, 188.1)
- added D6: RCLAMP0524P-N, easyeda2kicad:DFN-10L_L2.5-W1.0-P0.50-BL, F.Cu at (52.8, 191.0)
- added HDMI1: HDMI-019S, easyeda2kicad:HDMI-SMD_HDMI-019S, F.Cu at (11.8, 180.9)
- added HDMI2: HDMI-019S, easyeda2kicad:HDMI-SMD_HDMI-019S, F.Cu at (11.8, 194.6)
- added L1: 2.2uH, easyeda2kicad:IND-SMD_L3.5-W3.0, F.Cu at (-5.21, 111.1)
- added L2: HY602401, easyeda2kicad:XFMR-SMD_HY602401, F.Cu at (-2.98, 84.6)
- added L3: 6.8uH, Inductor_SMD:L_APV_APH0530, F.Cu at (12.3, 78.6)
- added L4: 6.8uH, Inductor_SMD:L_APV_APH0530, F.Cu at (12.3, 85.4)
- added L5: 6.8uH, Inductor_SMD:L_APV_APH0530, F.Cu at (12.3, 92.1)
- added Q1: 2N7002-SOT23, easyeda2kicad:SOT-23_L2.9-W1.3-P1.90-LS2.4-BR, F.Cu at (22.5, 199.7)
- added Q2: 2N7002-SOT23, easyeda2kicad:SOT-23_L2.9-W1.3-P1.90-LS2.4-BR, F.Cu at (22.5, 204.0)
- added R1: 10k, Resistor_SMD:R_0402_1005Metric, F.Cu at (63.4, 76.3)
- added R10: 12.4K, Resistor_SMD:R_0402_1005Metric, F.Cu at (58.5, 104.8)
- added R11: 120k, Resistor_SMD:R_0402_1005Metric, F.Cu at (59.3, 138.9)
- added R12: 10k, Resistor_SMD:R_0402_1005Metric, F.Cu at (59.3, 140.9)
- added R13: 10k, Resistor_SMD:R_0402_1005Metric, F.Cu at (59.3, 142.9)
- added R14: 680R, Resistor_SMD:R_0402_1005Metric, F.Cu at (0.82, 144.7)
- added R15: 10k, Resistor_SMD:R_0402_1005Metric, F.Cu at (-30.2, 106.7)
- added R16: 10k, Resistor_SMD:R_0402_1005Metric, F.Cu at (-30.2, 108.7)
- added R17: 160k, Resistor_SMD:R_0402_1005Metric, F.Cu at (-30.2, 110.7)
- added R18: 270k, Resistor_SMD:R_0402_1005Metric, F.Cu at (-30.2, 112.7)
- added R19: 10k, Resistor_SMD:R_0402_1005Metric, F.Cu at (-27.3, 106.7)
- added R2: 10K, Resistor_SMD:R_0402_1005Metric, F.Cu at (52.7, 100.8)
- added R20: 10k, Resistor_SMD:R_0402_1005Metric, F.Cu at (-27.3, 108.7)
- added R21: 1K, Resistor_SMD:R_0402_1005Metric, F.Cu at (-27.3, 110.7)
- added R22: 2.49k, Resistor_SMD:R_0402_1005Metric, F.Cu at (-27.3, 112.7)
- added R23: 75R, Resistor_SMD:R_0402_1005Metric, F.Cu at (-24.4, 106.7)
- added R24: 75R, Resistor_SMD:R_0402_1005Metric, F.Cu at (-24.4, 108.7)
- added R25: 75R, Resistor_SMD:R_0402_1005Metric, F.Cu at (-24.4, 110.7)
- added R26: 75R, Resistor_SMD:R_0402_1005Metric, F.Cu at (-24.4, 112.7)
- added R27: 160k, Resistor_SMD:R_0402_1005Metric, F.Cu at (17.6, 76.3)
- added R28: 160k, Resistor_SMD:R_0402_1005Metric, F.Cu at (17.6, 78.2)
- added R29: 160k, Resistor_SMD:R_0402_1005Metric, F.Cu at (17.6, 80.2)
- added R3: 10K, Resistor_SMD:R_0402_1005Metric, F.Cu at (52.7, 102.8)
- added R30: 150k, Resistor_SMD:R_0402_1005Metric, F.Cu at (17.6, 82.2)
- added R31: 150k, Resistor_SMD:R_0402_1005Metric, F.Cu at (17.6, 84.2)
- added R32: 150k, Resistor_SMD:R_0402_1005Metric, F.Cu at (17.6, 86.2)
- added R33: 51k, Resistor_SMD:R_0402_1005Metric, F.Cu at (17.6, 88.2)
- added R34: 51k, Resistor_SMD:R_0402_1005Metric, F.Cu at (20.5, 76.3)
- added R35: 51k, Resistor_SMD:R_0402_1005Metric, F.Cu at (20.5, 78.2)
- added R36: 3.6k, Resistor_SMD:R_0402_1005Metric, F.Cu at (20.5, 80.2)
- added R37: 3.6k, Resistor_SMD:R_0402_1005Metric, F.Cu at (20.5, 82.2)
- added R38: 3.6k, Resistor_SMD:R_0402_1005Metric, F.Cu at (20.5, 84.2)
- added R39: 220k, Resistor_SMD:R_0402_1005Metric, F.Cu at (20.5, 86.2)
- added R4: 10K, Resistor_SMD:R_0402_1005Metric, F.Cu at (52.7, 104.8)
- added R40: 43k, Resistor_SMD:R_0402_1005Metric, F.Cu at (20.5, 88.2)
- added R41: 220k, Resistor_SMD:R_0402_1005Metric, F.Cu at (23.4, 76.3)
- added R42: 43k, Resistor_SMD:R_0402_1005Metric, F.Cu at (23.4, 78.2)
- added R43: 220k, Resistor_SMD:R_0402_1005Metric, F.Cu at (23.4, 80.2)
- added R44: 43k, Resistor_SMD:R_0402_1005Metric, F.Cu at (23.4, 82.2)
- added R45: 10K, Resistor_SMD:R_0402_1005Metric, F.Cu at (52.7, 76.3)
- added R46: 10K, Resistor_SMD:R_0402_1005Metric, F.Cu at (52.7, 78.2)
- added R47: 10K, Resistor_SMD:R_0402_1005Metric, F.Cu at (52.7, 80.2)
- added R48: 10K, Resistor_SMD:R_0402_1005Metric, F.Cu at (55.6, 76.3)
- added R49: 10K, Resistor_SMD:R_0402_1005Metric, F.Cu at (55.6, 78.2)
- added R5: 10K, Resistor_SMD:R_0402_1005Metric, F.Cu at (55.6, 100.8)
- added R50: 10K, Resistor_SMD:R_0402_1005Metric, F.Cu at (55.6, 80.2)
- added R51: 47k, Resistor_SMD:R_0402_1005Metric, F.Cu at (58.5, 76.3)
- added R52: 100k, Resistor_SMD:R_0402_1005Metric, F.Cu at (58.5, 78.2)
- added R53: 12.4K, Resistor_SMD:R_0402_1005Metric, F.Cu at (58.5, 80.2)
- added R54: 120k, Resistor_SMD:R_0402_1005Metric, F.Cu at (31.7, 123.0)
- added R55: 10k, Resistor_SMD:R_0402_1005Metric, F.Cu at (31.7, 125.0)
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Connections:
- net Net-(A1-VIN-Pad250) renamed VBUS
- A1 pad 1: unconnected-(A1-~{PWRBTN}-Pad1) -> Net-(A1-~{PWRBTN})
- A1 pad 10: unconnected-(A1-SIO_UART_TX-Pad10) -> SIO_UART_TX
- A1 pad 100: unconnected-(A1-~{CLKREQ3}-Pad100) -> PCIE_CLKREQ3#
- A1 pad 101: Net-(A1-GND-Pad101) -> GND
- A1 pad 102: unconnected-(A1-~{CLKREQ4}-Pad102) -> PCIE_CLKREQ4#
- A1 pad 103: unconnected-(A1-~{WAKE}-Pad103) -> PCIE_WAKE
- A1 pad 105: unconnected-(A1-~{PLTRST}-Pad105) -> PCIE_RST
- A1 pad 106: unconnected-(A1-SMB_CLK-Pad106) -> SMB_CLK
- A1 pad 107: Net-(A1-GND-Pad101) -> GND
- A1 pad 108: unconnected-(A1-SMB_DATA-Pad108) -> SMB_DATA
- A1 pad 109: unconnected-(A1-USB2_P5--Pad109) -> USB2_P5-
- A1 pad 11: Net-(A1-GND-Pad101) -> GND
- A1 pad 110: Net-(A1-GND-Pad101) -> GND
- A1 pad 111: unconnected-(A1-USB2_P5+-Pad111) -> USB2_P5+
- A1 pad 112: unconnected-(A1-USB2_P6+-Pad112) -> DP_ALT_USB_D+
- A1 pad 113: Net-(A1-GND-Pad101) -> GND
- A1 pad 114: unconnected-(A1-USB2_P6--Pad114) -> DP_ALT_USB_D-
- A1 pad 115: unconnected-(A1-VBAT-Pad115) -> Net-(A1-VBAT)
- A1 pad 116: Net-(A1-GND-Pad101) -> GND
- A1 pad 12: unconnected-(A1-SIO_UART_RX-Pad12) -> SIO_UART_RX
- A1 pad 125: unconnected-(A1-GPP_B11-Pad125) -> PMCALERT
- A1 pad 129: unconnected-(A1-~{USB_OC}-Pad129) -> USB_OC#
- A1 pad 13: unconnected-(A1-HSIO0_TX+-Pad13) -> /USB_3/SS_HUB_0_TX+
- A1 pad 131: unconnected-(A1-SUSCLK-Pad131) -> SUSCLK_WIFI
- A1 pad 132: unconnected-(A1-GPP_D2-Pad132) -> GPP_D2
- A1 pad 133: unconnected-(A1-~{BIOS_SEL}-Pad133) -> BIOS_SEL#
- A1 pad 135: Net-(A1-GND-Pad101) -> GND
- A1 pad 136: Net-(A1-GND-Pad101) -> GND
- A1 pad 14: Net-(A1-GND-Pad101) -> GND
- A1 pad 145: unconnected-(A1-SML1_DATA-Pad145) -> SML1_DATA
- A1 pad 147: unconnected-(A1-SML1_CLK-Pad147) -> SML1_CLK
- A1 pad 15: unconnected-(A1-HSIO0_TX--Pad15) -> /USB_3/SS_HUB_0_TX-
- A1 pad 151: Net-(A1-GND-Pad101) -> GND
- A1 pad 153: unconnected-(A1-SPI_IO3-Pad153) -> BIOS_SPI_IO3
- A1 pad 154: unconnected-(A1-I2C2_SCL-Pad154) -> I2C2_SCL
- A1 pad 155: unconnected-(A1-SPI_CLK-Pad155) -> BIOS_SPI_CLK
- A1 pad 156: unconnected-(A1-I2C2_SDA-Pad156) -> I2C2_SDA
- A1 pad 158: Net-(A1-GND-Pad101) -> GND
- A1 pad 159: unconnected-(A1-SPI_MOSI/SPI_IO0-Pad159) -> BIOS_SPI_IO0
- A1 pad 16: unconnected-(A1-HSIO0_RX+-Pad16) -> /USB_3/SS_HUB_0_RX+
- A1 pad 161: unconnected-(A1-SPI_IO2-Pad161) -> BIOS_SPI_IO2
- A1 pad 163: unconnected-(A1-SPI_MISO/SPI_IO1-Pad163) -> BIOS_SPI_IO1
- A1 pad 165: unconnected-(A1-~{SPI_CS}-Pad165) -> BIOS_SPI_CS
- A1 pad 167: Net-(A1-GND-Pad101) -> GND
- A1 pad 169: unconnected-(A1-DDIB_DDC_SDA-Pad169) -> /HDMI/HDMI_0_SDA
- A1 pad 17: Net-(A1-GND-Pad101) -> GND
- A1 pad 170: Net-(A1-GND-Pad101) -> GND
- A1 pad 171: unconnected-(A1-DDIB_DDC_SCL-Pad171) -> /HDMI/HDMI_0_SCL
- A1 pad 172: unconnected-(A1-HDA_RST-Pad172) -> HDA_RST
- A1 pad 173: unconnected-(A1-TCP1_DDC_SDA-Pad173) -> /DP_ALT_USB/TCP1_SDA
- A1 pad 174: unconnected-(A1-HDA_BCLK-Pad174) -> HDA_BCLK
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
Commit message: .
Parts:
- removed L4, L5: 6.8uH, Inductor_SMD:L_APV_APH0530
- removed TP1, TP2, TP3: Vout testpoint, TestPoint:TestPoint_Pad_2.0x2.0mm
- added B1: BS-02-A1AJ010, easyeda2kicad:BAT-TH_BS-02-A1AJ010, F.Cu at (-180.6, 81.9)
- added C162: 1uF, Capacitor_SMD:C_0603_1608Metric, F.Cu at (-65.4, 100.9)
- added C163: 100nF, Capacitor_SMD:C_0402_1005Metric, F.Cu at (-61.9, 100.6)
- added C164: 100nF, Capacitor_SMD:C_0402_1005Metric, F.Cu at (-61.9, 102.6)
- added C165: 220nF, Capacitor_SMD:C_0402_1005Metric, F.Cu at (-61.9, 104.5)
- added C166: 100nF, Capacitor_SMD:C_0402_1005Metric, F.Cu at (146.7, 33.8)
- added C167: 10uF, Capacitor_SMD:C_0805_2012Metric, F.Cu at (-65.4, 103.4)
- added C168: 10uF, Capacitor_SMD:C_0805_2012Metric, F.Cu at (-65.4, 105.9)
- added C169: 10uF, Capacitor_SMD:C_0805_2012Metric, F.Cu at (-65.4, 108.4)
- added C170: 10uF, Capacitor_SMD:C_0805_2012Metric, F.Cu at (-65.4, 110.9)
- added C171: 220nF, Capacitor_SMD:C_0402_1005Metric, F.Cu at (-61.9, 106.5)
- added C172: 220nF, Capacitor_SMD:C_0402_1005Metric, F.Cu at (-61.9, 108.5)
- added C173: 220nF, Capacitor_SMD:C_0402_1005Metric, F.Cu at (-61.9, 110.4)
- added C174: 100nF, Capacitor_SMD:C_0402_1005Metric, F.Cu at (148.6, 41.0)
- added C175: 100nF, Capacitor_SMD:C_0402_1005Metric, F.Cu at (48.6, 74.2)
- added C176: 100nF, Capacitor_SMD:C_0402_1005Metric, F.Cu at (48.6, 76.2)
- added C177: 100nF, Capacitor_SMD:C_0402_1005Metric, F.Cu at (-30.1, 159.2)
- added C178: 100nF, Capacitor_SMD:C_0402_1005Metric, F.Cu at (-30.1, 161.1)
- added C179: 10uF, Capacitor_SMD:C_0805_2012Metric, F.Cu at (-33.7, 164.8)
- added C180: 100nF, Capacitor_SMD:C_0402_1005Metric, F.Cu at (-30.1, 163.1)
- added C181: 10uF, Capacitor_SMD:C_0805_2012Metric, F.Cu at (-33.7, 167.8)
- added C182: 100nF, Capacitor_SMD:C_0402_1005Metric, F.Cu at (-30.1, 165.1)
- added C183: 10uF, Capacitor_SMD:C_0805_2012Metric, F.Cu at (-33.7, 170.8)
- added C184: 100nF, Capacitor_SMD:C_0402_1005Metric, F.Cu at (-30.1, 167.1)
- added C185: 10uF, Capacitor_SMD:C_0805_2012Metric, F.Cu at (-33.7, 173.8)
- added CN5: WAFER-PH2.0-4PZZ, easyeda2kicad:CONN-TH_4P-P2.00_FWF20001-S04S22W5B, F.Cu at (30.1, 91.3)
- added CN6: 47053-1000, easyeda2kicad:CONN-TH_47053-1000, F.Cu at (29.2, 99.9)
- added CN7: PJ-393-8P_C49284725, easyeda2kicad:AUDIO-TH_PJ-393-8P, F.Cu at (70.7, 141.7)
- added D10: RCLAMP0524P-N, easyeda2kicad:DFN-10L_L2.5-W1.0-P0.50-BL, F.Cu at (147.6, 44.4)
- added D11: RCLAMP0524P-N, easyeda2kicad:DFN-10L_L2.5-W1.0-P0.50-BL, F.Cu at (123.8, 122.9)
- added D12: RCLAMP0524P-N, easyeda2kicad:DFN-10L_L2.5-W1.0-P0.50-BL, F.Cu at (122.3, 135.4)
- added D13: RCLAMP0524P-N, easyeda2kicad:DFN-10L_L2.5-W1.0-P0.50-BL, F.Cu at (90.5, 129.9)
- added D14: RCLAMP0524P-N, easyeda2kicad:DFN-10L_L2.5-W1.0-P0.50-BL, F.Cu at (108.6, 129.6)
- added D15: RCLAMP0524P-N, easyeda2kicad:DFN-10L_L2.5-W1.0-P0.50-BL, F.Cu at (-21.5, 117.1)
- added D16: RCLAMP0524P-N, easyeda2kicad:DFN-10L_L2.5-W1.0-P0.50-BL, F.Cu at (105.1, 41.5)
- added D7: RCLAMP0524P-N, easyeda2kicad:DFN-10L_L2.5-W1.0-P0.50-BL, F.Cu at (133.4, 35.0)
- added D8: RCLAMP0524P-N, easyeda2kicad:DFN-10L_L2.5-W1.0-P0.50-BL, F.Cu at (127.1, 33.4)
- added D9: RCLAMP0524P-N, easyeda2kicad:DFN-10L_L2.5-W1.0-P0.50-BL, F.Cu at (147.6, 47.1)
- added J1: USB_C_Receptacle_USB2.0_16P, Connector_USB:USB_C_Receptacle_GCT_USB4105-xx-A_16P_TopMnt_Horizontal, F.Cu at (215.8, 25.1)
- added J2: Conn_01x04_Socket, Connector_PinSocket_2.54mm:PinSocket_1x04_P2.54mm_Vertical, F.Cu at (-50.6, 31.8)
- added L6: 3.3H, Inductor_SMD:L_APV_APH1040, F.Cu at (-74.9, 105.4)
- added L7: 3.3H, Inductor_SMD:L_APV_APH1040, F.Cu at (-74.9, 116.9)
- added LED1: XL-5050SURC, easyeda2kicad:LED-ARRAY-SMD_6P-L5.0-W5.0-TL-RD-2, F.Cu at (223.4, 147.5)
- added Q3: AON7403, easyeda2kicad:PQFN-8_L3.1-W3.1-P0.65-LS3.3-BL, F.Cu at (-53.4, 114.5)
- added Q4: 2N7002-SOT23, easyeda2kicad:SOT-23_L2.9-W1.3-P1.90-LS2.4-BR, F.Cu at (-41.3, 156.4)
- added Q5: AON7402, easyeda2kicad:PDFN-8_L3.1-W3.1-P0.65-LS3.4-BL, F.Cu at (-65.2, 122.6)
- added Q6: AON7402, easyeda2kicad:PDFN-8_L3.1-W3.1-P0.65-LS3.4-BL, F.Cu at (-60.9, 122.6)
- added Q7: AON7402, easyeda2kicad:PDFN-8_L3.1-W3.1-P0.65-LS3.4-BL, F.Cu at (-56.6, 122.6)
- added Q8: AON7402, easyeda2kicad:PDFN-8_L3.1-W3.1-P0.65-LS3.4-BL, F.Cu at (-52.3, 122.6)
- added Q9: 2N7002-SOT23, easyeda2kicad:SOT-23_L2.9-W1.3-P1.90-LS2.4-BR, F.Cu at (-41.3, 160.6)
- added R100: 13k, Resistor_SMD:R_0402_1005Metric, F.Cu at (-60.1, 115.1)
- added R101: 20k, Resistor_SMD:R_0402_1005Metric, F.Cu at (-60.1, 117.1)
- added R102: 13k, Resistor_SMD:R_0402_1005Metric, F.Cu at (-60.1, 119.1)
- added R103: 20k, Resistor_SMD:R_0402_1005Metric, F.Cu at (-57.2, 113.2)
- added R104: 0R, Resistor_SMD:R_0402_1005Metric, F.Cu at (-57.2, 115.1)
- added R105: 10K, Resistor_SMD:R_0402_1005Metric, F.Cu at (-57.2, 117.1)
- added R106: 3K, Resistor_SMD:R_0402_1005Metric, F.Cu at (-57.2, 119.1)
- added R107: 120k, Resistor_SMD:R_0402_1005Metric, F.Cu at (-18.1, 106.6)
- added R108: 10k, Resistor_SMD:R_0402_1005Metric, F.Cu at (-18.1, 108.6)
- added R109: 10k, Resistor_SMD:R_0402_1005Metric, F.Cu at (-18.1, 110.6)
- added R110: 10k, Resistor_SMD:R_0402_1005Metric, F.Cu at (-32.8, 89.9)
- added R111: ?k, Resistor_SMD:R_0402_1005Metric, F.Cu at (-18.1, 112.5)
- added R112: ?k, Resistor_SMD:R_0402_1005Metric, F.Cu at (-18.1, 114.5)
- added R113: 10k, Resistor_SMD:R_0402_1005Metric, F.Cu at (-32.8, 91.9)
- added R114: 10K, Resistor_SMD:R_0402_1005Metric, F.Cu at (-37.7, 85.3)
- added R115: 1K, Resistor_SMD:R_0402_1005Metric, F.Cu at (-37.7, 87.3)
- added R91: 10R, Resistor_SMD:R_0402_1005Metric, F.Cu at (-65.9, 113.2)
- added R92: 50K, Resistor_SMD:R_0402_1005Metric, F.Cu at (-65.9, 115.1)
- added R93: 5.1K, Resistor_SMD:R_0402_1005Metric, F.Cu at (-65.9, 117.1)
- added R94: 14K, Resistor_SMD:R_0402_1005Metric, F.Cu at (-65.9, 119.1)
- added R95: 22.6k, Resistor_SMD:R_0402_1005Metric, F.Cu at (-63.0, 113.2)
- added R96: 8.2R, Resistor_SMD:R_0402_1005Metric, F.Cu at (-63.0, 115.1)
- added R97: 6.8R, Resistor_SMD:R_0402_1005Metric, F.Cu at (-63.0, 117.1)
- added R98: 30.9K, Resistor_SMD:R_0402_1005Metric, F.Cu at (-63.0, 119.1)
- added R99: 33.2K, Resistor_SMD:R_0402_1005Metric, F.Cu at (-60.1, 113.2)
- added SW1: TS-1089S-02526, easyeda2kicad:SW-SMD_4P-L4.2-W3.3-P2.15-LS5.1, F.Cu at (-79.1, 58.3)
- added SW2: TS-1089S-02526, easyeda2kicad:SW-SMD_4P-L4.2-W3.3-P2.15-LS5.1, B.Cu at (168.7, 127.8)
- added SW3: TC-1102N-C-A-B, easyeda2kicad:SW-TH_TC-1102N-C-A-B, F.Cu at (213.1, 147.7)
- added SW4: TC-1102N-C-A-B, easyeda2kicad:SW-TH_TC-1102N-C-A-B, F.Cu at (201.8, 147.6)
- added SW6: DSHP01TSGER, easyeda2kicad:SW-SMD_DSHP01TSGER, F.Cu at (-41.2, 89.3)
- added TP4: MUX3A/TXD1, TestPoint:TestPoint_Pad_D1.0mm, F.Cu at (-61.7, 142.3)
- added TP5: GP2_IT, TestPoint:TestPoint_Pad_D1.0mm, F.Cu at (-61.7, 145.4)
- added TP6: Vin TestPoint, TestPoint:TestPoint_Pad_2.0x2.0mm, F.Cu at (-71.4, 124.7)
- added U14: IT8851, Package_DFN_QFN:VQFN-28-1EP_4x4mm_P0.45mm_EP2.4x2.4mm, F.Cu at (217.5, 42.5)
- added U16: HUSB238_002DD, easyeda2kicad:DFN-10_L3.0-W3.0-P0.50-BL-EP2.5, F.Cu at (-75.6, 125.0)
- added U17: TPS51275RUKR, easyeda2kicad:WQFN-20_L3.0-W3.0-P0.40-BL-EP1.7, F.Cu at (-80.1, 125.1)
- added U18: VL162, easyeda2kicad:MQFN-28_L4.5-W3.5-P0.40-BL-EP, F.Cu at (143.8, 42.4)
- added U19: TPS54202DDCR, easyeda2kicad:SOT-23-6_L2.9-W1.6-P0.95-LS2.8-BL, F.Cu at (-118.7, 114.6)
- added U20: TPS2560DRCR, easyeda2kicad:VSON-10_L3.0-W3.0-P0.50-BL-EP_TPS62410DRCR, F.Cu at (-36.1, 120.8)
- added U21: TPS2560DRCR, easyeda2kicad:VSON-10_L3.0-W3.0-P0.50-BL-EP_TPS62410DRCR, F.Cu at (-32.0, 120.8)
- added U22: W25N01GVZEIG_C907680, easyeda2kicad:WSON-8_L8.0-W6.10-P1.27-BL-EP, F.Cu at (188.9, 123.9)
- added U23: ALC269Q-VC3-GR, easyeda2kicad:QFN-48_L7.0-W7.0-P0.50-BL-EP5.3, F.Cu at (70.0, 123.7)
- added U24: ESP32-C3-WROOM-02, RF_Module:ESP32-C3-WROOM-02, B.Cu at (179.1, 137.8)
- added USB5: AF SS-JB17.6, easyeda2kicad:USB-A-TH_AF-SS-JB17.6, F.Cu at (115.7, 34.0)
- C100: value 120pF -> 100nF
- C101, C99: value 120pF -> 10uF; footprint Capacitor_SMD:C_0402_1005Metric -> Capacitor_SMD:C_0805_2012Metric
- C71, C72, C73, C74, CN2, CN3, CN4, Card1: moved to B.Cu
- C81, C82, C83: value 10uF -> 100nF; footprint Capacitor_SMD:C_0805_2012Metric -> Capacitor_SMD:C_0402_1005Metric
- C85, C86: value 100nF -> 220uF; footprint Capacitor_SMD:C_0402_1005Metric -> Capacitor_SMD:C_Elec_6.3x7.7
- C87, C88, C89, C90, C91: value 22uF -> 220uF; footprint Capacitor_SMD:C_0805_2012Metric -> Capacitor_SMD:C_Elec_6.3x7.7
- C92: value 22uF -> 1uF; footprint Capacitor_SMD:C_0805_2012Metric -> Capacitor_SMD:C_0603_1608Metric
- C93: value 100nF -> 47pF
- C95: value 100nF -> 10uF; footprint Capacitor_SMD:C_0402_1005Metric -> Capacitor_SMD:C_0805_2012Metric
- C96: value 10nf -> 100nF
- C97, C98: value 10nf -> 1uF; footprint Capacitor_SMD:C_0402_1005Metric -> Capacitor_SMD:C_0603_1608Metric
- L3: value 6.8uH -> 8.2uH; footprint Inductor_SMD:L_APV_APH0530 -> Inductor_SMD:L_Changjiang_FXL0420
- R1: value 10k -> 27K
- R27, R28, R29: value 160k -> ?k
- R30, R31: value 150k -> 0R
- R32: value 150k -> 27K
- R33: value 51k -> 100R
- R34, R35: value 51k -> R
- R36: value 3.6k -> R
- R37, R38: value 3.6k -> 10k
- R39: value 220k -> 100R
- R40: value 43k -> 100K
- R41: value 220k -> 5.2K
- R42: value 43k -> 1K
- R43: value 220k -> 1K
- R44: value 43k -> 20K
- U10, U8: value TPS54335-1ADRCT -> TPS2560DRCR; footprint easyeda2kicad:VSON-10_L3.0-W3.0-P0.50-TL-EP -> easyeda2kicad:VSON-10_L3.0-W3.0-P0.50-BL-EP_TPS62410DRCR
- U9: value TPS54335-1ADRCT -> TPS2553DRVR-1; footprint easyeda2kicad:VSON-10_L3.0-W3.0-P0.50-TL-EP -> easyeda2kicad:WSON-6_L2.0-W2.0-P0.65-BL-EP
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Connections:
- net /USB_3/USB_HUB_0/HUB_0_PORTS/DFP3TXC+ renamed /USB_3/USB_HUB_0/HUB_0_PORTS/H0_DFP3TXC+
- net /USB_3/USB_HUB_0/HUB_0_PORTS/DFP3TXC- renamed /USB_3/USB_HUB_0/HUB_0_PORTS/H0_DFP3TXC-
- net /USB_3/USB_HUB_0/HUB_0_PORTS/DFP4TXC+ renamed /USB_3/USB_HUB_0/HUB_0_PORTS/H0_DFP4TXC+
- net /USB_3/USB_HUB_0/HUB_0_PORTS/DFP4TXC- renamed /USB_3/USB_HUB_0/HUB_0_PORTS/H0_DFP4TXC-
- net /USB_3/USB_HUB_1/HUB_1_PORTS/DFP2TX1+ renamed /USB_3/USB_HUB_1/HUB_1_PORTS/H1_DFP2TX1+
- net /USB_3/USB_HUB_1/HUB_1_PORTS/DFP2TX1- renamed /USB_3/USB_HUB_1/HUB_1_PORTS/H1_DFP2TX1-
- net /USB_3/USB_HUB_1/HUB_1_PORTS/DFP2TX2+ renamed /USB_3/USB_HUB_1/HUB_1_PORTS/H1_DFP2TX2+
- net /USB_3/USB_HUB_1/HUB_1_PORTS/DFP2TX2- renamed /USB_3/USB_HUB_1/HUB_1_PORTS/H1_DFP2TX2-
- net /USB_3/USB_HUB_1/HUB_1_PORTS/DFP3TXC+ renamed /USB_3/USB_HUB_1/HUB_1_PORTS/H1_DFP3TXC+
- net /USB_3/USB_HUB_1/HUB_1_PORTS/DFP3TXC- renamed /USB_3/USB_HUB_1/HUB_1_PORTS/H1_DFP3TXC-
- net /USB_3/USB_HUB_1/HUB_1_PORTS/DFP4TXC+ renamed /USB_3/USB_HUB_1/HUB_1_PORTS/H1_DFP4TXC+
- net /USB_3/USB_HUB_1/HUB_1_PORTS/DFP4TXC- renamed /USB_3/USB_HUB_1/HUB_1_PORTS/H1_DFP4TXC-
- net Net-(C71-Pad1) renamed /PCIE_SSD/PCIE2_L1TX-
- net Net-(C72-Pad1) renamed /PCIE_SSD/PCIE2_L1TX+
- net Net-(C73-Pad1) renamed /PCIE_SSD/PCIE2_L0TX-
- net Net-(C74-Pad1) renamed /PCIE_SSD/PCIE2_L0TX+
- net Net-(C75-Pad1) renamed /PCIE_SSD/PCIE3_L1TX-
- net Net-(C76-Pad1) renamed /PCIE_SSD/PCIE3_L1TX+
- net Net-(C77-Pad1) renamed /PCIE_SSD/PCIE3_L0TX-
- net Net-(C78-Pad1) renamed /PCIE_SSD/PCIE3_L0TX+
- net Net-(C79-Pad1) renamed /PCIE_SSD/PCIE4TX-
- net Net-(C80-Pad1) renamed /PCIE_SSD/PCIE4TX+
- net Net-(U7-HSIN) renamed /PCIE_WIFI_ETH/HSIN-
- net Net-(U7-HSIP) renamed /PCIE_WIFI_ETH/HSIN+
- net Net-(U7-HSON) renamed /PCIE_WIFI_ETH/HSON-
- net Net-(U7-HSOP) renamed /PCIE_WIFI_ETH/HSIO+
- A1 pad 1: Net-(A1-~{PWRBTN}) -> /PWR_LED_SW/PWR_SW
- A1 pad 133: BIOS_SEL# -> Net-(A1-~{BIOS_SEL})
- A1 pad 172: HDA_RST -> /ALC269Q/HDA_RST
- A1 pad 174: HDA_BCLK -> /ALC269Q/HDA_BCLK
- A1 pad 176: HDA_SYNC -> /ALC269Q/HDA_SYNC
- A1 pad 178: HDA_SDOUT -> /ALC269Q/HDA_SDOUT
- A1 pad 180: HDA_SDIN -> /ALC269Q/HDA_SDIN
- A1 pad 3: Net-(A1-~{RSTBTN}) -> /PWR_LED_SW/RST_SW
- A1 pad 5: S0_PWR_IND -> /PWR_LED_SW/S0_PWR_IND
- A1 pad 7: S3_PWR_IND -> /PWR_LED_SW/S3_PWR_IND
- A1 pad 70: USB2_P4+ -> /ESP32/ESP32_D+
- A1 pad 72: USB2_P4- -> /ESP32/ESP32_D-
- A1 pad 76: USB2_P7+ -> /USB_2_PORTS/USB2_0+
- A1 pad 78: USB2_P7- -> /USB_2_PORTS/USB2_0-
- A1 pad 82: USB2_P8+ -> /USB_2_PORTS/USB2_1+
- A1 pad 84: USB2_P8- -> /USB_2_PORTS/USB2_1-
- C100 pad 1: Net-(U9-COMP) -> +3.3V
- C101 pad 1: Net-(U10-COMP) -> +5V
- C101 pad 2: GND -> GND_AUD
- C120 pad 1: DFP2_TX_1+ -> H1_DFP2_TX_1+
- C121 pad 2: DFP2_TX_1- -> H1_DFP2_TX_1-
- C122 pad 1: DFP2_TX_2- -> H1_DFP2_TX_2-
- C123 pad 2: DFP2_TX_2+ -> H1_DFP2_TX_2+
- C48 pad 2: +3.3VA -> +3.3V
- C51 pad 2: +3.3VA -> +3.3V
- C53 pad 1: +3.3VA -> +3.3V
- C59 pad 2: +3.3VA -> +3.3V
- C60 pad 2: +3.3VA -> +3.3V
- C61 pad 2: +3.3VA -> +3.3V
- C64 pad 2: +3.3VA -> +3.3V
- C65 pad 2: +3.3VA -> +3.3V
- C81 pad 1: VBUS -> /USB_3/USB_HUB_0/GL3224/DFP1_RX-
- C81 pad 2: GND -> /USB_3/USB_HUB_0/GL3224/DFP1_DRX-
- C82 pad 1: VBUS -> /USB_3/USB_HUB_0/GL3224/DFP1_DRX+
- C82 pad 2: GND -> /USB_3/USB_HUB_0/GL3224/DFP1_RX+
- C83 pad 1: VBUS -> /USB_3/USB_HUB_0/GL3224/DFP1_TX-
- C83 pad 2: GND -> /USB_3/USB_HUB_0/GL3224/DFP1_DTX-
- C84 pad 1: VBUS -> /USB_3/USB_HUB_0/GL3224/DFP1_DTX+
- C84 pad 2: GND -> /USB_3/USB_HUB_0/GL3224/DFP1_TX+
- C85 pad 1: VBUS -> +5V_DFP3
- C86 pad 1: VBUS -> +5V_DFP4
- C87 pad 1: +3.3V_SSD1 -> +5V_DFP2
- C88 pad 1: +3.3V_SSD2 -> +5V_DFP4
- C89 pad 1: +3.3V_SSD0 -> +5V_DFP3
- C90 pad 1: +3.3V_SSD1 -> +5V_DFP2
- C91 pad 1: +3.3V_SSD2 -> +5V_DFP1
- C92 pad 1: +3.3V_SSD0 -> PD_VBUS_GATE
- C93 pad 1: Net-(U8-BOOT) -> +12V
- C93 pad 2: SW_5V -> Net-(U19-FB)
- C94 pad 1: Net-(U9-BOOT) -> Net-(U19-BOOT)
- C94 pad 2: SW_5V -> +12V
- C95 pad 1: Net-(U10-BOOT) -> +3.3V
- C95 pad 2: SW_5V -> GND
- C96 pad 1: GND -> +3.3V
- C96 pad 2: Net-(C96-Pad2) -> GND
- C97 pad 1: GND -> Net-(U23-CPVEE)
- C97 pad 2: Net-(C97-Pad2) -> GND_AUD
- C98 pad 1: GND -> Net-(U23-CBN)
- C98 pad 2: Net-(C98-Pad2) -> Net-(U23-CBP)
- C99 pad 1: Net-(U8-COMP) -> +3.3V
- CN2 pad 12: +3.3V_SSD0 -> +3.3V
- CN2 pad 14: +3.3V_SSD0 -> +3.3V
- CN2 pad 16: +3.3V_SSD0 -> +3.3V
- CN2 pad 18: +3.3V_SSD0 -> +3.3V
- CN2 pad 2: +3.3V_SSD0 -> +3.3V
- CN2 pad 4: +3.3V_SSD0 -> +3.3V
- CN2 pad 70: +3.3V_SSD0 -> +3.3V
- CN2 pad 72: +3.3V_SSD0 -> +3.3V
- CN2 pad 74: +3.3V_SSD0 -> +3.3V
- CN3 pad 12: +3.3V_SSD1 -> +3.3V
- CN3 pad 14: +3.3V_SSD1 -> +3.3V
- CN3 pad 16: +3.3V_SSD1 -> +3.3V
- CN3 pad 18: +3.3V_SSD1 -> +3.3V
- CN3 pad 2: +3.3V_SSD1 -> +3.3V
- CN3 pad 4: +3.3V_SSD1 -> +3.3V
- CN3 pad 70: +3.3V_SSD1 -> +3.3V
- CN3 pad 72: +3.3V_SSD1 -> +3.3V
- CN3 pad 74: +3.3V_SSD1 -> +3.3V
- CN4 pad 12: +3.3V_SSD2 -> +3.3V
- CN4 pad 14: +3.3V_SSD2 -> +3.3V
- CN4 pad 16: +3.3V_SSD2 -> +3.3V
- CN4 pad 18: +3.3V_SSD2 -> +3.3V
- CN4 pad 2: +3.3V_SSD2 -> +3.3V
- CN4 pad 4: +3.3V_SSD2 -> +3.3V
- CN4 pad 70: +3.3V_SSD2 -> +3.3V
- CN4 pad 72: +3.3V_SSD2 -> +3.3V
- CN4 pad 74: +3.3V_SSD2 -> +3.3V
- D3 pad 10: /HDMI/H_0_TX1- -> /HDMI/H_0_TX2+
- D3 pad 6: /HDMI/H_0_TX2+ -> /HDMI/H_0_TX1-
- D3 pad 7: /HDMI/H_0_TX2- -> /HDMI/H_0_TX1+
- D3 pad 9: /HDMI/H_0_TX1+ -> /HDMI/H_0_TX2-
- D5 pad 1: /DP_ALT_USB/DP_TX1+ -> /DP_ALT_USB/DP_RX2-
- D5 pad 10: /DP_ALT_USB/DP_TX1+ -> /DP_ALT_USB/DP_RX2-
- D5 pad 2: /DP_ALT_USB/DP_TX1- -> /DP_ALT_USB/DP_RX2+
- D5 pad 4: /DP_ALT_USB/DP_RX2- -> /DP_ALT_USB/DP_TX2+
- D5 pad 5: /DP_ALT_USB/DP_RX2+ -> /DP_ALT_USB/DP_TX2-
- D5 pad 6: /DP_ALT_USB/DP_RX2+ -> /DP_ALT_USB/DP_TX2-
- D5 pad 7: /DP_ALT_USB/DP_RX2- -> /DP_ALT_USB/DP_TX2+
- D5 pad 9: /DP_ALT_USB/DP_TX1- -> /DP_ALT_USB/DP_RX2+
- D6 pad 1: /DP_ALT_USB/DP_RX1+ -> /DP_ALT_USB/DP_RX1-
- D6 pad 10: /DP_ALT_USB/DP_RX1+ -> /DP_ALT_USB/DP_RX1-
- D6 pad 2: /DP_ALT_USB/DP_RX1- -> /DP_ALT_USB/DP_RX1+
- D6 pad 4: /DP_ALT_USB/DP_TX2- -> /DP_ALT_USB/DP_TX1+
- D6 pad 5: /DP_ALT_USB/DP_TX2+ -> /DP_ALT_USB/DP_TX1-
- D6 pad 6: /DP_ALT_USB/DP_TX2+ -> /DP_ALT_USB/DP_TX1-
- D6 pad 7: /DP_ALT_USB/DP_TX2- -> /DP_ALT_USB/DP_TX1+
- D6 pad 8: unconnected-(D6-Pad8) -> GND
- D6 pad 9: /DP_ALT_USB/DP_RX1- -> /DP_ALT_USB/DP_RX1+
- L3 pad 1: +3.3V_SSD1 -> +12V
- L3 pad 2: SW_5V -> Net-(U19-SW)
- R1 pad 1: +3.3V -> FAN2_TAC
- R1 pad 2: Net-(A1-~{PWRBTN}) -> Net-(CN6-Pad3)
- R27 pad 1: Net-(U8-VSENSE) -> GND
- R27 pad 2: +3.3V_SSD1 -> Net-(U8-ILIM)
- R28 pad 1: Net-(U9-VSENSE) -> GND
- R28 pad 2: +3.3V_SSD2 -> Net-(U9-ILIM)
- R29 pad 1: Net-(U10-VSENSE) -> GND
- R29 pad 2: +3.3V_SSD0 -> Net-(U10-ILIM)
- R30 pad 1: Net-(U8-RT) -> Net-(U10-EN1)
- R31 pad 1: Net-(U9-RT) -> Net-(U10-EN2)
- R32 pad 1: Net-(U10-RT) -> FAN1_TAC
- R32 pad 2: GND -> Net-(CN5-Pad3)
- R33 pad 1: Net-(U8-VSENSE) -> FAN1_PWM
- R33 pad 2: GND -> Net-(CN5-Pad4)
- R34 pad 1: Net-(U9-VSENSE) -> Net-(LED1-K-Pad4)
- R35 pad 1: Net-(U10-VSENSE) -> Net-(LED1-K-Pad5)
- R36 pad 1: Net-(C96-Pad2) -> Net-(LED1-K-Pad6)
- R36 pad 2: Net-(U8-COMP) -> GND
- R37 pad 1: Net-(C97-Pad2) -> +3.3V
- R37 pad 2: Net-(U9-COMP) -> /PWR_LED_SW/PWR_SW
- R38 pad 1: Net-(C98-Pad2) -> +3.3V
- R38 pad 2: Net-(U10-COMP) -> /PWR_LED_SW/RST_SW
- R39 pad 1: VBUS -> FAN2_PWM
- R39 pad 2: Net-(U8-EN) -> Net-(CN6-Pad4)
- R40 pad 1: Net-(U8-EN) -> +12V
- R40 pad 2: GND -> Net-(U19-FB)
- R41 pad 1: VBUS -> Net-(U19-FB)
- R41 pad 2: Net-(U9-EN) -> GND
- R42 pad 1: Net-(U9-EN) -> +3.3V
- R42 pad 2: GND -> BIOS_SPI_IO3
- R43 pad 1: VBUS -> BIOS_SPI_IO2
- R43 pad 2: Net-(U10-EN) -> GND
- R44 pad 1: Net-(U10-EN) -> GND_AUD
- R44 pad 2: GND -> Net-(U23-JDREF)
- R73 pad 1: /HDMI/H_0_TX2+ -> /HDMI/H_0_TX0+
- R74 pad 1: /HDMI/H_0_TX2- -> /HDMI/H_0_TX0-
- R75 pad 1: /HDMI/H_0_TX1+ -> /HDMI/H_0_CLK+
- R76 pad 1: /HDMI/H_0_TX1- -> /HDMI/H_0_CLK-
- U1 pad 20: USBOC3 -> H0_USBOC3
- U1 pad 21: USBPE3 -> H0_USBPE3
- U1 pad 39: USBPE4 -> H0_USBPE4
- U1 pad 40: USBOC4 -> H0_USBOC4
- U1 pad 75: USBOC2 -> H0_USBOC2
- U1 pad 76: USBPE2 -> H0_USBPE2
- U10 pad 1: VBUS -> GND
- U10 pad 10: Net-(U10-RT) -> unconnected-(U10-~{FAULT1}-Pad10)
- U10 pad 2: SW_5V -> +5V
- U10 pad 3: GND -> +5V
- U10 pad 4: GND -> Net-(U10-EN1)
- U10 pad 5: GND -> Net-(U10-EN2)
- U10 pad 6: Net-(U10-VSENSE) -> USB_OC#
- U10 pad 7: Net-(U10-COMP) -> Net-(U10-ILIM)
- U10 pad 8: Net-(U10-EN) -> +5V_USB2_1
- U10 pad 9: Net-(U10-BOOT) -> +5V_USB2_0
- U11 pad 20: USBOC3 -> H1_USBOC3
- U11 pad 21: USBPE3 -> H1_USBPE3
- U11 pad 3: /USB_3/USB_HUB_1/DFP1_TX+ -> /USB_3/USB_HUB_1/HUB_1_PORTS/DFP1_TX+
- U11 pad 39: USBPE4 -> H1_USBPE4
- U11 pad 4: /USB_3/USB_HUB_1/DFP1_TX- -> /USB_3/USB_HUB_1/HUB_1_PORTS/DFP1_TX-
- U11 pad 40: USBOC4 -> H1_USBOC4
- U11 pad 6: /USB_3/USB_HUB_1/DFP1_RX+ -> /USB_3/USB_HUB_1/HUB_1_PORTS/DFP1_RX+
- U11 pad 7: /USB_3/USB_HUB_1/DFP1_RX- -> /USB_3/USB_HUB_1/HUB_1_PORTS/DFP1_RX-
- U11 pad 75: USBOC2 -> H1_USBOC2
- U11 pad 76: USBPE2 -> H1_USBPE2
- U13 pad 1: CC1_DFP2 -> H1_CC1_DFP2
- U13 pad 28: CC2_DFP2 -> H1_CC2_DFP2
- U13 pad 6: DFP2_RX_1+ -> H1_DFP2_RX_1+
- U13 pad 7: DFP2_RX_1- -> H1_DFP2_RX_1-
- U13 pad 8: DFP2_RX_2- -> H1_DFP2_RX_2-
- U13 pad 9: DFP2_RX_2+ -> H1_DFP2_RX_2+
- U3 pad 1: CC1_DFP2 -> H0_CC1_DFP2
- U3 pad 28: CC2_DFP2 -> H0_CC2_DFP2
- U3 pad 6: DFP2_RX_1+ -> DFP2_H0_RX_1+
- U3 pad 7: DFP2_RX_1- -> DFP2_H0_RX_1-
- U3 pad 8: DFP2_RX_2- -> DFP2_H0_RX_2-
- U3 pad 9: DFP2_RX_2+ -> DFP2_H0_RX_2+
- U4 pad 10: /USB_3/USB_HUB_0/GL3224/DFP1_RX- -> /USB_3/USB_HUB_0/GL3224/DFP1_DTX-
- U4 pad 11: /USB_3/USB_HUB_0/GL3224/DFP1_RX+ -> /USB_3/USB_HUB_0/GL3224/DFP1_DTX+
- U4 pad 7: /USB_3/USB_HUB_0/GL3224/DFP1_TX- -> /USB_3/USB_HUB_0/GL3224/DFP1_DRX-
- U4 pad 8: /USB_3/USB_HUB_0/GL3224/DFP1_TX+ -> /USB_3/USB_HUB_0/GL3224/DFP1_DRX+
- U6 pad 5: +3.3VA -> +3.3V
- U7 pad 15: +3.3VA -> +3.3V
- U7 pad 19: +3.3VA -> +3.3V
- U7 pad 29: +3.3VA -> +3.3V
- U7 pad 33: +3.3VA -> +3.3V
- U7 pad 34: +3.3VA -> +3.3V
- U7 pad 43: +3.3VA -> +3.3V
- U7 pad 46: +3.3VA -> +3.3V
- U8 pad 1: VBUS -> GND
- U8 pad 10: Net-(U8-RT) -> H0_USBOC1
- U8 pad 2: SW_5V -> +5V
- U8 pad 3: GND -> +5V
- U8 pad 4: GND -> H0_USBPE1
- U8 pad 5: GND -> H0_USBPE2
- U8 pad 6: Net-(U8-VSENSE) -> H0_USBOC2
- U8 pad 7: Net-(U8-COMP) -> Net-(U8-ILIM)
- U8 pad 8: Net-(U8-EN) -> +5V_H0_DFP2
- U8 pad 9: Net-(U8-BOOT) -> +5V_H0_DFP1
- U9 pad 1: VBUS -> +5V_H0_DFP3
- U9 pad 2: SW_5V -> Net-(U9-ILIM)
- U9 pad 3: GND -> H0_USBOC3
- U9 pad 4: GND -> H0_USBPE3
- U9 pad 6: Net-(U9-VSENSE) -> +5V
- U9 pad 7: Net-(U9-COMP) -> GND
- USB1 pad A10: DFP2_RX_2- -> DFP2_H0_RX_2-
- USB1 pad A11: DFP2_RX_2+ -> DFP2_H0_RX_2+
- USB1 pad A2: DFP2_TX_1+ -> DFP2_H0_TX_1+
- USB1 pad A3: DFP2_TX_1- -> DFP2_H0_TX_1-
- USB1 pad A5: CC1_DFP2 -> H0_CC1_DFP2
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Routing:
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Other:
- board outline added: 189.8 x 138.6 mm
- copper layers 2 -> 4
- board text added: "2242"
- board text added: "2280"
