File: PCIE_SSD.kicad_sch (KiCad schematic)
At the start: 13 parts, among them CN2 APCI0107-P001A, CN3 APCI0107-P001A, CN4 APCI0107-P001A

Commit message: .
Connections:
- net +3.3V_SSD1 is gone; now on net +3.3V: CN3.12, CN3.14, CN3.16, CN3.18, CN3.2, CN3.4, CN3.70, CN3.72, CN3.74
- net +3.3V_SSD2 is gone; now on net +3.3V: CN4.12, CN4.14, CN4.16, CN4.18, CN4.2, CN4.4, CN4.70, CN4.72, CN4.74
- net PCIE3_L0TX+: now reaches C78.1, CN3.49
- net PCIE3_L1TX-: now reaches C75.1, CN3.35
- net PCIE2_L0TX-: now reaches C73.1, CN2.47
- net PCIE4TX-: now reaches C79.1, CN4.47
- net PCIE2_L0TX+: now reaches C74.1, CN2.49
- net PCIE4TX+: now reaches C80.1, CN4.49
- net PCIE3_L1TX+: now reaches C76.1, CN3.37
- net PCIE3_L0TX-: now reaches C77.1, CN3.47
- net PCIE2_L1TX-: now reaches C71.1, CN2.35
- net PCIE2_L1TX+: now reaches C72.1, CN2.37
- net +3.3V_SSD0 renamed +3.3V
Other:
- removed sheet SSD_PWR
- moved on the sheet: C71, C72, C73, C74, C75, C76, C77, C78, C79, C80, CN4

Commit message: .
Parts:
- added U25, U26, U27, U28: SMTWE2025MTJ, easyeda2kicad:SMD_BD4.4-L4.4-D2.8, symbol da:SMTWE2025MTJ
Connections:
- net GND: now also U25.1, U26.1, U27.1, U28.1

Commit message: .
Connections:
- removed net SUSCLK_WIFI: CN2.68, CN3.68, CN4.68
- no-connect marks 91 -> 97
Changed lines of the file:
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@@
+	)
+	(no_connect
+		(at 72.39 74.93)
 	)
 	(no_connect
@@
 	)
 	(no_connect
+		(at 255.27 104.14)
+	)
+	(no_connect
 		(at 240.03 71.12)
 	)
@@
 	)
 	(no_connect
+		(at 161.29 76.2)
+	)
+	(no_connect
 		(at 72.39 100.33)
 	)
@@
 	)
 	(no_connect
+		(at 72.39 105.41)
+	)
+	(no_connect
 		(at 72.39 64.77)
 	)
@@
 	)
 	(no_connect
+		(at 161.29 106.68)
+	)
+	(no_connect
 		(at 161.29 83.82)
 	)
 	(no_connect
 		(at 240.03 35.56)
+	)
+	(no_connect
+		(at 255.27 73.66)
 	)
 	(no_connect
@@
 		)
 	)
-	(global_label "SUSCLK_WIFI"
-		(shape input)
-		(at 255.27 104.14 0)
-		(fields_autoplaced yes)
-		(effects
-			(font
-				(size 1.27 1.27)
-			)
-			(justify left)
-		)
-		(property "Intersheetrefs" "${INTERSHEET_REFS}"
-			(at 270.29 104.14 0)
-			(effects
-				(font
-					(size 1.27 1.27)
-				)
-				(justify left)
-				(hide yes)
-			)
-		)
-	)
-	(global_label "SUSCLK_WIFI"
-		(shape input)
-		(at 161.29 106.68 0)
-		(fields_autoplaced yes)
-		(effects
-			(font
-				(size 1.27 1.27)
-			)
-			(justify left)
-		)
-		(property "Intersheetrefs" "${INTERSHEET_REFS}"
-			(at 176.31 106.68 0)
-			(effects
-				(font
-					(size 1.27 1.27)
-				)
-				(justify left)
-				(hide yes)
-			)
-		)
-	)
 	(global_label "PCIE_RST"
 		(shape input)
@@
 			(effects
 				(font
-					(size 1.27 1.27)
-				)
-				(justify left)
-				(hide yes)
-			)
-		)
-	)
-	(global_label "SUSCLK_WIFI"
-		(shape input)
-		(at 72.39 105.41 0)
-		(fields_autoplaced yes)
-		(effects
-			(font
-				(size 1.27 1.27)
-			)
-			(justify left)
-		)
-		(property "Intersheetrefs" "${INTERSHEET_REFS}"
-			(at 87.41 105.41 0)
-			(effects
-				(font
