File: TYPE_C_PORTS_1.kicad_sch (KiCad schematic)
At the start: 8 parts

Commit message: .
Connections:
- net DFP1_RX_2+: now also D9.5, D9.6; no longer D10.5, D10.6
- net DFP1_RX_2-: now also D9.4, D9.7; no longer D10.4, D10.7
- net DFP1_TX_2+: now also D10.5, D10.6; no longer D9.5, D9.6
- net DFP1_TX_2-: now also D10.4, D10.7; no longer D9.4, D9.7

Commit message: .
Connections:
- net +5V_DFP1: no longer C91.1, USB7.B4 (VBUS), USB7.B9 (VBUS)
- net +5V_DFP2: no longer C90.1, USB4.B4 (VBUS), USB4.B9 (VBUS)
- new net +5V_H1_DFP3: C90.1, USB4.B4 (VBUS), USB4.B9 (VBUS)
- new net +5V_H1_DFP4: C91.1, USB7.B4 (VBUS), USB7.B9 (VBUS)
Changed lines of the file:
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@@
 			)
 		)
-		(property "Value" "+5V_DFP2"
+		(property "Value" "+5V_H1_DFP3"
 			(at 129.54 39.37 0)
 			(effects
@@
 			)
 		)
-		(property "Value" "+5V_DFP1"
-			(at 130.81 105.4099 0)
-			(effects
-				(font
-					(size 1.27 1.27)
-				)
-				(justify right)
-			)
-		)
+		(property "Value" "+5V_H1_DFP4"
+			(at 128.27 101.6 0)
+			(effects
+				(font
+					(size 1.27 1.27)
+				)
+			)
+		)

Commit message: .
Connections:
- net +5V_DFP1 is gone; now on net +5V_H1_DFP4: USB7.A4 (VBUS), USB7.A9 (VBUS)
- net +5V_DFP2 is gone; now on net +5V_H1_DFP3: USB4.A4 (VBUS), USB4.A9 (VBUS)
Changed lines of the file:
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@@
 			)
 		)
-		(property "Value" "+5V_DFP1"
+		(property "Value" "+5V_H1_DFP4"
 			(at 44.45 117.856 0)
 			(effects
@@
 			)
 		)
-		(property "Value" "+5V_DFP2"
+		(property "Value" "+5V_H1_DFP3"
 			(at 45.72 55.626 0)
 			(effects
