File: ALC269Q.kicad_sch (KiCad schematic)
At the start: 19 parts, among them CN7 PJ-393-8P_C49284725, U23 ALC269Q-VC3-GR

Commit message: .
Connections:
- net AUDIO_R: now also CN7.2, CN7.6; no longer CN7.4, CN7.8
- net MIC: now also CN7.4, CN7.8; no longer CN7.2, CN7.6
Changed lines of the file:
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@@
+	)
+	(junction
+		(at 43.18 137.16)
+		(diameter 0)
+		(color 0 0 0 0)
 	)
 	(junction
@@
 	)
 	(junction
-		(at 43.18 137.16)
-		(diameter 0)
-		(color 0 0 0 0)
-	)
-	(junction
 		(at 222.25 68.58)
 		(diameter 0)
@@
 			(width 0)
 			(type default)
-		)
-	)
-	(global_label "AUDIO_R"
-		(shape input)
-		(at 43.18 132.08 0)
-		(fields_autoplaced yes)
-		(effects
-			(font
-				(size 1.27 1.27)
-			)
-			(justify left)
-		)
-		(property "Intersheetrefs" "${INTERSHEET_REFS}"
-			(at 54.0272 132.08 0)
-			(effects
-				(font
-					(size 1.27 1.27)
-				)
-				(justify left)
-				(hide yes)
-			)
 		)
 	)
@@
 		)
 	)
+	(global_label "AUDIO_R"
+		(shape input)
+		(at 43.18 142.24 0)
+		(fields_autoplaced yes)
+		(effects
+			(font
+				(size 1.27 1.27)
+			)
+			(justify left)
+		)
+		(property "Intersheetrefs" "${INTERSHEET_REFS}"
+			(at 54.0272 142.24 0)
+			(effects
+				(font
+					(size 1.27 1.27)
+				)
+				(justify left)
+				(hide yes)
+			)
+		)
+	)
+	(global_label "AUDIO_R"
+		(shape input)
+		(at 146.05 83.82 0)
+		(fields_autoplaced yes)
+		(effects
+			(font
+				(size 1.27 1.27)
+			)
+			(justify left)
+		)
+		(property "Intersheetrefs" "${INTERSHEET_REFS}"
+			(at 156.8972 83.82 0)
+			(effects
+				(font
+					(size 1.27 1.27)
+				)
+				(justify left)
+				(hide yes)
+			)
+		)
+	)
 	(global_label "AUDIO_L"
 		(shape input)
@@
 		)
 	)
-	(global_label "AUDIO_R"
-		(shape input)
-		(at 146.05 83.82 0)
-		(fields_autoplaced yes)
-		(effects
-			(font
-				(size 1.27 1.27)
-			)
-			(justify left)
-		)
-		(property "Intersheetrefs" "${INTERSHEET_REFS}"
-			(at 156.8972 83.82 0)
-			(effects
-				(font
-					(size 1.27 1.27)
-				)
-				(justify left)
-				(hide yes)
-			)
-		)
-	)
 	(global_label "AUDIO_L"
 		(shape input)
@@
 	(global_label "MIC"
 		(shape input)
-		(at 43.18 142.24 0)
+		(at 43.18 132.08 0)
 		(fields_autoplaced yes)
 		(effects
@@
 		)
 		(property "Intersheetrefs" "${INTERSHEET_REFS}"
-			(at 49.4914 142.24 0)
+			(at 49.4914 132.08 0)
 			(effects
 				(font

Commit message: .
Parts:
- added C189, C190, C191, C192: 10uF, Capacitor_SMD:C_0805_2012Metric, symbol Device:C
- added R128: 39.2K, Resistor_SMD:R_0402_1005Metric, symbol Device:R
- added R129: 20K, Resistor_SMD:R_0402_1005Metric, symbol Device:R
- added R130, R131: 2.2K, Resistor_SMD:R_0402_1005Metric, symbol Device:R
- added R132, R45: 1k, Resistor_SMD:R_0402_1005Metric, symbol Device:R
- added R133, R134: 75R, Resistor_SMD:R_0402_1005Metric, symbol Device:R
- added TP1: PD#, TestPoint:TestPoint_Pad_D1.0mm, symbol Connector:TestPoint
Connections:
- net AUDIO_L: now also R134.1; no longer CN7.1, CN7.5
- net AUDIO_R: now also R133.2; no longer CN7.2, CN7.6
- net GND_AUD: now also U23.31 (CPVREF)
- net MIC: now also C189.1, C190.1, R130.2, R131.2; no longer CN7.8, U23.21 (MIC1-L), U23.22 (MIC1-R)
- net SenseA: now reaches U23.13 (SenseA)
- net SenseA: now also R128.1, R129.1
- net at U23.28 (MIC1-VREFO-L): now also R131.1
- net at U23.30 (MIC1-VREFO-R): now also R130.1
- net at U23.4 (~{PD}): now also TP1.1
- new net: C189.2, R132.1
- new net: R132.2, U23.21 (MIC1-L)
- new net: C191.2, R133.1
- new net: R45.1, U23.22 (MIC1-R)
- new net: C192.2, R134.2
- new net: C190.2, R45.2
- new net AUDIO_L_OUT: C192.1, CN7.5
- new net AUDIO_R_OUT: C191.1, CN7.2, CN7.6
- new net HP-SENSE: CN7.1, R128.2
- new net MIC-SENSE: CN7.8, R129.2
- no-connect marks 19 -> 18
Other:
- moved on the sheet: C97
