File: ALC269Q.kicad_sch (KiCad schematic)
At the start: 32 parts, among them CN7 PJ-393-8P_C49284725, U23 ALC269Q-VC3-GR

Commit message: .
Parts:
- C101, C179, C181, C183, C185, C189, C190, C191, C192, C95, C99: value 10uF -> 22uF
Changed lines of the file:
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@@
 		(dnp no)
 		(property "Reference" "C182"
-			(at 218.44 71.1199 0)
+			(at 230.632 71.374 0)
 			(effects
 				(font
@@
 		)
 		(property "Value" "100nF"
-			(at 218.694 73.914 0)
+			(at 230.886 74.1681 0)
 			(effects
 				(font
@@
 		(fields_autoplaced yes)
 		(property "Reference" "C179"
-			(at 205.74 101.5999 0)
+			(at 213.36 101.5999 0)
 			(effects
 				(font
 					(size 1.27 1.27)
 				)
-				(justify left)
+				(justify right)
 			)
 		)
-		(property "Value" "10uF"
-			(at 205.74 104.1399 0)
+		(property "Value" "22uF"
+			(at 213.36 104.1399 0)
 			(effects
 				(font
 					(size 1.27 1.27)
 				)
-				(justify left)
+				(justify right)
 			)
 		)
@@
 			)
 		)
-		(property "Value" "10uF"
+		(property "Value" "22uF"
 			(at 52.07 71.1199 0)
 			(effects
@@
 		(on_board yes)
 		(dnp no)
-		(fields_autoplaced yes)
 		(property "Reference" "C191"
-			(at 172.72 139.7 90)
+			(at 173.482 136.652 90)
 			(effects
 				(font
@@
 			)
 		)
-		(property "Value" "10uF"
-			(at 172.72 137.16 90)
+		(property "Value" "22uF"
+			(at 173.482 139.192 90)
 			(effects
 				(font
@@
 		(fields_autoplaced yes)
 		(property "Reference" "C183"
-			(at 229.87 71.1199 0)
+			(at 237.49 71.1199 0)
 			(effects
 				(font
 					(size 1.27 1.27)
 				)
-				(justify left)
+				(justify right)
 			)
 		)
-		(property "Value" "10uF"
-			(at 229.87 73.6599 0)
+		(property "Value" "22uF"
+			(at 237.49 73.6599 0)
 			(effects
 				(font
 					(size 1.27 1.27)
 				)
-				(justify left)
+				(justify right)
 			)
 		)
@@
 		(fields_autoplaced yes)
 		(property "Reference" "C101"
-			(at 177.8 106.6799 0)
+			(at 185.42 106.6799 0)
 			(effects
 				(font
 					(size 1.27 1.27)
 				)
-				(justify left)
+				(justify right)
 			)
 		)
-		(property "Value" "10uF"
-			(at 177.8 109.2199 0)
+		(property "Value" "22uF"
+			(at 185.42 109.2199 0)
 			(effects
 				(font
 					(size 1.27 1.27)
 				)
-				(justify left)
+				(justify right)
 			)
 		)
@@
 			)
 		)
-		(property "Value" "10uF"
+		(property "Value" "22uF"
 			(at 30.48 50.7999 0)
 			(effects
@@
 		(fields_autoplaced yes)
 		(property "Reference" "C181"
-			(at 200.66 77.4699 0)
+			(at 208.28 77.4699 0)
 			(effects
 				(font
 					(size 1.27 1.27)
 				)
-				(justify left)
+				(justify right)
 			)
 		)
-		(property "Value" "10uF"
-			(at 200.66 80.0099 0)
+		(property "Value" "22uF"
+			(at 208.28 80.0099 0)
 			(effects
 				(font
 					(size 1.27 1.27)
 				)
-				(justify left)
+				(justify right)
 			)
 		)
@@
 			)
 		)
-		(property "Value" "10uF"
+		(property "Value" "22uF"
 			(at 58.42 104.14 90)
 			(effects
@@
 			)
 		)
-		(property "Value" "10uF"
+		(property "Value" "22uF"
 			(at 52.07 91.44 90)
 			(effects
@@
 		(fields_autoplaced yes)
 		(property "Reference" "C185"
-			(at 229.87 53.3399 0)
+			(at 237.49 53.3399 0)
 			(effects
 				(font
 					(size 1.27 1.27)
 				)
-				(justify left)
+				(justify right)
 			)
 		)
-		(property "Value" "10uF"
-			(at 229.87 55.8799 0)
+		(property "Value" "22uF"
+			(at 237.49 55.8799 0)
 			(effects
 				(font
 					(size 1.27 1.27)
 				)
-				(justify left)
+				(justify right)
 			)
 		)
@@
 			)
 		)
-		(property "Value" "10uF"
+		(property "Value" "22uF"
 			(at 166.37 124.46 90)
 			(effects
@@
 		(on_board yes)
 		(dnp no)
-		(fields_autoplaced yes)
 		(property "Reference" "C180"
-			(at 189.23 77.4699 0)
+			(at 201.422 77.724 0)
 			(effects
 				(font
@@
 		)
 		(property "Value" "100nF"
-			(at 189.23 80.0099 0)
+			(at 201.422 80.264 0)
 			(effects
 				(font
