File: MiniLatte.kicad_sch (KiCad schematic)
At the start: 1 part

Commit message: .
Parts:
- added BT1: Battery, symbol Device:Battery
- added R1: 10k, Resistor_SMD:R_0402_1005Metric, symbol Device:R
- added SW1, SW2: SW_Push, symbol Switch:SW_Push
Connections:
- net at A1.1 (~{PWRBTN}): now also R1.2, SW1.2
- net SIO_UART_TX: now reaches A1.10 (SIO_UART_TX)
- net PCIE_CLKREQ3#: now reaches A1.100 (~{CLKREQ3})
- net GND: now reaches A1.101 (GND), A1.107 (GND), A1.11 (GND), A1.110 (GND), A1.113 (GND), A1.116 (GND), A1.135 (GND), A1.136 (GND), A1.14 (GND), A1.151 (GND), A1.158 (GND), A1.167 (GND), A1.17 (GND), A1.170 (GND), A1.181 (GND), A1.182 (GND), A1.188 (GND), A1.189 (GND), A1.194 (GND), A1.195 (GND), A1.20 (GND), A1.200 (GND), A1.201 (GND), A1.206 (GND), A1.207 (GND), A1.212 (GND), A1.213 (GND), A1.218 (GND), A1.219 (GND), A1.224 (GND), A1.225 (GND), A1.23 (GND), A1.230 (GND), A1.231 (GND), A1.236 (GND), A1.237 (GND), A1.242 (GND), A1.243 (GND), A1.248 (GND), A1.249 (GND), A1.26 (GND), A1.29 (GND), A1.32 (GND), A1.35 (GND), A1.38 (GND), A1.41 (GND), A1.44 (GND), A1.47 (GND), A1.50 (GND), A1.53 (GND), A1.56 (GND), A1.59 (GND), A1.62 (GND), A1.65 (GND), A1.68 (GND), A1.71 (GND), A1.74 (GND), A1.77 (GND), A1.80 (GND), A1.83 (GND), A1.86 (GND), A1.89 (GND), A1.92 (GND), A1.95 (GND), A1.98 (GND)
- net GND: now also A1.MP (Mountinge_Pads), BT1.2 (-), SW1.1, SW2.1
- net PCIE_CLKREQ4#: now reaches A1.102 (~{CLKREQ4})
- net PCIE_WAKE: now reaches A1.103 (~{WAKE})
- net PCIE_RST: now reaches A1.105 (~{PLTRST})
- net SMB_CLK: now reaches A1.106 (SMB_CLK)
- net SMB_DATA: now reaches A1.108 (SMB_DATA)
- net USB2_P5-: now reaches A1.109 (USB2_P5-)
- net USB2_P5+: now reaches A1.111 (USB2_P5+)
- net DP_ALT_USB_D+: now reaches A1.112 (USB2_P6+)
- net DP_ALT_USB_D-: now reaches A1.114 (USB2_P6-)
- net at A1.115 (VBAT): now also BT1.1 (+)
- net SIO_UART_RX: now reaches A1.12 (SIO_UART_RX)
- net PMCALERT: now reaches A1.125 (GPP_B11)
- net USB_OC#: now reaches A1.129 (~{USB_OC})
- net SUSCLK_WIFI: now reaches A1.131 (SUSCLK)
- net BIOS_SEL#: now reaches A1.133 (~{BIOS_SEL})
- net SML1_DATA: now reaches A1.145 (SML1_DATA)
- net SML1_CLK: now reaches A1.147 (SML1_CLK)
- net BIOS_SPI_IO3: now reaches A1.153 (SPI_IO3)
- net I2C2_SCL: now reaches A1.154 (I2C2_SCL)
- net BIOS_SPI_CLK: now reaches A1.155 (SPI_CLK)
- net I2C2_SDA: now reaches A1.156 (I2C2_SDA)
- net BIOS_SPI_IO0: now reaches A1.159 (SPI_MOSI/SPI_IO0)
- net BIOS_SPI_IO2: now reaches A1.161 (SPI_IO2)
- net BIOS_SPI_IO1: now reaches A1.163 (SPI_MISO/SPI_IO1)
- net BIOS_SPI_CS: now reaches A1.165 (~{SPI_CS})
- net HDMI/HDMI_0_SDA: now reaches A1.169 (DDIB_DDC_SDA)
- net HDMI/HDMI_0_SCL: now reaches A1.171 (DDIB_DDC_SCL)
- net HDA_RST: now reaches A1.172 (HDA_RST)
- net HDA_BCLK: now reaches A1.174 (HDA_BCLK)
- net HDA_SYNC: now reaches A1.176 (HDA_SYNC)
- net HDMI/HDMI_1_SDA: now reaches A1.177 (TCP0_DDC_SDA)
- net HDA_SDOUT: now reaches A1.178 (HDA_SDOUT)
- net HDMI/HDMI_1_SCL: now reaches A1.179 (TCP0_DDC_SCL)
- net HDA_SDIN: now reaches A1.180 (HDA_SDIN)
- net HDMI/HDMI_0_HPD: now reaches A1.183 (DDIB_HPD)
- net DP_ALT_HPD: now reaches A1.185 (TCP1_HPD)
- net HDMI/HDMI_1_HPD: now reaches A1.187 (TCP0_HPD)
- net HDMI/HDMI_0_CLK-: now reaches A1.197 (DDIB_TX3-)
- net HDMI/HDMI_0_CLK+: now reaches A1.199 (DDIB_TX3+)
- net FAN1_PWM: now reaches A1.2 (FAN1_PWM)
- net HDMI/HDMI_0_TX0-: now reaches A1.203 (DDIB_TX2-)
- net HDMI/HDMI_0_TX0+: now reaches A1.205 (DDIB_TX2+)
- net HDMI/HDMI_0_TX1-: now reaches A1.209 (DDIB_TX1-)
- net HDMI/HDMI_0_TX1+: now reaches A1.211 (DDIB_TX1+)
- net HDMI/HDMI_0_TX2-: now reaches A1.215 (DDIB_TX0-)
- net HDMI/HDMI_0_TX2+: now reaches A1.217 (DDIB_TX0+)
- net DP_ALT_TX1+: now reaches A1.220 (TCP1_TX0+)
- net DP_ALT_TX1-: now reaches A1.222 (TCP1_TX0-)
- net DP_ALT_RX1+: now reaches A1.226 (TCP1_TXRX0+)
- net HDMI/HDMI_1_CLK-: now reaches A1.227 (TCP0_TXRX1-)
- net DP_ALT_RX1-: now reaches A1.228 (TCP1_TXRX0-)
- net HDMI/HDMI_1_CLK+: now reaches A1.229 (TCP0_TXRX1+)
- net DP_ALT_TX2+: now reaches A1.232 (TCP1_TX1+)
- net HDMI/HDMI_1_TX0-: now reaches A1.233 (TCP0_TX1-)
- net DP_ALT_TX2-: now reaches A1.234 (TCP1_TX1-)
- net HDMI/HDMI_1_TX0+: now reaches A1.235 (TCP0_TX1+)
- net DP_ALT_RX2+: now reaches A1.238 (TCP1_TXRX1+)
- net HDMI/HDMI_1_TX1-: now reaches A1.239 (TCP0_TXRX0-)
- net DP_ALT_RX2-: now reaches A1.240 (TCP1_TXRX1-)
- net HDMI/HDMI_1_TX1+: now reaches A1.241 (TCP0_TXRX0+)
- net DP_ALT_AUX+: now reaches A1.244 (TCP1_AUX+)
- net HDMI/HDMI_1_TX2-: now reaches A1.245 (TCP0_TX0-)
- net DP_ALT_AUX-: now reaches A1.246 (TCP1_AUX-)
- net HDMI/HDMI_1_TX2+: now reaches A1.247 (TCP0_TX0+)
- net VBUS: now reaches A1.250 (VIN), A1.251 (VIN), A1.252 (VIN), A1.253 (VIN), A1.254 (VIN), A1.255 (VIN), A1.256 (VIN), A1.257 (VIN), A1.258 (VIN), A1.259 (VIN), A1.260 (VIN)
- net at A1.3 (~{RSTBTN}): now also SW2.2
- net FAN1_TAC: now reaches A1.4 (FAN1_TAC)
- net S0_PWR_IND: now reaches A1.5 (SLS_S0)
- net FAN2_PWM: now reaches A1.6 (FAN2_PWM)
- net USB2_P1-: now reaches A1.67 (USB2_P1-)
- net USB2_P1+: now reaches A1.69 (USB2_P1+)
- net S3_PWR_IND: now reaches A1.7 (SLS_S3)
- net USB2_P4+: now reaches A1.70 (USB2_P4+)
- net USB2_P4-: now reaches A1.72 (USB2_P4-)
- net USB2_P2-: now reaches A1.73 (USB2_P2-)
- net USB2_P2+: now reaches A1.75 (USB2_P2+)
- net USB2_P7+: now reaches A1.76 (USB2_P7+)
- net USB2_P7-: now reaches A1.78 (USB2_P7-)
- net USB2_P3-: now reaches A1.79 (USB2_P3-)
- net FAN2_TAC: now reaches A1.8 (FAN2_TAC)
- net USB2_P3+: now reaches A1.81 (USB2_P3+)
- net USB2_P8+: now reaches A1.82 (USB2_P8+)
- net USB2_P8-: now reaches A1.84 (USB2_P8-)
- net PCIE_0_CLK+: now reaches A1.85 (REFCLK0+)
- net PCIE_0_CLK-: now reaches A1.87 (REFCLK0-)
- net PCIE_3_CLK+: now reaches A1.88 (REFCLK3+)
- net PCIE_3_CLK-: now reaches A1.90 (REFCLK3-)
- net PCIE_1_CLK+: now reaches A1.91 (REFCLK1+)
- net PCIE_1_CLK-: now reaches A1.93 (REFCLK1-)
- net PCIE_4_CLK+: now reaches A1.94 (REFCLK4+)
- net PCIE_4_CLK-: now reaches A1.96 (REFCLK4-)
- net PCIE_2_CLK+: now reaches A1.97 (REFCLK2+)
- net PCIE_2_CLK-: now reaches A1.99 (REFCLK2-)
- net PCIE_0_RX+ renamed PCIE_WIFI_ETH/PCIE_0_RX+
- net PCIE_0_RX- renamed PCIE_WIFI_ETH/PCIE_0_RX-
- net PCIE_0_TX+ renamed PCIE_WIFI_ETH/PCIE_0_TX+
- net PCIE_0_TX- renamed PCIE_WIFI_ETH/PCIE_0_TX-
- net PCIE_1_RX+ renamed PCIE_WIFI_ETH/PCIE_1_RX+
- net PCIE_1_RX- renamed PCIE_WIFI_ETH/PCIE_1_RX-
- net PCIE_1_TX+ renamed PCIE_WIFI_ETH/PCIE_1_TX+
- net PCIE_1_TX- renamed PCIE_WIFI_ETH/PCIE_1_TX-
- net PCIE_2_L0_RX+ renamed PCIE_SSD/PCIE_2_L0_RX+
- net PCIE_2_L0_RX- renamed PCIE_SSD/PCIE_2_L0_RX-
- net PCIE_2_L0_TX+ renamed PCIE_SSD/PCIE_2_L0_TX+
- net PCIE_2_L0_TX- renamed PCIE_SSD/PCIE_2_L0_TX-
- net PCIE_2_L1_RX+ renamed PCIE_SSD/PCIE_2_L1_RX+
- net PCIE_2_L1_RX- renamed PCIE_SSD/PCIE_2_L1_RX-
- net PCIE_2_L1_TX+ renamed PCIE_SSD/PCIE_2_L1_TX+
- net PCIE_2_L1_TX- renamed PCIE_SSD/PCIE_2_L1_TX-
- net PCIE_3_L0_RX+ renamed PCIE_SSD/PCIE_3_L0_RX+
- net PCIE_3_L0_RX- renamed PCIE_SSD/PCIE_3_L0_RX-
- net PCIE_3_L0_TX+ renamed PCIE_SSD/PCIE_3_L0_TX+
- net PCIE_3_L0_TX- renamed PCIE_SSD/PCIE_3_L0_TX-
- net PCIE_3_L1_RX+ renamed PCIE_SSD/PCIE_3_L1_RX+
- net PCIE_3_L1_RX- renamed PCIE_SSD/PCIE_3_L1_RX-
- net PCIE_3_L1_TX+ renamed PCIE_SSD/PCIE_3_L1_TX+
- net PCIE_3_L1_TX- renamed PCIE_SSD/PCIE_3_L1_TX-
- net PCIE_4_RX+ renamed PCIE_SSD/PCIE_4_RX+
- net PCIE_4_RX- renamed PCIE_SSD/PCIE_4_RX-
- net PCIE_4_TX+ renamed PCIE_SSD/PCIE_4_TX+
- net PCIE_4_TX- renamed PCIE_SSD/PCIE_4_TX-
- net SS_HUB_0_RX+ renamed USB_3/SS_HUB_0_RX+
- net SS_HUB_0_RX- renamed USB_3/SS_HUB_0_RX-
- net SS_HUB_0_TX+ renamed USB_3/SS_HUB_0_TX+
- net SS_HUB_0_TX- renamed USB_3/SS_HUB_0_TX-
- net SS_HUB_1_RX+ renamed USB_3/SS_HUB_1_RX+
- net SS_HUB_1_RX- renamed USB_3/SS_HUB_1_RX-
- net SS_HUB_1_TX+ renamed USB_3/SS_HUB_1_TX+
- net SS_HUB_1_TX- renamed USB_3/SS_HUB_1_TX-
- new net +3.3V: R1.1
- no-connect marks 0 -> 40
Other:
- added sheet HDMI (HDMI.kicad_sch)
- added sheet PCIE_SSD (PCIE_SSD.kicad_sch)
- added sheet PCIE_WIFI_ETH (PCIE_WIFI_ETH.kicad_sch)
- added sheet USB_3 (USB_3.kicad_sch)
- note added: "Not actual RX/TX, using usb conenctor names for easier management"
- note added: "P1: HUB0 P2: HUB1 P3: PCIE_WIFI"
- note added: "TO DO power for all ic"
- note added: "TO do HUB1"
- note added: "to read more on usb oc"
- moved on the sheet: A1

Commit message: .
Connections:
- net GPP_D2: now reaches A1.132 (GPP_D2)
- net DP_ALT_USB/TCP1_SDA: now reaches A1.173 (TCP1_DDC_SDA)
- net DP_ALT_USB/TCP1_SCL: now reaches A1.175 (TCP1_DDC_SCL)
- net DP_ALT_AUX+ renamed DP_ALT_USB/DP_ALT_AUX+
- net DP_ALT_AUX- renamed DP_ALT_USB/DP_ALT_AUX-
- net DP_ALT_HPD renamed DP_ALT_USB/DP_ALT_HPD
- net DP_ALT_RX1+ renamed DP_ALT_USB/DP_ALT_RX1+
- net DP_ALT_RX1- renamed DP_ALT_USB/DP_ALT_RX1-
- net DP_ALT_RX2+ renamed DP_ALT_USB/DP_ALT_RX2+
- net DP_ALT_RX2- renamed DP_ALT_USB/DP_ALT_RX2-
- net DP_ALT_TX1+ renamed DP_ALT_USB/DP_ALT_TX1+
- net DP_ALT_TX1- renamed DP_ALT_USB/DP_ALT_TX1-
- net DP_ALT_TX2+ renamed DP_ALT_USB/DP_ALT_TX2+
- net DP_ALT_TX2- renamed DP_ALT_USB/DP_ALT_TX2-
- no-connect marks 40 -> 37
Other:
- added sheet DP_ALT_USB (DP_ALT_USB.kicad_sch)
- added sheet PD_Power (PD_Power.kicad_sch)
- note added: "HUB0: - HSIO0: USB3.2 10Gbps HUB1: - HSIO1: USB3.2 10Gbps ETH: - HSIO2: PCIe 3.0 x1 WIFI: - HSIO3: PCIe 3.0 x1 SSD0: - HSIO8: PCIe 3.0 x2 (Lane 0) - HSIO9: PCIe 3.0 x2 (Lane 1) SSD1: - HSIO10: PCIe 3.0 x2 (Lane 0) - HSIO11: PCIe 3.0 x2 (Lane 1) SSD2: - HSIO6: PCIe 3.0 x1"
- note added: "Video: - DDIB: HDMI 2.0 - TCP0: HDMI 2.0 - TCP1: USB TypeC DP ALT MODE"

Commit message: .
Parts:
- removed BT1: Battery, symbol Device:Battery
- removed SW1, SW2: SW_Push, symbol Switch:SW_Push
- added B1: BS-02-A1AJ010, easyeda2kicad:BAT-TH_BS-02-A1AJ010, symbol da:BS-02-A1AJ010
- added C92: 1uF, Capacitor_SMD:C_0603_1608Metric, symbol Device:C
- added C93: 47pF, Capacitor_SMD:C_0402_1005Metric, symbol Device:C
- added C94: 100nF, Capacitor_SMD:C_0402_1005Metric, symbol Device:C
- added CN5: WAFER-PH2.0-4PZZ, easyeda2kicad:CONN-TH_4P-P2.00_FWF20001-S04S22W5B, symbol da:WAFER-PH2.0-4PZZ
- added CN6: 47053-1000, easyeda2kicad:CONN-TH_47053-1000, symbol da:47053-1000
- added L3: 8.2uH, Inductor_SMD:L_Changjiang_FXL0420, symbol Device:L
- added R114: 10K, Resistor_SMD:R_0402_1005Metric, symbol Device:R
- added R115, R42, R43: 1K, Resistor_SMD:R_0402_1005Metric, symbol Device:R
- added R32: 27K, Resistor_SMD:R_0402_1005Metric, symbol Device:R
- added R33, R39: 100R, Resistor_SMD:R_0402_1005Metric, symbol Device:R
- added R40: 100K, Resistor_SMD:R_0402_1005Metric, symbol Device:R
- added R41: 5.2K, Resistor_SMD:R_0402_1005Metric, symbol Device:R
- added SW6: DSHP01TSGER, easyeda2kicad:SW-SMD_DSHP01TSGER, symbol da:DSHP01TSGER
- added U19: TPS54202DDCR, easyeda2kicad:SOT-23-6_L2.9-W1.6-P0.95-LS2.8-BL, symbol da:TPS54202DDCR
- added U22: W25N01GVZEIG_C907680, easyeda2kicad:WSON-8_L8.0-W6.10-P1.27-BL-EP, symbol da:W25N01GVZEIG_C907680
- R1: value 10k -> 27K
Connections:
- net +3.3V: now also R115.1, R42.1, U19.5 (EN), U22.8 (VCC); no longer R1.1
- net BIOS_SPI_CLK: now also U22.6 (CLK)
- net BIOS_SPI_CS: now also U22.1 (~{CS})
- net BIOS_SPI_IO0: now also U22.5 (DI(DQ0))
- net BIOS_SPI_IO1: now also U22.2 (DO(DQ1))
- net BIOS_SPI_IO2: now also R43.1, U22.3 (WP#(DQ2))
- net BIOS_SPI_IO3: now also R42.2, U22.7 (HOLD#(DQ3))
- net FAN1_PWM: now also R33.1
- net FAN1_TAC: now also R32.1
- net FAN2_PWM: now also R39.1
- net FAN2_TAC: now also R1.1
- net GND: now also B1.1, C92.2, CN5.1, CN6.1, R114.2, R41.2, R43.2, U19.1 (GND), U22.4 (VSS), U22.9 (EP)
- net PWR_LED_SW/RST_SW: now reaches A1.3 (~{RSTBTN})
- net at A1.115 (VBAT): now also B1.2
- net at R1.2: now also CN6.3; no longer A1.1 (~{PWRBTN})
- net BIOS_SEL#: no longer names the net of A1.133 (~{BIOS_SEL})
- net BIOS_SEL#: now also R114.1, SW6.1
- net HDA_BCLK renamed ALC269Q/HDA_BCLK
- net HDA_RST renamed ALC269Q/HDA_RST
- net HDA_SDIN renamed ALC269Q/HDA_SDIN
- net HDA_SDOUT renamed ALC269Q/HDA_SDOUT
- net HDA_SYNC renamed ALC269Q/HDA_SYNC
- net S0_PWR_IND renamed PWR_LED_SW/S0_PWR_IND
- net S3_PWR_IND renamed PWR_LED_SW/S3_PWR_IND
- net USB2_P4+ renamed ESP32/ESP32_D+
- net USB2_P4- renamed ESP32/ESP32_D-
- net USB2_P7+ renamed USB_2_PORTS/USB2_0+
- net USB2_P7- renamed USB_2_PORTS/USB2_0-
- net USB2_P8+ renamed USB_2_PORTS/USB2_1+
- net USB2_P8- renamed USB_2_PORTS/USB2_1-
- new net: L3.2, U19.2 (SW)
- new net: C93.2, R40.2, R41.1, U19.4 (FB)
- new net: C94.1, U19.6 (BOOT)
- new net: CN6.4, R39.2
- new net: R115.2, SW6.2
- new net: CN5.3, R32.2
- new net: CN5.4, R33.2
- new net +12V: C93.1, C94.2, CN6.2, L3.1, R40.1
- new net +5V: CN5.2
- new net PD_VBUS_GATE: C92.1, U19.3 (VIN)
- new net PWR_LED_SW/PWR_SW: A1.1 (~{PWRBTN})
- no-connect marks 37 -> 38
Other:
- added sheet ALC269Q (ALC269Q.kicad_sch)
- added sheet ESP32 (ESP32.kicad_sch)
- added sheet PWR_LED_SW (PWR_LED.kicad_sch)
- added sheet USB_2_PORTS (USB_2_PORTS.kicad_sch)
- note added: "3.3V-> integrated bios gnd -> carrier bios"
- note added: "I2C2 and SML1 used for USB PD Alt Mode Controller (DisplayPort alt mode)"
- note added: "No mipi csi camera connector on board"
- note added: "P1: HUB0 P2: HUB1 P3: PCIE_WIFI P4: ESP32 P7: USB2_0 P8: USB2_1"
- note added: "PCIE reference clock (100Mhz)"
- note added: "USB_OC Connected to USB2"
- note removed: "P1: HUB0 P2: HUB1 P3: PCIE_WIFI"
- note removed: "to read more on usb oc"

Commit message: .
Parts:
- added CN8, CN9: SMTWE2055MTJ, easyeda2kicad:SMD_BD4.4-L4.4-D2.8_H5.5, symbol da:SMTWE2055MTJ
Connections:
- net GND: now also CN8.1, CN9.1

Commit message: .
Connections:
- no-connect marks 38 -> 50
Changed lines of the file:
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@@
+	)
+	(no_connect
+		(at 176.53 205.74)
+	)
+	(no_connect
+		(at 176.53 208.28)
 	)
 	(no_connect
@@
 	(no_connect
 		(at 176.53 130.81)
+	)
+	(no_connect
+		(at 176.53 157.48)
 	)
 	(no_connect
@@
 	)
 	(no_connect
+		(at 176.53 198.12)
+	)
+	(no_connect
 		(at 176.53 38.1)
 	)
@@
 	)
 	(no_connect
+		(at 176.53 165.1)
+	)
+	(no_connect
 		(at 176.53 287.02)
 	)
 	(no_connect
+		(at 176.53 167.64)
+	)
+	(no_connect
 		(at 176.53 187.96)
+	)
+	(no_connect
+		(at 176.53 200.66)
+	)
+	(no_connect
+		(at 176.53 203.2)
 	)
 	(no_connect
@@
 	(no_connect
 		(at 176.53 248.92)
+	)
+	(no_connect
+		(at 176.53 154.94)
 	)
 	(no_connect
@@
 	)
 	(no_connect
+		(at 176.53 210.82)
+	)
+	(no_connect
+		(at 176.53 162.56)
+	)
+	(no_connect
 		(at 176.53 238.76)
 	)
@@
 	)
 	(no_connect
+		(at 176.53 160.02)
+	)
+	(no_connect

Commit message: .
Parts:
- removed B1: BS-02-A1AJ010, easyeda2kicad:BAT-TH_BS-02-A1AJ010, symbol da:BS-02-A1AJ010
- added BT1: BS-06-B4AK001, easyeda2kicad:BAT-SMD_BS-06-B4AA012, symbol da:BS-06-B4AK001
Connections:
- net VBUS is gone; now on net PD_VBUS_GATE: A1.250 (VIN), A1.251 (VIN), A1.252 (VIN), A1.253 (VIN), A1.254 (VIN), A1.255 (VIN), A1.256 (VIN), A1.257 (VIN), A1.258 (VIN), A1.259 (VIN), A1.260 (VIN)
- net GND: now also BT1.2
- net at A1.115 (VBAT): now also BT1.1
Changed lines of the file:
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@@
-	)
-	(symbol
-		(lib_id "da:BS-02-A1AJ010")
-		(at 148.59 25.4 180)
-		(unit 1)
-		(exclude_from_sim no)
-		(in_bom yes)
-		(on_board yes)
-		(dnp no)
-		(fields_autoplaced yes)
-		(property "Reference" "B1"
-			(at 148.59 17.78 0)
-			(effects
-				(font
-					(size 1.27 1.27)
-				)
-			)
-		)
-		(property "Value" "BS-02-A1AJ010"
-			(at 148.59 20.32 0)
-			(effects
-				(font
-					(size 1.27 1.27)
-				)
-			)
-		)
-		(property "Footprint" "easyeda2kicad:BAT-TH_BS-02-A1AJ010"
-			(at 148.59 17.78 0)
-			(effects
-				(font
-					(size 1.27 1.27)
-				)
-				(hide yes)
-			)
-		)
-		(property "Datasheet" ""
-			(at 148.59 25.4 0)
-			(effects
-				(font
-					(size 1.27 1.27)
-				)
-				(hide yes)
-			)
-		)
-		(property "Description" ""
-			(at 148.59 25.4 0)
-			(effects
-				(font
-					(size 1.27 1.27)
-				)
-				(hide yes)
-			)
-		)
-		(property "LCSC Part" "C5239862"
-			(at 148.59 15.24 0)
-			(effects
-				(font
-					(size 1.27 1.27)
-				)
-				(hide yes)
-			)
-		)
-		(pin "1"
-		)
-		(pin "2"
-		)
-		(instances
-			(project ""
-				(path "/ffe475c5-d6e9-41b5-8ca1-322659dd88d8"
-					(reference "B1")
-					(unit 1)
-				)
-			)
-		)
 	)
 	(symbol
@@
 		(on_board yes)
 		(dnp no)
-		(fields_autoplaced yes)
 		(property "Reference" "#PWR04"
 			(at 134.62 34.29 0)
@@
 			)
 		)
-		(property "Value" "VBUS"
-			(at 134.62 25.4 0)
+		(property "Value" "PD_VBUS_GATE"
+			(at 131.826 25.146 0)
 			(effects
 				(font
@@
 					(unit 1)
 				)
+			)
+		)
+	)
+	(symbol
+		(lib_id "da:BS-06-B4AK001")
+		(at 148.59 25.4 0)
+		(unit 1)
+		(exclude_from_sim no)
+		(in_bom yes)
+		(on_board yes)
+		(dnp no)
+		(fields_autoplaced yes)
+		(property "Reference" "BT1"
+			(at 148.59 17.78 0)
+			(effects
+				(font
+					(size 1.27 1.27)
+				)
+			)
+		)
+		(property "Value" "BS-06-B4AK001"
+			(at 148.59 20.32 0)
+			(effects
+				(font
+					(size 1.27 1.27)
+				)
+			)
+		)
+		(property "Footprint" "easyeda2kicad:BAT-SMD_BS-06-B4AA012"
+			(at 148.59 33.02 0)
+			(effects
+				(font
+					(size 1.27 1.27)
+				)
+				(hide yes)
+			)
+		)
+		(property "Datasheet" ""
+			(at 148.59 25.4 0)
+			(effects
+				(font
+					(size 1.27 1.27)
+				)
+				(hide yes)
+			)
+		)
+		(property "Description" ""
+			(at 148.59 25.4 0)
+			(effects
+				(font
+					(size 1.27 1.27)
+				)
+				(hide yes)
+			)
+		)
+		(property "LCSC Part" "C964760"
+			(at 148.59 35.56 0)
+			(effects
+				(font
+					(size 1.27 1.27)
+				)
+				(hide yes)
+			)
+		)
+		(pin "2"
+		)
+		(pin "1"
+		)
+		(instances
+			(project ""
+				(path "/ffe475c5-d6e9-41b5-8ca1-322659dd88d8"
+					(reference "BT1")
+					(unit 1)
+				)

Commit message: .
Parts:
- removed C92: 1uF, Capacitor_SMD:C_0603_1608Metric, symbol Device:C
- removed C93: 47pF, Capacitor_SMD:C_0402_1005Metric, symbol Device:C
- removed C94: 100nF, Capacitor_SMD:C_0402_1005Metric, symbol Device:C
- removed CN6: 47053-1000, easyeda2kicad:CONN-TH_47053-1000, symbol da:47053-1000
- removed L3: 8.2uH, Inductor_SMD:L_Changjiang_FXL0420, symbol Device:L
- removed R1: 27K, Resistor_SMD:R_0402_1005Metric, symbol Device:R
- removed R39: 100R, Resistor_SMD:R_0402_1005Metric, symbol Device:R
- removed R40: 100K, Resistor_SMD:R_0402_1005Metric, symbol Device:R
- removed R41: 5.2K, Resistor_SMD:R_0402_1005Metric, symbol Device:R
- removed U19: TPS54202DDCR, easyeda2kicad:SOT-23-6_L2.9-W1.6-P0.95-LS2.8-BL, symbol da:TPS54202DDCR

Commit message: .
Connections:
- net +3.3V: now also R43.2
- net GND: no longer R43.2
Changed lines of the file:
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@@
 	)
 	(junction
-		(at 238.76 218.44)
-		(diameter 0)
-		(color 0 0 0 0)
-	)
-	(junction
 		(at 293.37 200.66)
 		(diameter 0)
@@
 	(wire
 		(pts
+			(xy 231.14 219.71) (xy 223.52 219.71)
+		)
+		(stroke
+			(width 0)
+			(type default)
+		)
+	)
+	(wire
+		(pts
 			(xy 76.2 281.94) (xy 95.25 281.94)
 		)
@@
 	(wire
 		(pts
-			(xy 231.14 218.44) (xy 238.76 218.44)
-		)
-		(stroke
-			(width 0)
-			(type default)
-		)
-	)
-	(wire
-		(pts
 			(xy 91.44 111.76) (xy 95.25 111.76)
 		)
@@
 	(wire
 		(pts
+			(xy 231.14 218.44) (xy 231.14 219.71)
+		)
+		(stroke
+			(width 0)
+			(type default)
+		)
+	)
+	(wire
+		(pts
 			(xy 91.44 73.66) (xy 95.25 73.66)
 		)
@@
 					(unit 1)
 				)
+			)
+		)
+	)
+	(symbol
+		(lib_id "power:+3.3V")
+		(at 223.52 219.71 0)
+		(unit 1)
+		(exclude_from_sim no)
+		(in_bom yes)
+		(on_board yes)
+		(dnp no)
+		(fields_autoplaced yes)
+		(property "Reference" "#PWR0527"
+			(at 223.52 223.52 0)
+			(effects
+				(font
+					(size 1.27 1.27)
+				)
+				(hide yes)
+			)
+		)
+		(property "Value" "+3.3V"
+			(at 223.52 214.63 0)
+			(effects
+				(font
+					(size 1.27 1.27)
+				)
+			)
+		)
+		(property "Footprint" ""
+			(at 223.52 219.71 0)
+			(effects
+				(font
+					(size 1.27 1.27)
+				)
+				(hide yes)
+			)
+		)
+		(property "Datasheet" ""
+			(at 223.52 219.71 0)
+			(effects
+				(font
+					(size 1.27 1.27)
+				)
+				(hide yes)
+			)
+		)
+		(property "Description" "Power symbol creates a global label with name \"+3.3V\""
+			(at 223.52 219.71 0)
+			(effects
+				(font
+					(size 1.27 1.27)
+				)
+				(hide yes)
+			)
+		)
+		(pin "1"
+		)
+		(instances
+			(project "MiniLatte"
+				(path "/ffe475c5-d6e9-41b5-8ca1-322659dd88d8"
+					(reference "#PWR0527")
+					(unit 1)
+				)
