File: MiniLatte.kicad_sch (KiCad schematic)
At the start: 13 parts, among them CN5 WAFER-PH2.0-4PZZ, CN8 SMTWE2055MTJ, CN9 SMTWE2055MTJ, SW6 DSHP01TSGER, U22 W25N01GVZEIG_C907680

Commit message: .
Connections:
- net PD_VBUS_GATE renamed VBUS_MU
Changed lines of the file:
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@@
 			)
 		)
-		(property "Value" "PD_VBUS_GATE"
+		(property "Value" "VBUS_MU"
 			(at 131.826 25.146 0)
 			(effects

Commit message: .
Parts:
- removed CN5: WAFER-PH2.0-4PZZ, easyeda2kicad:CONN-TH_4P-P2.00_FWF20001-S04S22W5B, symbol da:WAFER-PH2.0-4PZZ
- added CN6: ZX-HY2.0-4PLT, easyeda2kicad:CONN-SMD_4P-P2.00_HY2.0-4P, symbol da:ZX-HY2.0-4PLT
- added H1, H2, H3, H4: MountingHole_Pad, MountingHole:MountingHole_3.2mm_M3_DIN965_Pad_TopOnly, symbol Mechanical:MountingHole_Pad
Connections:
- net +5V: now also CN6.2
- net GND: now also CN6.1, CN6.5, CN6.6, H1.1, H2.1, H3.1, H4.1
- net at R32.2: now also CN6.3
- net at R33.2: now also CN6.4
Other:
- moved on the sheet: R32, R33

Commit message: .
Parts:
- removed CN6: ZX-HY2.0-4PLT, easyeda2kicad:CONN-SMD_4P-P2.00_HY2.0-4P, symbol da:ZX-HY2.0-4PLT
- added CN5: WAFER-PH2.0-4PLB, easyeda2kicad:CONN-SMD_4P-P2.00_WAFER-200L-4A, symbol da:WAFER-PH2.0-4PLB
Connections:
- net +5V: now also CN5.2
- net GND: now also CN5.1, CN5.5, CN5.6
- net at R32.2: now also CN5.3
- net at R33.2: now also CN5.4
Changed lines of the file:
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@@
-	)
-	(symbol
-		(lib_id "da:ZX-HY2.0-4PLT")
-		(at 283.21 96.52 0)
-		(unit 1)
-		(exclude_from_sim no)
-		(in_bom yes)
-		(on_board yes)
-		(dnp no)
-		(fields_autoplaced yes)
-		(property "Reference" "CN6"
-			(at 288.29 95.2499 0)
-			(effects
-				(font
-					(size 1.27 1.27)
-				)
-				(justify left)
-			)
-		)
-		(property "Value" "ZX-HY2.0-4PLT"
-			(at 288.29 97.7899 0)
-			(effects
-				(font
-					(size 1.27 1.27)
-				)
-				(justify left)
-			)
-		)
-		(property "Footprint" "easyeda2kicad:CONN-SMD_4P-P2.00_HY2.0-4P"
-			(at 283.21 113.03 0)
-			(effects
-				(font
-					(size 1.27 1.27)
-				)
-				(hide yes)
-			)
-		)
-		(property "Datasheet" ""
-			(at 283.21 96.52 0)
-			(effects
-				(font
-					(size 1.27 1.27)
-				)
-				(hide yes)
-			)
-		)
-		(property "Description" ""
-			(at 283.21 96.52 0)
-			(effects
-				(font
-					(size 1.27 1.27)
-				)
-				(hide yes)
-			)
-		)
-		(property "LCSC Part" "C7429562"
-			(at 283.21 115.57 0)
-			(effects
-				(font
-					(size 1.27 1.27)
-				)
-				(hide yes)
-			)
-		)
-		(pin "4"
-		)
-		(pin "3"
-		)
-		(pin "6"
-		)
-		(pin "1"
-		)
-		(pin "5"
-		)
-		(pin "2"
-		)
-		(instances
-			(project ""
-				(path "/ffe475c5-d6e9-41b5-8ca1-322659dd88d8"
-					(reference "CN6")
-					(unit 1)
-				)
-			)
-		)
 	)
 	(symbol
@@
 					(unit 1)
 				)
+			)
+		)
+	)
+	(symbol
+		(lib_id "da:WAFER-PH2.0-4PLB")
+		(at 283.21 96.52 0)
+		(unit 1)
+		(exclude_from_sim no)
+		(in_bom yes)
+		(on_board yes)
+		(dnp no)
+		(fields_autoplaced yes)
+		(property "Reference" "CN5"
+			(at 289.56 95.2499 0)
+			(effects
+				(font
+					(size 1.27 1.27)
+				)
+				(justify left)
+			)
+		)
+		(property "Value" "WAFER-PH2.0-4PLB"
+			(at 289.56 97.7899 0)
+			(effects
+				(font
+					(size 1.27 1.27)
+				)
+				(justify left)
+			)
+		)
+		(property "Footprint" "easyeda2kicad:CONN-SMD_4P-P2.00_WAFER-200L-4A"
+			(at 283.21 113.03 0)
+			(effects
+				(font
+					(size 1.27 1.27)
+				)
+				(hide yes)
+			)
+		)
+		(property "Datasheet" ""
+			(at 283.21 96.52 0)
+			(effects
+				(font
+					(size 1.27 1.27)
+				)
+				(hide yes)
+			)
+		)
+		(property "Description" ""
+			(at 283.21 96.52 0)
+			(effects
+				(font
+					(size 1.27 1.27)
+				)
+				(hide yes)
+			)
+		)
+		(property "LCSC Part" "C3029433"
+			(at 283.21 115.57 0)
+			(effects
+				(font
+					(size 1.27 1.27)
+				)
+				(hide yes)
+			)
+		)
+		(pin "4"
+		)
+		(pin "2"
+		)
+		(pin "6"
+		)
+		(pin "1"
+		)
+		(pin "5"
+		)
+		(pin "3"
+		)
+		(instances
+			(project ""
+				(path "/ffe475c5-d6e9-41b5-8ca1-322659dd88d8"
+					(reference "CN5")
+					(unit 1)
+				)

Commit message: .
Parts:
- removed U22: W25N01GVZEIG_C907680, easyeda2kicad:WSON-8_L8.0-W6.10-P1.27-BL-EP, symbol da:W25N01GVZEIG_C907680
- added D20: 1N5819WS S4_C2939001, easyeda2kicad:SOD-323_L1.7-W1.3-LS2.6-RD-1, symbol da:1N5819WSS4_C2939001
- added Q14: 2N7002-SOT23, easyeda2kicad:SOT-23_L2.9-W1.3-P1.90-LS2.4-BR, symbol da:2N7002-SOT23
- added R159, R160: 10k, Resistor_SMD:R_0402_1005Metric, symbol Device:R
- added U24: W25Q128JVEIQ, easyeda2kicad:WSON-8_L6.0-W8.0-P1.27-BL-EP, symbol da:W25Q128JVEIQ
Connections:
- net +3.3V: now also U24.8 (VCC)
- net +5V: now also CN5.3, D20.1 (K), R160.1; no longer CN5.2
- net BIOS_SPI_CLK: now also U24.6 (CLK)
- net BIOS_SPI_CS: now also U24.1 (/CS)
- net BIOS_SPI_IO0: now also U24.5 (DI(IO0))
- net BIOS_SPI_IO1: now also U24.2 (DO(IO1))
- net BIOS_SPI_IO2: now also U24.3 (/WP(IO2))
- net BIOS_SPI_IO3: now also U24.7 (/HOLDor/RESET(IO3))
- net GND: now also Q14.2 (S), R159.1, U24.4 (GND), U24.9 (EP); no longer CN5.1
- net at R32.2: now also CN5.2, D20.2 (A), R160.2; no longer CN5.3
- net at CN5.4: now also Q14.3 (D); no longer R33.2
- net PWR_LED_SW/S0_PWR_IND renamed S0_PWR
- new net: CN5.1, R33.2
- new net S0_PWR_IND: Q14.1 (G), R159.2
Other:
- moved on the sheet: R32, R33, R42, R43
