File: HUB_0_PORTS.kicad_sch (KiCad schematic)
At the start: 15 parts, among them U3 VL162

Commit message: .
Parts:
- added C85, C86, C87: 220uF, Capacitor_SMD:C_Elec_6.3x7.7, symbol Device:C
- added D11, D12, D13, D14: RCLAMP0524P-N, easyeda2kicad:DFN-10L_L2.5-W1.0-P0.50-BL, symbol da:RCLAMP0524P-N
- added R27, R28: ?k, Resistor_SMD:R_0402_1005Metric, symbol Device:R
- added U8: TPS2560DRCR, easyeda2kicad:VSON-10_L3.0-W3.0-P0.50-BL-EP_TPS62410DRCR, symbol da:TPS2560DRCR
- added U9: TPS2553DRVR-1, easyeda2kicad:WSON-6_L2.0-W2.0-P0.65-BL-EP, symbol da:TPS2553DRVR-1
Connections:
- net +5V: now also U8.2 (IN), U8.3 (IN), U9.6 (IN)
- net +5V_DFP2: now also C87.1
- net +5V_DFP3: now also C85.1
- net +5V_DFP4: now also C86.1
- net DFP2_TX_1+: no longer USB1.A2 (SSTXP1)
- net DFP2_TX_1-: no longer USB1.A3 (SSTXn1)
- net DFP2_TX_2+: no longer USB1.B2 (SSTXp2)
- net DFP2_TX_2-: no longer USB1.B3 (SSTXn2)
- net DFP3_RX+: now also D13.2, D13.9
- net DFP3_RX-: now also D13.1, D13.10
- net DFP4_RX+: now also D14.2, D14.9
- net DFP4_RX-: now also D14.1, D14.10
- net GND: now also C85.2, C86.2, C87.2, D11.3, D11.8, D12.3, D12.8, D13.3, D13.8, D14.3, D14.8, R27.1, R28.1, U8.1 (GND), U8.11 (EPAD), U9.5 (GND), U9.7 (EP)
- net CC1_DFP2 renamed H0_CC1_DFP2
- net CC2_DFP2 renamed H0_CC2_DFP2
- net DFP2_RX_1+ renamed DFP2_H0_RX_1+
- net DFP2_H0_RX_1+: now also D11.1, D11.10
- net DFP2_RX_1- renamed DFP2_H0_RX_1-
- net DFP2_H0_RX_1-: now also D11.2, D11.9
- net DFP2_RX_2+ renamed DFP2_H0_RX_2+
- net DFP2_H0_RX_2+: now also D12.5, D12.6
- net DFP2_RX_2- renamed DFP2_H0_RX_2-
- net DFP2_H0_RX_2-: now also D12.4, D12.7
- net DFP3TXC+ renamed H0_DFP3TXC+
- net H0_DFP3TXC+: now also D13.5, D13.6
- net DFP3TXC- renamed H0_DFP3TXC-
- net H0_DFP3TXC-: now also D13.4, D13.7
- net DFP4TXC+ renamed H0_DFP4TXC+
- net H0_DFP4TXC+: now also D14.5, D14.6
- net DFP4TXC- renamed H0_DFP4TXC-
- net H0_DFP4TXC-: now also D14.4, D14.7
- new net: R28.2, U9.2 (ILIM)
- new net: R27.2, U8.7 (ILIM)
- new net +5V_H0_DFP1: U8.9 (OUT1)
- new net +5V_H0_DFP2: U8.8 (OUT2)
- new net +5V_H0_DFP3: U9.1 (OUT)
- new net DFP2_H0_TX_1+: D12.1, D12.10, USB1.A2 (SSTXP1)
- new net DFP2_H0_TX_1-: D12.2, D12.9, USB1.A3 (SSTXn1)
- new net DFP2_H0_TX_2+: D11.5, D11.6, USB1.B2 (SSTXp2)
- new net DFP2_H0_TX_2-: D11.4, D11.7, USB1.B3 (SSTXn2)
- new net H0_USBOC1: U8.10 (~{FAULT1})
- new net H0_USBOC2: U8.6 (~{FAULT2})
- new net H0_USBOC3: U9.3 (~{FAULT})
- new net H0_USBPE1: U8.4 (EN1)
- new net H0_USBPE2: U8.5 (EN2)
- new net H0_USBPE3: U9.4 (EN)
Other:
- moved on the sheet: C23, C24, R11, USB1, USB2

Commit message: .
Connections:
- net +5V_DFP3 is gone; now on net +5V_H0_DFP3: C85.1, USB3.1 (VBUS)
- net +5V_DFP2: no longer C87.1, USB1.B4 (VBUS), USB1.B9 (VBUS)
- net +5V_H0_DFP2: now also C87.1, USB1.B4 (VBUS), USB1.B9 (VBUS)
- net +5V_DFP4 renamed +5V_H0_DFP4
- net DFP4_D+ renamed DFP1_D+
- net DFP4_D- renamed DFP1_D-
- net DFP4_RX+ renamed DFP1_RX+
- net DFP4_RX- renamed DFP1_RX-
- net DFP4_TX+ renamed DFP1_TX+
- net DFP4_TX- renamed DFP1_TX-
- net H0_DFP4TXC+ renamed H0_DFP1TXC+
- net H0_DFP4TXC- renamed H0_DFP1TXC-
Other:
- moved on the sheet: C87
Changed lines of the file:
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@@
 	(wire
 		(pts
+			(xy 87.63 134.62) (xy 87.63 125.73)
+		)
+		(stroke
+			(width 0)
+			(type default)
+		)
+	)
+	(wire
+		(pts
 			(xy 74.93 27.94) (xy 74.93 29.21)
 		)
@@
 		)
 	)
-	(label "H0_DFP4TXC+"
+	(label "H0_DFP1TXC+"
 		(at 127 118.11 0)
 		(effects
@@
 		)
 	)
-	(label "H0_DFP4TXC-"
+	(label "H0_DFP1TXC-"
 		(at 127 113.03 0)
 		(effects
@@
 		)
 	)
-	(label "H0_DFP4TXC+"
+	(label "H0_DFP1TXC+"
 		(at 231.14 59.69 0)
 		(effects
@@
 		)
 	)
-	(label "H0_DFP4TXC-"
+	(label "H0_DFP1TXC-"
 		(at 185.42 113.03 180)
 		(effects
@@
 		)
 	)
-	(label "H0_DFP4TXC-"
+	(label "H0_DFP1TXC-"
 		(at 231.14 57.15 0)
 		(effects
@@
 		)
 	)
-	(label "H0_DFP4TXC+"
+	(label "H0_DFP1TXC+"
 		(at 185.42 118.11 180)
 		(effects
@@
 		)
 	)
-	(hierarchical_label "DFP4_TX-"
+	(hierarchical_label "DFP1_TX-"
 		(shape input)
 		(at 222.25 57.15 180)
@@
 		)
 	)
-	(hierarchical_label "DFP4_D-"
+	(hierarchical_label "DFP1_D-"
 		(shape input)
 		(at 245.11 41.91 180)
@@
 		)
 	)
-	(hierarchical_label "DFP4_TX+"
+	(hierarchical_label "DFP1_TX+"
 		(shape input)
 		(at 222.25 59.69 180)
@@
 		)
 	)
-	(hierarchical_label "DFP4_RX+"
+	(hierarchical_label "DFP1_RX+"
 		(shape input)
 		(at 168.91 107.95 0)
@@
 		)
 	)
-	(hierarchical_label "DFP4_RX-"
+	(hierarchical_label "DFP1_RX-"
 		(shape input)
 		(at 245.11 49.53 180)
@@
 		)
 	)
-	(hierarchical_label "DFP4_D+"
+	(hierarchical_label "DFP1_D+"
 		(shape input)
 		(at 245.11 44.45 180)
@@
 		)
 	)
-	(hierarchical_label "DFP4_RX+"
+	(hierarchical_label "DFP1_RX+"
 		(shape input)
 		(at 245.11 52.07 180)
@@
 		)
 	)
-	(hierarchical_label "DFP4_RX+"
+	(hierarchical_label "DFP1_RX+"
 		(shape input)
 		(at 143.51 107.95 180)
@@
 		)
 	)
-	(hierarchical_label "DFP4_RX-"
+	(hierarchical_label "DFP1_RX-"
 		(shape input)
 		(at 168.91 102.87 0)
@@
 		)
 	)
-	(hierarchical_label "DFP4_RX-"
+	(hierarchical_label "DFP1_RX-"
 		(shape input)
 		(at 143.51 102.87 180)
@@
 	(symbol
 		(lib_id "Device:C")
-		(at 87.63 129.54 0)
+		(at 87.63 138.43 0)
 		(unit 1)
 		(exclude_from_sim no)
@@
 		(fields_autoplaced yes)
 		(property "Reference" "C87"
-			(at 91.44 128.2699 0)
+			(at 91.44 137.1599 0)
 			(effects
 				(font
@@
 		)
 		(property "Value" "220uF"
-			(at 91.44 130.8099 0)
+			(at 91.44 139.6999 0)
 			(effects
 				(font
@@
 		)
 		(property "Footprint" "Capacitor_SMD:C_Elec_6.3x7.7"
-			(at 88.5952 133.35 0)
+			(at 88.5952 142.24 0)
 			(effects
 				(font
@@
 		)
 		(property "Datasheet" "~"
-			(at 87.63 129.54 0)
+			(at 87.63 138.43 0)
 			(effects
 				(font
@@
 		)
 		(property "Description" "Unpolarized capacitor"
-			(at 87.63 129.54 0)
+			(at 87.63 138.43 0)
 			(effects
 				(font
@@
 			)
 		)
-		(property "Value" "+5V_DFP2"
+		(property "Value" "+5V_H0_DFP2"
 			(at 87.63 104.14 0)
 			(effects
@@
 			)
 		)
-		(property "Value" "+5V_DFP3"
+		(property "Value" "+5V_H0_DFP3"
 			(at 215.9 84.582 0)
 			(effects
@@
 			)
 		)
-		(property "Value" "+5V_DFP4"
+		(property "Value" "+5V_H0_DFP4"
 			(at 213.36 31.242 0)
 			(effects
@@
 	(symbol
 		(lib_id "power:GND")
-		(at 87.63 133.35 0)
+		(at 87.63 142.24 0)
 		(unit 1)
 		(exclude_from_sim no)
@@
 		(fields_autoplaced yes)
 		(property "Reference" "#PWR0452"
-			(at 87.63 139.7 0)
+			(at 87.63 148.59 0)
 			(effects
 				(font
@@
 		)
 		(property "Value" "GND"
-			(at 87.63 138.43 0)
+			(at 87.63 147.32 0)
 			(effects
 				(font
@@
 		)
 		(property "Footprint" ""
-			(at 87.63 133.35 0)
+			(at 87.63 142.24 0)
 			(effects
 				(font
@@
 		)
 		(property "Datasheet" ""
-			(at 87.63 133.35 0)
+			(at 87.63 142.24 0)
 			(effects
 				(font
@@
 		)
 		(property "Description" "Power symbol creates a global label with name \"GND\" , ground"
-			(at 87.63 133.35 0)
+			(at 87.63 142.24 0)
 			(effects
 				(font

Commit message: .
Parts:
- added R117, R118, R119: 100k, Resistor_SMD:R_0402_1005Metric, symbol Device:R
- R27, R28: value ?k -> 35K
Connections:
- net +5V_DFP2 is gone; now on net +5V_H0_DFP3: USB1.A4 (VBUS), USB1.A9 (VBUS)
- net +5V_H0_DFP4 is gone; now on net +5V_H0_DFP1: C86.1, USB2.1 (VBUS)
- net DFP2_TX_1+ is gone; now on net DFP3_H0_TX_1+: C19.1
- net DFP2_TX_1- is gone; now on net DFP3_H0_TX_1-: C20.2
- net +5V: now also R117.1, R118.1, R119.1
- net +5V_H0_DFP2: now also C85.1, USB3.1 (VBUS); no longer C87.1, USB1.B4 (VBUS), USB1.B9 (VBUS)
- net +5V_H0_DFP3: now also C87.1, USB1.B4 (VBUS), USB1.B9 (VBUS); no longer C85.1, USB3.1 (VBUS)
- net DFP2_D+: now also USB3.3 (D+); no longer USB1.A6 (DP1), USB1.B6 (DP2)
- net DFP2_D-: now also USB3.2 (D-); no longer USB1.A7 (DN1), USB1.B7 (DN2)
- net DFP2_RX+: now also D13.2, D13.9, USB3.6 (STDA_SSRX+); no longer U3.18 (RX_P)
- net DFP2_RX-: now also D13.1, D13.10, USB3.5 (STDA_SSRX-); no longer U3.17 (RX_N)
- net DFP2_TX+: now also C26.2; no longer U3.21 (TXP)
- net DFP2_TX-: now also C25.1; no longer U3.20 (TXN)
- net DFP3_D+: now also USB1.A6 (DP1), USB1.B6 (DP2); no longer USB3.3 (D+)
- net DFP3_D-: now also USB1.A7 (DN1), USB1.B7 (DN2); no longer USB3.2 (D-)
- net DFP3_RX+: now also U3.18 (RX_P); no longer D13.2, D13.9, USB3.6 (STDA_SSRX+)
- net DFP3_RX-: now also U3.17 (RX_N); no longer D13.1, D13.10, USB3.5 (STDA_SSRX-)
- net DFP3_TX+: now also U3.21 (TXP); no longer C26.2
- net DFP3_TX-: now also U3.20 (TXN); no longer C25.1
- net H0_USBOC1: now also R118.2
- net H0_USBOC2: now also R119.2
- net H0_USBOC3: now also R117.2
- net DFP2TX1+ renamed DFP3TX1+
- net DFP2TX1- renamed DFP3TX1-
- net DFP2TX2+ renamed DFP3TX2+
- net DFP2TX2- renamed DFP3TX2-
- net DFP2_H0_RX_1+ renamed DFP3_H0_RX_1+
- net DFP2_H0_RX_1- renamed DFP3_H0_RX_1-
- net DFP2_H0_RX_2+ renamed DFP3_H0_RX_2+
- net DFP3_H0_RX_2+: now also D11.5, D11.6; no longer D12.5, D12.6
- net DFP2_H0_RX_2- renamed DFP3_H0_RX_2-
- net DFP3_H0_RX_2-: now also D11.4, D11.7; no longer D12.4, D12.7
- net DFP2_H0_TX_1+ renamed DFP3_H0_TX_1+
- net DFP2_H0_TX_1- renamed DFP3_H0_TX_1-
- removed net DFP2_H0_TX_2+: D11.5, D11.6, USB1.B2 (SSTXp2)
- removed net DFP2_H0_TX_2-: D11.4, D11.7, USB1.B3 (SSTXn2)
- net DFP2_TX_2+ renamed DFP3_H0_TX_2+
- net DFP3_H0_TX_2+: now also D12.5, D12.6, USB1.B2 (SSTXp2)
- net DFP2_TX_2- renamed DFP3_H0_TX_2-
- net DFP3_H0_TX_2-: now also D12.4, D12.7, USB1.B3 (SSTXn2)
- net H0_CC1_DFP2 renamed H0_CC1_DFP3
- net H0_CC2_DFP2 renamed H0_CC2_DFP3
- net H0_DFP3TXC+ renamed H0_DFP2TXC+
- net H0_DFP3TXC- renamed H0_DFP2TXC-
Other:
- note added: "TO RENAME RCLAMP PORTS TO BE ACCURATE"
- note removed: "TO ADD CAPS ON TX LINES + TO ADD TVS DIODE"
- moved on the sheet: D11, D13, R27, R28

Commit message: .
Parts:
- removed U8: TPS2560DRCR, easyeda2kicad:VSON-10_L3.0-W3.0-P0.50-BL-EP_TPS62410DRCR, symbol da:TPS2560DRCR
- added U10: TPS2561DRCR, easyeda2kicad:VSON-10_L3.0-W3.0-P0.50-TL-EP_TPS62410DRCR, symbol da:TPS2561DRCR
Connections:
- net +5V: now also U10.2 (IN), U10.3 (IN)
- net +5V_H0_DFP1: now also U10.9 (OUT1)
- net +5V_H0_DFP2: now also U10.8 (OUT2)
- net GND: now also U10.1 (GND), U10.11 (EP)
- net H0_USBOC1: now also U10.10 (~{FAULT1})
- net H0_USBOC2: now also U10.6 (~{FAULT2})
- net H0_USBPE1: now also U10.4 (EN1)
- net H0_USBPE2: now also U10.5 (EN2)
- net at R27.2: now also U10.7 (ILIM)
Other:
- moved on the sheet: R118, R119, R27
