File: MU_PWR.kicad_sch (KiCad schematic)
At the start: 15 parts, among them U30 TPS54561DPRR

Commit message: .
Parts:
- added TP10: +17V TestPoint, TestPoint:TestPoint_Pad_D1.5mm, symbol Connector:TestPoint
- C193, C195, C196: value 20uF -> 22uF
Connections:
- net VBUS_MU: now also TP10.1
Changed lines of the file:
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@@
 		(color 0 0 0 0)
 	)
+	(junction
+		(at 201.93 66.04)
+		(diameter 0)
+		(color 0 0 0 0)
+	)
 	(wire
 		(pts
@@
 	(wire
 		(pts
+			(xy 201.93 66.04) (xy 210.82 66.04)
+		)
+		(stroke
+			(width 0)
+			(type default)
+		)
+	)
+	(wire
+		(pts
 			(xy 181.61 66.04) (xy 196.85 66.04)
 		)
@@
 	(wire
 		(pts
-			(xy 196.85 66.04) (xy 210.82 66.04)
+			(xy 196.85 66.04) (xy 201.93 66.04)
 		)
 		(stroke
@@
 			)
 		)
-		(property "Value" "20uF"
+		(property "Value" "22uF"
 			(at 83.82 71.1199 0)
 			(effects
@@
 			)
 		)
-		(property "Value" "20uF"
+		(property "Value" "22uF"
 			(at 200.66 71.1199 0)
 			(effects
@@
 			)
 		)
-		(property "Value" "20uF"
+		(property "Value" "22uF"
 			(at 214.63 71.1199 0)
 			(effects
@@
 					(unit 1)
 				)
+			)
+		)
+	)
+	(symbol
+		(lib_id "Connector:TestPoint")
+		(at 201.93 66.04 0)
+		(unit 1)
+		(exclude_from_sim no)
+		(in_bom yes)
+		(on_board yes)
+		(dnp no)
+		(fields_autoplaced yes)
+		(property "Reference" "TP10"
+			(at 204.47 61.4679 0)
+			(effects
+				(font
+					(size 1.27 1.27)
+				)
+				(justify left)
+			)
+		)
+		(property "Value" "+17V TestPoint"
+			(at 204.47 64.0079 0)
+			(effects
+				(font
+					(size 1.27 1.27)
+				)
+				(justify left)
+			)
+		)
+		(property "Footprint" "TestPoint:TestPoint_Pad_D1.5mm"
+			(at 207.01 66.04 0)
+			(effects
+				(font
+					(size 1.27 1.27)
+				)
+				(hide yes)
+			)
+		)
+		(property "Datasheet" "~"
+			(at 207.01 66.04 0)
+			(effects
+				(font
+					(size 1.27 1.27)
+				)
+				(hide yes)
+			)
+		)
+		(property "Description" "test point"
+			(at 201.93 66.04 0)
+			(effects
+				(font
+					(size 1.27 1.27)
+				)
+				(hide yes)
+			)
+		)
+		(pin "1"
+		)
+		(instances
+			(project "MiniLatte"
+				(path "/ffe475c5-d6e9-41b5-8ca1-322659dd88d8/3f07c54d-c68c-4501-9d1d-0870eca96d91/7bd99a80-fb36-45f7-b59d-1a7a6d3dcaf0"
+					(reference "TP10")
+					(unit 1)
+				)
