File: USB_2_PORTS.kicad_sch (KiCad schematic)
At the start: 5 parts, among them U10 TPS2560DRCR

Commit message: .
Other:
- note added: "tps2561!!!!!!!! needs logic high"
Changed lines of the file:
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@@
 	(generator_version "9.0")
 	(paper "A4")
+	(text "tps2561!!!!!!!! needs logic high "
+		(exclude_from_sim no)
+		(at 184.658 27.94 0)
+		(effects
+			(font
+				(size 1.27 1.27)
+			)
+		)
+	)
 	(junction
 		(at 151.13 41.91)

Commit message: .
Parts:
- removed U10: TPS2560DRCR, easyeda2kicad:VSON-10_L3.0-W3.0-P0.50-BL-EP_TPS62410DRCR, symbol da:TPS2560DRCR
- added U32: TPS2561DRCR, easyeda2kicad:VSON-10_L3.0-W3.0-P0.50-TL-EP_TPS62410DRCR, symbol da:TPS2561DRCR
- R29: value ?k -> 35k
- R30, R31: value 0R -> 100k
Connections:
- net +5V: now also R30.1, R31.1, U32.2 (IN), U32.3 (IN), U32.4 (EN1), U32.5 (EN2)
- net +5V_USB2_0: now also U32.9 (OUT1)
- net +5V_USB2_1: now also U32.8 (OUT2)
- net GND: now also U32.1 (GND), U32.11 (EP); no longer R30.2, R31.2
- net USB_OC#: now also R31.2, U32.6 (~{FAULT2})
- net at R29.2: now also U32.7 (ILIM)
- new net: R30.2, U32.10 (~{FAULT1})
- no-connect marks 1 -> 0
Other:
- note removed: "tps2561!!!!!!!! needs logic high"
- moved on the sheet: R29
