File: USB_HUB_0.kicad_sch (KiCad schematic)
At the start: 30 parts, among them U1 VL822-QFN76, U2 W25Q32JVZPIQ, Y1 25Mhz

Commit message: .
Connections:
- net USBOC2 renamed H0_USBOC2
- net USBOC3 renamed H0_USBOC3
- net USBOC4 renamed H0_USBOC4
- net USBPE2 renamed H0_USBPE2
- net USBPE3 renamed H0_USBPE3
- net USBPE4 renamed H0_USBPE4
Other:
- moved on the sheet: C1, C10, C11, C12, C13, C14, C15, C16, C17, C18, C2, C3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

Commit message: .
Connections:
- net GL3224/DFP1_D+ renamed HUB_0_PORTS/DFP1_D+
- net GL3224/DFP1_D- renamed HUB_0_PORTS/DFP1_D-
- net GL3224/DFP1_RX+ renamed HUB_0_PORTS/DFP1_RX+
- net GL3224/DFP1_RX- renamed HUB_0_PORTS/DFP1_RX-
- net GL3224/DFP1_TX+ renamed HUB_0_PORTS/DFP1_TX+
- net GL3224/DFP1_TX- renamed HUB_0_PORTS/DFP1_TX-
- net HUB_0_PORTS/DFP4_D+ renamed GL3224/DFP4_D+
- net HUB_0_PORTS/DFP4_D- renamed GL3224/DFP4_D-
- net HUB_0_PORTS/DFP4_RX+ renamed GL3224/DFP4_RX+
- net HUB_0_PORTS/DFP4_RX- renamed GL3224/DFP4_RX-
- net HUB_0_PORTS/DFP4_TX+ renamed GL3224/DFP4_TX+
- net HUB_0_PORTS/DFP4_TX- renamed GL3224/DFP4_TX-
Other:
- sheet GL3224 ports: added DFP4_D+, DFP4_D-, DFP4_RX+, DFP4_RX-, DFP4_TX+, DFP4_TX-; removed DFP1_D+, DFP1_D-, DFP1_RX+, DFP1_RX-, DFP1_TX+, DFP1_TX-
- sheet HUB_0_PORTS ports: added DFP1_D+, DFP1_D-, DFP1_RX+, DFP1_RX-, DFP1_TX+, DFP1_TX-; removed DFP4_D+, DFP4_D-, DFP4_RX+, DFP4_RX-, DFP4_TX+, DFP4_TX-
Changed lines of the file:
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@@
 	)
 	(sheet
-		(at 38.1 41.91)
-		(size 12.7 22.86)
+		(at 38.1 115.57)
+		(size 12.7 20.32)
 		(exclude_from_sim no)
 		(in_bom yes)
@@
 		)
 		(property "Sheetname" "GL3224"
-			(at 38.1 41.1984 0)
+			(at 37.592 115.316 0)
 			(effects
 				(font
@@
 		)
 		(property "Sheetfile" "GL3224.kicad_sch"
-			(at 25.654 61.722 0)
+			(at 25.654 135.382 0)
 			(effects
 				(font
@@
 			)
 		)
-		(pin "DFP1_TX+" input
-			(at 50.8 45.72 0)
-			(effects
-				(font
-					(size 1.27 1.27)
-				)
-				(justify right)
-			)
-		)
-		(pin "DFP1_D-" input
-			(at 50.8 63.5 0)
-			(effects
-				(font
-					(size 1.27 1.27)
-				)
-				(justify right)
-			)
-		)
-		(pin "DFP1_TX-" input
-			(at 50.8 48.26 0)
-			(effects
-				(font
-					(size 1.27 1.27)
-				)
-				(justify right)
-			)
-		)
-		(pin "DFP1_RX+" input
-			(at 50.8 53.34 0)
-			(effects
-				(font
-					(size 1.27 1.27)
-				)
-				(justify right)
-			)
-		)
-		(pin "DFP1_D+" input
-			(at 50.8 60.96 0)
-			(effects
-				(font
-					(size 1.27 1.27)
-				)
-				(justify right)
-			)
-		)
-		(pin "DFP1_RX-" input
-			(at 50.8 55.88 0)
+		(pin "DFP4_RX+" input
+			(at 50.8 124.46 0)
+			(effects
+				(font
+					(size 1.27 1.27)
+				)
+				(justify right)
+			)
+		)
+		(pin "DFP4_TX-" input
+			(at 50.8 119.38 0)
+			(effects
+				(font
+					(size 1.27 1.27)
+				)
+				(justify right)
+			)
+		)
+		(pin "DFP4_D+" input
+			(at 50.8 132.08 0)
+			(effects
+				(font
+					(size 1.27 1.27)
+				)
+				(justify right)
+			)
+		)
+		(pin "DFP4_TX+" input
+			(at 50.8 116.84 0)
+			(effects
+				(font
+					(size 1.27 1.27)
+				)
+				(justify right)
+			)
+		)
+		(pin "DFP4_D-" input
+			(at 50.8 134.62 0)
+			(effects
+				(font
+					(size 1.27 1.27)
+				)
+				(justify right)
+			)
+		)
+		(pin "DFP4_RX-" input
+			(at 50.8 127 0)
 			(effects
 				(font
@@
 	)
 	(sheet
-		(at 38.1 67.31)
-		(size 12.7 72.39)
+		(at 38.1 43.18)
+		(size 12.7 69.85)
 		(exclude_from_sim no)
 		(in_bom yes)
@@
 		)
 		(property "Sheetname" "HUB_0_PORTS"
-			(at 37.338 66.802 0)
+			(at 37.338 42.672 0)
 			(effects
 				(font
@@
 		)
 		(property "Sheetfile" "HUB_0_PORTS.kicad_sch"
-			(at 38.1 141.5546 0)
+			(at 6.604 109.22 0)
 			(effects
 				(font
@@
 				)
 				(justify left top)
+				(hide yes)
 			)
 		)
@@
 			)
 		)
-		(pin "DFP4_RX+" input
-			(at 50.8 124.46 0)
-			(effects
-				(font
-					(size 1.27 1.27)
-				)
-				(justify right)
-			)
-		)
-		(pin "DFP4_TX+" input
-			(at 50.8 116.84 0)
-			(effects
-				(font
-					(size 1.27 1.27)
-				)
-				(justify right)
-			)
-		)
-		(pin "DFP4_RX-" input
-			(at 50.8 127 0)
-			(effects
-				(font
-					(size 1.27 1.27)
-				)
-				(justify right)
-			)
-		)
-		(pin "DFP4_TX-" input
-			(at 50.8 119.38 0)
-			(effects
-				(font
-					(size 1.27 1.27)
-				)
-				(justify right)
-			)
-		)
 		(pin "DFP3_D+" input
 			(at 50.8 93.98 0)
@@
 			)
 		)
-		(pin "DFP4_D+" input
-			(at 50.8 132.08 0)
-			(effects
-				(font
-					(size 1.27 1.27)
-				)
-				(justify right)
-			)
-		)
-		(pin "DFP4_D-" input
-			(at 50.8 134.62 0)
-			(effects
-				(font
-					(size 1.27 1.27)
-				)
-				(justify right)
-			)
-		)
 		(pin "DFP2_TX+" input
 			(at 50.8 68.58 0)
@@
 			(effects
 				(font
+					(size 1.27 1.27)
+				)
+				(justify right)
+			)
+		)
+		(pin "DFP1_TX-" input
+			(at 50.8 48.26 0)
+			(effects
+				(font
+					(size 1.27 1.27)
+				)
+				(justify right)
+			)
+		)
+		(pin "DFP1_D-" input
+			(at 50.8 63.5 0)
+			(effects
+				(font
+					(size 1.27 1.27)
+				)
+				(justify right)
+			)
+		)
+		(pin "DFP1_D+" input
+			(at 50.8 60.96 0)
+			(effects
+				(font
+					(size 1.27 1.27)
+				)
+				(justify right)
+			)
+		)
+		(pin "DFP1_RX+" input
+			(at 50.8 53.34 0)
+			(effects
+				(font
+					(size 1.27 1.27)
+				)
+				(justify right)
+			)
+		)
+		(pin "DFP1_TX+" input
+			(at 50.8 45.72 0)
+			(effects
+				(font
+					(size 1.27 1.27)
+				)
+				(justify right)
+			)
+		)
+		(pin "DFP1_RX-" input
+			(at 50.8 55.88 0)
+			(effects
+				(font

Commit message: .
Connections:
- net H0_USBOC4 is gone; now on an unnamed net: U1.40 (USBOC4)
- net at R2.2: no longer U1.1 (USBOC1)
- net H0_USBPE1: now reaches U1.2 (USBPE1)
- net H0_USBPE4: no longer names the net of U1.39 (USBPE4)
- new net H0_USBOC1: U1.1 (USBOC1)
Other:
- moved on the sheet: C12, R2, R3, R8, R9

Commit message: .
Parts:
- added C92, C94: 10uF, Capacitor_SMD:C_0805_2012Metric, symbol Device:C
- added C93: 22pF, Capacitor_SMD:C_0402_1005Metric, symbol Device:C
- added L3: 2.2uH, easyeda2kicad:IND-SMD_L3.5-W3.0, symbol Device:L
- added R1: 200k, Resistor_SMD:R_0402_1005Metric, symbol Device:R
- added R39: 270k, Resistor_SMD:R_0402_1005Metric, symbol Device:R
- added U19: TPS62590DRVT, easyeda2kicad:WSON-6_L2.0-W2.0-P0.65-TL-EP, symbol da:TPS62590DRVT
Connections:
- net +3.3V: now also C94.1, U19.4 (EN), U19.5 (VIN)
- net GND: now also C92.2, C94.2, R39.2, U19.2 (MODE), U19.6 (GND), U19.7 (EP)
- net +1.05V renamed +1.05V_H1
- net +1.05V_H1: now also C92.1, C93.1, L3.1, R1.1
- new net: C93.2, R1.2, R39.1, U19.3 (FB)
- new net: L3.2, U19.1 (SW)
Other:
- note added: "TPS62590 STEPDOWN CONVERTER"
- moved on the sheet: C1, C10, C11, C12, C13, C14, C15, C16, C17, C18, C2, C3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

Commit message: .
Parts:
- added TP7: +1.05V_H1, TestPoint:TestPoint_Pad_D1.5mm, symbol Connector:TestPoint
- C17, C92, C94: value 10uF -> 22uF
Connections:
- net +1.05V_H1: now also TP7.1
Changed lines of the file:
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@@
 	)
 	(junction
+		(at 35.56 172.72)
+		(diameter 0)
+		(color 0 0 0 0)
+	)
+	(junction
 		(at 31.75 187.96)
 		(diameter 0)
@@
 	(wire
 		(pts
-			(xy 31.75 172.72) (xy 41.91 172.72)
+			(xy 31.75 172.72) (xy 35.56 172.72)
 		)
 		(stroke
@@
 	(wire
 		(pts
+			(xy 35.56 172.72) (xy 41.91 172.72)
+		)
+		(stroke
+			(width 0)
+			(type default)
+		)
+	)
+	(wire
+		(pts
 			(xy 50.8 77.47) (xy 101.6 77.47)
 		)
@@
 	)
 	(symbol
+		(lib_id "Connector:TestPoint")
+		(at 35.56 172.72 0)
+		(unit 1)
+		(exclude_from_sim no)
+		(in_bom yes)
+		(on_board yes)
+		(dnp no)
+		(property "Reference" "TP7"
+			(at 38.1 168.1479 0)
+			(effects
+				(font
+					(size 1.27 1.27)
+				)
+				(justify left)
+			)
+		)
+		(property "Value" "+1.05V_H1"
+			(at 36.068 170.434 0)
+			(effects
+				(font
+					(size 1.27 1.27)
+				)
+				(justify left)
+			)
+		)
+		(property "Footprint" "TestPoint:TestPoint_Pad_D1.5mm"
+			(at 40.64 172.72 0)
+			(effects
+				(font
+					(size 1.27 1.27)
+				)
+				(hide yes)
+			)
+		)
+		(property "Datasheet" "~"
+			(at 40.64 172.72 0)
+			(effects
+				(font
+					(size 1.27 1.27)
+				)
+				(hide yes)
+			)
+		)
+		(property "Description" "test point"
+			(at 35.56 172.72 0)
+			(effects
+				(font
+					(size 1.27 1.27)
+				)
+				(hide yes)
+			)
+		)
+		(pin "1"
+		)
+		(instances
+			(project "MiniLatte"
+				(path "/ffe475c5-d6e9-41b5-8ca1-322659dd88d8/9db433ce-ea3f-4d40-ac5c-6665012436f8/5705bc22-e535-41fc-83c9-7f58378ed5fb"
+					(reference "TP7")
+					(unit 1)
+				)
+			)
+		)
+	)
+	(symbol
 		(lib_id "power:GND")
 		(at 213.36 78.74 0)
@@
 			)
 		)
-		(property "Value" "10uF"
+		(property "Value" "22uF"
 			(at 245.11 107.9499 0)
 			(effects
@@
 			)
 		)
-		(property "Value" "10uF"
+		(property "Value" "22uF"
 			(at 24.384 179.07 0)
 			(effects
@@
 			)
 		)
-		(property "Value" "10uF"
+		(property "Value" "22uF"
 			(at 92.456 183.896 0)
 			(effects
