File: USB_HUB_1.kicad_sch (KiCad schematic)
At the start: 30 parts, among them U11 VL822-QFN76, U12 W25Q32JVZPIQ, Y4 25Mhz

Commit message: .
Connections:
- net USBOC2 renamed H1_USBOC2
- net USBOC3 renamed H1_USBOC3
- net USBOC4 renamed H1_USBOC4
- net USBPE2 renamed H1_USBPE2
- net USBPE3 renamed H1_USBPE3
- net USBPE4 renamed H1_USBPE4
Changed lines of the file:
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@@
 		)
 	)
-	(global_label "USBPE3"
+	(global_label "H1_USBPE3"
 		(shape input)
 		(at 104.14 91.44 180)
@@
 		)
 		(property "Intersheetrefs" "${INTERSHEET_REFS}"
-			(at 93.7163 91.44 0)
+			(at 90.2087 91.44 0)
 			(effects
 				(font
@@
 		)
 	)
-	(global_label "USBPE2"
+	(global_label "H1_USBPE2"
 		(shape input)
 		(at 157.48 40.64 0)
@@
 		)
 		(property "Intersheetrefs" "${INTERSHEET_REFS}"
-			(at 167.9037 40.64 0)
+			(at 171.4113 40.64 0)
 			(effects
 				(font
@@
 		)
 	)
-	(global_label "USBOC4"
+	(global_label "H1_USBOC4"
 		(shape input)
 		(at 157.48 132.08 0)
@@
 		)
 		(property "Intersheetrefs" "${INTERSHEET_REFS}"
-			(at 168.0852 132.08 0)
+			(at 171.5928 132.08 0)
 			(effects
 				(font
@@
 		)
 	)
-	(global_label "USBPE4"
+	(global_label "H1_USBPE4"
 		(shape input)
 		(at 157.48 134.62 0)
@@
 		)
 		(property "Intersheetrefs" "${INTERSHEET_REFS}"
-			(at 167.9037 134.62 0)
+			(at 171.4113 134.62 0)
 			(effects
 				(font
@@
 		)
 	)
-	(global_label "USBOC2"
+	(global_label "H1_USBOC2"
 		(shape input)
 		(at 157.48 43.18 0)
@@
 		)
 		(property "Intersheetrefs" "${INTERSHEET_REFS}"
-			(at 168.0852 43.18 0)
+			(at 171.5928 43.18 0)
 			(effects
 				(font
@@
 		)
 	)
-	(global_label "USBOC3"
+	(global_label "H1_USBOC3"
 		(shape input)
 		(at 104.14 88.9 180)
@@
 		)
 		(property "Intersheetrefs" "${INTERSHEET_REFS}"
-			(at 93.5348 88.9 0)
+			(at 90.0272 88.9 0)
 			(effects
 				(font
@@
 		(dnp no)
 		(property "Reference" "R47"
-			(at 174.752 42.926 90)
+			(at 177.546 42.926 90)
 			(effects
 				(font
@@
 		)
 		(property "Value" "10K"
-			(at 170.434 42.672 90)
-			(effects
-				(font
+			(at 173.228 42.672 90)
+			(effects
+				(font

Commit message: .
Parts:
- added R116: 100k, Resistor_SMD:R_0402_1005Metric, symbol Device:R
- R51: value 47k -> 10k
- R52: value 100k -> 20k
Connections:
- net +3.3V: no longer R51.2
- net at R51.1, R52.2: now also R116.1; no longer U11.43 (VBUSDET0)
- new net: R116.2, U11.43 (VBUSDET0)
- new net +5V: R51.2
Other:
- moved on the sheet: R51, R52
Changed lines of the file:
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@@
 	)
 	(junction
-		(at 184.15 137.16)
+		(at 190.5 137.16)
 		(diameter 0)
 		(color 0 0 0 0)
@@
 	(wire
 		(pts
+			(xy 176.53 134.62) (xy 176.53 137.16)
+		)
+		(stroke
+			(width 0)
+			(type default)
+		)
+	)
+	(wire
+		(pts
 			(xy 171.45 139.7) (xy 171.45 129.54)
 		)
@@
 	(wire
 		(pts
-			(xy 173.99 124.46) (xy 173.99 137.16)
+			(xy 176.53 124.46) (xy 176.53 127)
 		)
 		(stroke
@@
 	(wire
 		(pts
-			(xy 157.48 124.46) (xy 173.99 124.46)
+			(xy 157.48 124.46) (xy 176.53 124.46)
 		)
 		(stroke
@@
 	(wire
 		(pts
-			(xy 173.99 137.16) (xy 184.15 137.16)
+			(xy 176.53 137.16) (xy 190.5 137.16)
 		)
 		(stroke
@@
 	(symbol
 		(lib_id "Device:R")
-		(at 184.15 140.97 180)
+		(at 190.5 140.97 180)
 		(unit 1)
 		(exclude_from_sim no)
@@
 		(dnp no)
 		(property "Reference" "R52"
-			(at 179.832 140.97 0)
+			(at 186.182 140.97 0)
 			(effects
 				(font
@@
 			)
 		)
-		(property "Value" "100k"
-			(at 180.086 143.002 0)
+		(property "Value" "20k"
+			(at 186.436 143.002 0)
 			(effects
 				(font
@@
 		)
 		(property "Footprint" "Resistor_SMD:R_0402_1005Metric"
-			(at 185.928 140.97 90)
+			(at 192.278 140.97 90)
 			(effects
 				(font
@@
 		)
 		(property "Datasheet" "~"
-			(at 184.15 140.97 0)
+			(at 190.5 140.97 0)
 			(effects
 				(font
@@
 		)
 		(property "Description" "Resistor"
-			(at 184.15 140.97 0)
+			(at 190.5 140.97 0)
 			(effects
 				(font
@@
 	(symbol
 		(lib_id "Device:R")
+		(at 176.53 130.81 180)
+		(unit 1)
+		(exclude_from_sim no)
+		(in_bom yes)
+		(on_board yes)
+		(dnp no)
+		(property "Reference" "R116"
+			(at 181.102 129.032 0)
+			(effects
+				(font
+					(size 1.27 1.27)
+				)
+			)
+		)
+		(property "Value" "100k"
+			(at 181.356 131.064 0)
+			(effects
+				(font
+					(size 1.27 1.27)
+				)
+			)
+		)
+		(property "Footprint" "Resistor_SMD:R_0402_1005Metric"
+			(at 178.308 130.81 90)
+			(effects
+				(font
+					(size 1.27 1.27)
+				)
+				(hide yes)
+			)
+		)
+		(property "Datasheet" "~"
+			(at 176.53 130.81 0)
+			(effects
+				(font
+					(size 1.27 1.27)
+				)
+				(hide yes)
+			)
+		)
+		(property "Description" "Resistor"
+			(at 176.53 130.81 0)
+			(effects
+				(font
+					(size 1.27 1.27)
+				)
+				(hide yes)
+			)
+		)
+		(pin "1"
+		)
+		(pin "2"
+		)
+		(instances
+			(project "MiniLatte"
+				(path "/ffe475c5-d6e9-41b5-8ca1-322659dd88d8/9db433ce-ea3f-4d40-ac5c-6665012436f8/b1fa3c58-3f32-4cbc-9190-eba41745c3ec"
+					(reference "R116")
+					(unit 1)
+				)
+			)
+		)
+	)
+	(symbol
+		(lib_id "Device:R")
 		(at 171.45 143.51 180)
 		(unit 1)
@@
 	(symbol
 		(lib_id "power:+3.3V")
-		(at 184.15 129.54 0)
+		(at 190.5 129.54 0)
 		(unit 1)
 		(exclude_from_sim no)
@@
 		(fields_autoplaced yes)
 		(property "Reference" "#PWR0270"
-			(at 184.15 133.35 0)
+			(at 190.5 133.35 0)
 			(effects
 				(font
@@
 			)
 		)
-		(property "Value" "+3.3V"
-			(at 184.15 124.46 0)
+		(property "Value" "+5V"
+			(at 190.5 124.46 0)
 			(effects
 				(font
@@
 		)
 		(property "Footprint" ""
-			(at 184.15 129.54 0)
+			(at 190.5 129.54 0)
 			(effects
 				(font
@@
 		)
 		(property "Datasheet" ""
-			(at 184.15 129.54 0)
+			(at 190.5 129.54 0)
 			(effects
 				(font
@@
 		)
 		(property "Description" "Power symbol creates a global label with name \"+3.3V\""
-			(at 184.15 129.54 0)
+			(at 190.5 129.54 0)
 			(effects
 				(font
@@
 	(symbol
 		(lib_id "Device:R")
-		(at 184.15 133.35 180)
+		(at 190.5 133.35 180)
 		(unit 1)
 		(exclude_from_sim no)
@@
 		(dnp no)
 		(property "Reference" "R51"
-			(at 179.832 133.35 0)
+			(at 186.182 133.35 0)
 			(effects
 				(font
@@
 			)
 		)
-		(property "Value" "47k"
-			(at 180.086 135.382 0)
+		(property "Value" "10k"
+			(at 186.436 135.382 0)
 			(effects
 				(font
@@
 		)
 		(property "Footprint" "Resistor_SMD:R_0402_1005Metric"
-			(at 185.928 133.35 90)
+			(at 192.278 133.35 90)
 			(effects
 				(font
@@
 		)
 		(property "Datasheet" "~"
-			(at 184.15 133.35 0)
+			(at 190.5 133.35 0)
 			(effects
 				(font
@@
 		)
 		(property "Description" "Resistor"
-			(at 184.15 133.35 0)
+			(at 190.5 133.35 0)
 			(effects
 				(font
@@
 	(symbol
 		(lib_id "power:GND")
-		(at 184.15 144.78 0)
+		(at 190.5 144.78 0)
 		(unit 1)
 		(exclude_from_sim no)
@@
 		(fields_autoplaced yes)
 		(property "Reference" "#PWR0271"
-			(at 184.15 151.13 0)
+			(at 190.5 151.13 0)
 			(effects
 				(font
@@
 		)
 		(property "Value" "GND"
-			(at 184.15 149.86 0)
+			(at 190.5 149.86 0)
 			(effects
 				(font
@@
 		)
 		(property "Footprint" ""
-			(at 184.15 144.78 0)
+			(at 190.5 144.78 0)
 			(effects
 				(font
@@
 		)
 		(property "Datasheet" ""
-			(at 184.15 144.78 0)
+			(at 190.5 144.78 0)
 			(effects
 				(font
@@
 		)
 		(property "Description" "Power symbol creates a global label with name \"GND\" , ground"
-			(at 184.15 144.78 0)
+			(at 190.5 144.78 0)
 			(effects
 				(font

Commit message: .
Parts:
- removed R45: 10K, Resistor_SMD:R_0402_1005Metric, symbol Device:R
- added C186, C188: 10uF, Capacitor_SMD:C_0805_2012Metric, symbol Device:C
- added C187: 22pF, Capacitor_SMD:C_0402_1005Metric, symbol Device:C
- added L4: 2.2uH, easyeda2kicad:IND-SMD_L3.5-W3.0, symbol Device:L
- added R40: 200k, Resistor_SMD:R_0402_1005Metric, symbol Device:R
- added R41: 270k, Resistor_SMD:R_0402_1005Metric, symbol Device:R
- added U29: TPS62590DRVT, easyeda2kicad:WSON-6_L2.0-W2.0-P0.65-TL-EP, symbol da:TPS62590DRVT
Connections:
- net +3.3V: now also C188.1, U29.4 (EN), U29.5 (VIN)
- net GND: now also C186.2, C188.2, R41.2, U29.2 (MODE), U29.6 (GND), U29.7 (EP)
- net H1_USBOC1: now reaches U11.1 (USBOC1)
- net H1_USBPE1: now reaches U11.2 (USBPE1)
- net +1.05V renamed +1.05V_H2
- net +1.05V_H2: now also C186.1, C187.1, L4.1, R40.1
- new net: C187.2, R40.2, R41.1, U29.3 (FB)
- new net: L4.2, U29.1 (SW)
- no-connect marks 9 -> 8
Other:
- note added: "TPS62590 STEPDOWN CONVERTER"
- moved on the sheet: C102, C103, C104, C105, C106, C107, C108, C109, C110, C111, C112, C113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

Commit message: .
Parts:
- added TP8: +1.05V_H1, TestPoint:TestPoint_Pad_D1.5mm, symbol Connector:TestPoint
- C118, C186, C188: value 10uF -> 22uF
Connections:
- net +1.05V_H2: now also TP8.1
Changed lines of the file:
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@@
 	)
 	(junction
+		(at 38.1 172.72)
+		(diameter 0)
+		(color 0 0 0 0)
+	)
+	(junction
 		(at 205.74 57.15)
 		(diameter 0)
@@
 	(wire
 		(pts
-			(xy 35.56 172.72) (xy 45.72 172.72)
+			(xy 35.56 172.72) (xy 38.1 172.72)
 		)
 		(stroke
@@
 	(wire
 		(pts
+			(xy 38.1 172.72) (xy 45.72 172.72)
+		)
+		(stroke
+			(width 0)
+			(type default)
+		)
+	)
+	(wire
+		(pts
 			(xy 88.9 115.57) (xy 105.41 115.57)
 		)
@@
 			)
 		)
-		(property "Value" "10uF"
+		(property "Value" "22uF"
 			(at 28.194 179.07 0)
 			(effects
@@
 	)
 	(symbol
+		(lib_id "Connector:TestPoint")
+		(at 38.1 172.72 0)
+		(unit 1)
+		(exclude_from_sim no)
+		(in_bom yes)
+		(on_board yes)
+		(dnp no)
+		(property "Reference" "TP8"
+			(at 40.64 168.1479 0)
+			(effects
+				(font
+					(size 1.27 1.27)
+				)
+				(justify left)
+			)
+		)
+		(property "Value" "+1.05V_H1"
+			(at 38.608 170.434 0)
+			(effects
+				(font
+					(size 1.27 1.27)
+				)
+				(justify left)
+			)
+		)
+		(property "Footprint" "TestPoint:TestPoint_Pad_D1.5mm"
+			(at 43.18 172.72 0)
+			(effects
+				(font
+					(size 1.27 1.27)
+				)
+				(hide yes)
+			)
+		)
+		(property "Datasheet" "~"
+			(at 43.18 172.72 0)
+			(effects
+				(font
+					(size 1.27 1.27)
+				)
+				(hide yes)
+			)
+		)
+		(property "Description" "test point"
+			(at 38.1 172.72 0)
+			(effects
+				(font
+					(size 1.27 1.27)
+				)
+				(hide yes)
+			)
+		)
+		(pin "1"
+		)
+		(instances
+			(project "MiniLatte"
+				(path "/ffe475c5-d6e9-41b5-8ca1-322659dd88d8/9db433ce-ea3f-4d40-ac5c-6665012436f8/b1fa3c58-3f32-4cbc-9190-eba41745c3ec"
+					(reference "TP8")
+					(unit 1)
+				)
+			)
+		)
+	)
+	(symbol
 		(lib_id "Device:C")
 		(at 232.41 109.22 180)
@@
 			)
 		)
-		(property "Value" "10uF"
+		(property "Value" "22uF"
 			(at 96.266 183.896 0)
 			(effects
@@
 			)
 		)
-		(property "Value" "10uF"
+		(property "Value" "22uF"
 			(at 248.92 110.4899 0)
 			(effects
