File: GL3224.kicad_sch (KiCad schematic)
At the start: 20 parts, among them U4 GL3224-ONY04, U5 W25Q32JVZPIQ, Y2 25Mhz

Commit message: .
Parts:
- added C81, C82, C83, C84: 100nF, Capacitor_SMD:C_0402_1005Metric, symbol Device:C_Small
Connections:
- net DFP1_RX+: now also C82.2; no longer U4.11 (RXP)
- net DFP1_RX-: now also C81.1; no longer U4.10 (RXN)
- net DFP1_TX+: now also C84.2; no longer U4.8 (TXP)
- net DFP1_TX-: now also C83.1; no longer U4.7 (TXN)
- new net DFP1_DRX+: C82.1, U4.8 (TXP)
- new net DFP1_DRX-: C81.2, U4.7 (TXN)
- new net DFP1_DTX+: C84.1, U4.11 (RXP)
- new net DFP1_DTX-: C83.2, U4.10 (RXN)
Other:
- moved on the sheet: C27, C28, C29, C30, C31, C32, C33, C34, C35, C36, C37, C38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

Commit message: .
Parts:
- renumbered C81 to C29, C82 to C30, C83 to C31, C84 to C32, C29 to C33, C30 to C34, C31 to C35, C32 to C36, C33 to C37, C34 to C38, C37 to C39, C38 to C40, C39 to C81, C40 to C82, C35 to C83, C36 to C84
Connections:
- net DFP1_D+ renamed DFP4_D+
- net DFP1_D- renamed DFP4_D-
- net DFP1_DRX+ renamed DFP4_DRX+
- net DFP1_DRX- renamed DFP4_DRX-
- net DFP1_DTX+ renamed DFP4_DTX+
- net DFP1_DTX- renamed DFP4_DTX-
- net DFP1_RX+ renamed DFP4_RX+
- net DFP1_RX- renamed DFP4_RX-
- net DFP1_TX+ renamed DFP4_TX+
- net DFP1_TX- renamed DFP4_TX-

Commit message: .
Parts:
- C83, C84: value 10uF -> 22uF
Changed lines of the file:
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@@
 			)
 		)
-		(property "Value" "10uF"
+		(property "Value" "22uF"
 			(at 269.24 144.78 90)
 			(effects
@@
 			)
 		)
-		(property "Value" "10uF"
+		(property "Value" "22uF"
 			(at 269.24 160.02 90)
 			(effects

Commit message: .
Connections:
- net +3.3V_GL: now reaches C27.2, U4.6 (AVDD33)
- net +3.3V_GL: now also C35.1, C36.1, C39.1, C82.2, U4.15 (AVDD33), U4.25 (DVDD33), U4.34 (DVDD33), U4.44 (DVDD33)
- net +1.2V_GL: now reaches C81.1, U4.26 (DVDD12)
- net +1.2V_GL: now also C28.1, U4.9 (AVDD12)
Other:
- moved on the sheet: C28, C35, C39
