File: HUB_1_PORTS.kicad_sch (KiCad schematic)
At the start: 15 parts, among them U13 VL162

Commit message: .
Parts:
- removed USB4, USB7: TYPEC-324-BCP24, easyeda2kicad:USB-C-SMD_TYPEC-324-BCP24, symbol da:TYPEC-324-BCP24
- added C166, C174, C175, C176: 100nF, Capacitor_SMD:C_0402_1005Metric, symbol Device:C_Small
- added C88, C89: 220uF, Capacitor_SMD:C_Elec_6.3x7.7, symbol Device:C
- added D15, D16: RCLAMP0524P-N, easyeda2kicad:DFN-10L_L2.5-W1.0-P0.50-BL, symbol da:RCLAMP0524P-N
- added R107: 120k, Resistor_SMD:R_0402_1005Metric, symbol Device:R
- added R108, R109: 10k, Resistor_SMD:R_0402_1005Metric, symbol Device:R
- added R111, R112: ?k, Resistor_SMD:R_0402_1005Metric, symbol Device:R
- added U18: VL162, easyeda2kicad:MQFN-28_L4.5-W3.5-P0.40-BL-EP, symbol da:VL162
- added U20, U21: TPS2560DRCR, easyeda2kicad:VSON-10_L3.0-W3.0-P0.50-BL-EP_TPS62410DRCR, symbol da:TPS2560DRCR
Connections:
- net +5V: now also U18.25 (CE), U18.26 (VCC5V), U18.27 (Vconn_5Vin), U20.2 (IN), U20.3 (IN), U21.2 (IN), U21.3 (IN)
- net +5V_DFP3: now also C89.1
- net +5V_DFP4: now also C88.1
- net DFP3_RX+: now also D15.2, D15.9
- net DFP3_RX-: now also D15.1, D15.10
- net DFP4_RX+: now also D16.2, D16.9
- net DFP4_RX-: now also D16.1, D16.10
- net GND: now also C88.2, C89.2, D15.3, D15.8, D16.3, D16.8, R107.1, R108.2, R109.2, R111.1, R112.1, U18.19 (GND), U18.29 (EP), U20.1 (GND), U20.11 (EPAD), U21.1 (GND), U21.11 (EPAD)
- net CC1_DFP2 renamed H1_CC1_DFP2
- net CC2_DFP2 renamed H1_CC2_DFP2
- net DFP2TX1+ renamed H1_DFP2TX1+
- net DFP2TX1- renamed H1_DFP2TX1-
- net DFP2TX2+ renamed H1_DFP2TX2+
- net DFP2TX2- renamed H1_DFP2TX2-
- net DFP2_RX_1+ renamed H1_DFP2_RX_1+
- net DFP2_RX_1- renamed H1_DFP2_RX_1-
- net DFP2_RX_2+ renamed H1_DFP2_RX_2+
- net DFP2_RX_2- renamed H1_DFP2_RX_2-
- net DFP2_TX_1+ renamed H1_DFP2_TX_1+
- net DFP2_TX_1- renamed H1_DFP2_TX_1-
- net DFP2_TX_2+ renamed H1_DFP2_TX_2+
- net DFP2_TX_2- renamed H1_DFP2_TX_2-
- net DFP3TXC+ renamed H1_DFP3TXC+
- net H1_DFP3TXC+: now also D15.5, D15.6
- net DFP3TXC- renamed H1_DFP3TXC-
- net H1_DFP3TXC-: now also D15.4, D15.7
- net DFP4TXC+ renamed H1_DFP4TXC+
- net H1_DFP4TXC+: now also D16.5, D16.6
- net DFP4TXC- renamed H1_DFP4TXC-
- net H1_DFP4TXC-: now also D16.4, D16.7
- new net: R109.1, U18.23 (CurrentSettingin<1>)
- new net: R112.2, U21.7 (ILIM)
- new net: R111.2, U20.7 (ILIM)
- new net: R108.1, U18.24 (CurrentSettingin<0>)
- new net: R107.2, U18.10 (REXT)
- new net +5V_H1_DFP1: U20.9 (OUT1)
- new net +5V_H1_DFP2: U20.8 (OUT2)
- new net +5V_H1_DFP3: U21.9 (OUT1)
- new net +5V_H1_DFP4: U21.8 (OUT2)
- new net DFP1_RX+: U18.18 (RX_P)
- new net DFP1_RX-: U18.17 (RX_N)
- new net DFP1_TX+: U18.21 (TXP)
- new net DFP1_TX-: U18.20 (TXN)
- new net H1_CC1_DFP1: U18.1 (CC1)
- new net H1_CC2_DFP1: U18.28 (CC2)
- new net H1_DFP1TX1+: C166.2, U18.2 (TX1_P)
- new net H1_DFP1TX1-: C174.1, U18.3 (TX1_N)
- new net H1_DFP1TX2+: C176.1, U18.5 (TX2_P)
- new net H1_DFP1TX2-: C175.2, U18.4 (TX2_N)
- new net H1_DFP1_RX_1+: U18.6 (RX1_P)
- new net H1_DFP1_RX_1-: U18.7 (RX1_N)
- new net H1_DFP1_RX_2+: U18.9 (RX2_P)
- new net H1_DFP1_RX_2-: U18.8 (RX2_N)
- new net H1_DFP1_TX_1+: C166.1
- new net H1_DFP1_TX_1-: C174.2
- new net H1_DFP1_TX_2+: C176.2
- new net H1_DFP1_TX_2-: C175.1
- new net H1_USBOC1: U20.10 (~{FAULT1})
- new net H1_USBOC2: U20.6 (~{FAULT2})
- new net H1_USBOC3: U21.10 (~{FAULT1})
- new net H1_USBOC4: U21.6 (~{FAULT2})
- new net H1_USBPE1: U20.4 (EN1)
- new net H1_USBPE2: U20.5 (EN2)
- new net H1_USBPE3: U21.4 (EN1)
- new net H1_USBPE4: U21.5 (EN2)
- no-connect marks 11 -> 14
Other:
- added sheet TYPE_C_PORTS_1 (TYPE_C_PORTS_1.kicad_sch)
- moved on the sheet: C120, C121, C122, C123, R54, R55, R56

Commit message: .
Parts:
- added D17: RCLAMP0524P-N, easyeda2kicad:DFN-10L_L2.5-W1.0-P0.50-BL, symbol da:RCLAMP0524P-N
Connections:
- net DFP3_D+: now also D15.1, D15.10
- net DFP3_D-: now also D15.2, D15.9
- net DFP3_RX+: now also D16.1, D16.10; no longer D15.2, D15.9
- net DFP3_RX-: now also D16.2, D16.9; no longer D15.1, D15.10
- net DFP4_D+: now also D16.4, D16.7
- net DFP4_D-: now also D16.5, D16.6
- net DFP4_RX+: now also D17.2, D17.9; no longer D16.2, D16.9
- net DFP4_RX-: now also D17.1, D17.10; no longer D16.1, D16.10
- net GND: now also D17.3, D17.8
- net H1_DFP4TXC+: now also D17.5, D17.6; no longer D16.5, D16.6
- net H1_DFP4TXC-: now also D17.4, D17.7; no longer D16.4, D16.7

Commit message: .
Connections:
- net +5V_DFP3 is gone; now on net +5V_H1_DFP2: C89.1, USB9.10 (VBUS2)
- net +5V_DFP4 is gone; now on net +5V_H1_DFP1: C88.1, USB9.1 (VBUS1)
- net DFP1_D+: now also D16.4, D16.7, USB9.3 (D1+)
- net DFP1_D-: now also D16.5, D16.6, USB9.2 (D1-)
- net DFP1_RX+: now also D17.2, D17.9, USB9.6 (StdA_SSRX1+); no longer U18.18 (RX_P)
- net DFP1_RX-: now also D17.1, D17.10, USB9.5 (StdA_SSRX1-); no longer U18.17 (RX_N)
- net DFP1_TX+: now also C125.2; no longer U18.21 (TXP)
- net DFP1_TX-: now also C124.1; no longer U18.20 (TXN)
- net DFP2_D+: now also D15.1, D15.10, USB9.12 (D2+)
- net DFP2_D-: now also D15.2, D15.9, USB9.11 (D2-)
- net DFP2_RX+: now also D16.1, D16.10, USB9.15 (StdA_SSRX2+); no longer U13.18 (RX_P)
- net DFP2_RX-: now also D16.2, D16.9, USB9.14 (StdA_SSRX2-); no longer U13.17 (RX_N)
- net DFP2_TX+: now also C127.2; no longer U13.21 (TXP)
- net DFP2_TX-: now also C126.1; no longer U13.20 (TXN)
- net DFP3_D+: no longer D15.1, D15.10, USB9.12 (D2+)
- net DFP3_D-: no longer D15.2, D15.9, USB9.11 (D2-)
- net DFP3_RX+: now also U13.18 (RX_P); no longer D16.1, D16.10, USB9.15 (StdA_SSRX2+)
- net DFP3_RX-: now also U13.17 (RX_N); no longer D16.2, D16.9, USB9.14 (StdA_SSRX2-)
- net DFP3_TX+: now also U13.21 (TXP); no longer C127.2
- net DFP3_TX-: now also U13.20 (TXN); no longer C126.1
- net DFP4_D+: no longer D16.4, D16.7, USB9.3 (D1+)
- net DFP4_D-: no longer D16.5, D16.6, USB9.2 (D1-)
- net DFP4_RX+: now also U18.18 (RX_P); no longer D17.2, D17.9, USB9.6 (StdA_SSRX1+)
- net DFP4_RX-: now also U18.17 (RX_N); no longer D17.1, D17.10, USB9.5 (StdA_SSRX1-)
- net DFP4_TX+: now also U18.21 (TXP); no longer C125.2
- net DFP4_TX-: now also U18.20 (TXN); no longer C124.1
- net H1_DFP3TXC+ renamed H1_DFP2TXC+
- net H1_DFP3TXC- renamed H1_DFP2TXC-
- net H1_DFP4TXC+ renamed H1_DFP1TXC+
- net H1_DFP4TXC- renamed H1_DFP1TXC-
Other:
- moved on the sheet: D15, D16, D17, R55, R56

Commit message: .
Parts:
- added R120, R121, R122, R123: 100k, Resistor_SMD:R_0402_1005Metric, symbol Device:R
- R111, R112: value ?k -> 35K
Connections:
- net +5V: now also R120.1, R121.1, R122.1, R123.1
- net H1_USBOC1: now also R120.2
- net H1_USBOC2: now also R121.2
- net H1_USBOC3: now also R123.2
- net H1_USBOC4: now also R122.2
- net H1_CC1_DFP1 renamed H1_CC1_DFP4
- net H1_CC1_DFP2 renamed H1_CC1_DFP3
- net H1_CC2_DFP1 renamed H1_CC2_DFP4
- net H1_CC2_DFP2 renamed H1_CC2_DFP3
- net H1_DFP1TX1+ renamed H1_DFP4TX1+
- net H1_DFP1TX1- renamed H1_DFP4TX1-
- net H1_DFP1TX2+ renamed H1_DFP4TX2+
- net H1_DFP1TX2- renamed H1_DFP4TX2-
- net H1_DFP1_RX_1+ renamed H1_DFP4_RX_1+
- net H1_DFP1_RX_1- renamed H1_DFP4_RX_1-
- net H1_DFP1_RX_2+ renamed H1_DFP4_RX_2+
- net H1_DFP1_RX_2- renamed H1_DFP4_RX_2-
- net H1_DFP1_TX_1+ renamed H1_DFP4_TX_1+
- net H1_DFP1_TX_1- renamed H1_DFP4_TX_1-
- net H1_DFP1_TX_2+ renamed H1_DFP4_TX_2+
- net H1_DFP1_TX_2- renamed H1_DFP4_TX_2-
- net H1_DFP2TX1+ renamed H1_DFP3TX1+
- net H1_DFP2TX1- renamed H1_DFP3TX1-
- net H1_DFP2TX2+ renamed H1_DFP3TX2+
- net H1_DFP2TX2- renamed H1_DFP3TX2-
- net H1_DFP2_RX_1+ renamed H1_DFP3_RX_1+
- net H1_DFP2_RX_1- renamed H1_DFP3_RX_1-
- net H1_DFP2_RX_2+ renamed H1_DFP3_RX_2+
- net H1_DFP2_RX_2- renamed H1_DFP3_RX_2-
- net H1_DFP2_TX_1+ renamed H1_DFP3_TX_1+
- net H1_DFP2_TX_1- renamed H1_DFP3_TX_1-
- net H1_DFP2_TX_2+ renamed H1_DFP3_TX_2+
- net H1_DFP2_TX_2- renamed H1_DFP3_TX_2-
Other:
- moved on the sheet: R111, R112

Commit message: .
Parts:
- removed U20, U21: TPS2560DRCR, easyeda2kicad:VSON-10_L3.0-W3.0-P0.50-BL-EP_TPS62410DRCR, symbol da:TPS2560DRCR
- added U31, U8: TPS2561DRCR, easyeda2kicad:VSON-10_L3.0-W3.0-P0.50-TL-EP_TPS62410DRCR, symbol da:TPS2561DRCR
Connections:
- net +5V: now also U31.2 (IN), U31.3 (IN), U8.2 (IN), U8.3 (IN)
- net +5V_H1_DFP1: now also U8.9 (OUT1)
- net +5V_H1_DFP2: now also U8.8 (OUT2)
- net +5V_H1_DFP3: now also U31.9 (OUT1)
- net +5V_H1_DFP4: now also U31.8 (OUT2)
- net GND: now also U31.1 (GND), U31.11 (EP), U8.1 (GND), U8.11 (EP)
- net H1_USBOC1: now also U8.10 (~{FAULT1})
- net H1_USBOC2: now also U8.6 (~{FAULT2})
- net H1_USBOC3: now also U31.10 (~{FAULT1})
- net H1_USBOC4: now also U31.6 (~{FAULT2})
- net H1_USBPE1: now also U8.4 (EN1)
- net H1_USBPE2: now also U8.5 (EN2)
- net H1_USBPE3: now also U31.4 (EN1)
- net H1_USBPE4: now also U31.5 (EN2)
- net at R112.2: now also U31.7 (ILIM)
- net at R111.2: now also U8.7 (ILIM)
Other:
- moved on the sheet: R111, R112, R120, R121, R122, R123

Commit message: .
Other:
- note removed: "TO ADD CAPS ON TX LINES + TO ADD TVS DIODE"
Changed lines of the file:
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@@
 	(generator_version "9.0")
 	(paper "A4")
-	(text "TO ADD CAPS ON TX LINES + TO ADD TVS DIODE\n"
-		(exclude_from_sim no)
-		(at 93.472 69.088 0)
-		(effects
-			(font
-				(size 1.27 1.27)
-			)
-		)
-	)
 	(junction
 		(at 151.13 34.29)
