File: DP_ALT_USB.kicad_sch (KiCad schematic)
At the start: 41 parts, among them U14 IT8851, U15 TPS2553DRVR-1

Commit message: .
Parts:
- TP4, TP5: footprint (none) -> TestPoint:TestPoint_Pad_D1.0mm
- U14: footprint (none) -> Package_DFN_QFN:VQFN-28-1EP_4x4mm_P0.45mm_EP2.4x2.4mm
Connections:
- net DP_ALT_AUX+: now also USB8.A8 (SBU1)
- net DP_ALT_AUX-: now also USB8.B8 (SBU2)
- net DP_RX1+: now also D6.2, D6.9; no longer D6.1, D6.10
- net DP_RX1-: now also D6.1, D6.10; no longer D6.2, D6.9
- net DP_RX2+: now also D5.2, D5.9; no longer D5.5, D5.6
- net DP_RX2-: now also D5.1, D5.10; no longer D5.4, D5.7
- net DP_TX1+: now also D6.4, D6.7; no longer D5.1, D5.10
- net DP_TX1-: now also D6.5, D6.6; no longer D5.2, D5.9
- net DP_TX2+: now also D5.4, D5.7; no longer D6.5, D6.6
- net DP_TX2-: now also D5.5, D5.6; no longer D6.4, D6.7
- net GND: now also D6.8

Commit message: .
Parts:
- added R124: 10K, Resistor_SMD:R_0402_1005Metric, symbol Device:R
- added R125: 35K, Resistor_SMD:R_0402_1005Metric, symbol Device:R
Connections:
- net +5V: now also R124.1
- net GND: now also R125.1
- net at U15.2 (ILIM): now also R125.2
- net at U15.3 (~{FAULT}): now also R124.2
- no-connect marks 5 -> 4
Other:
- moved on the sheet: C137

Commit message: .
Parts:
- C129, C130, C135, C137: value 10uF -> 22uF
Changed lines of the file:
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@@
 			)
 		)
-		(property "Value" "10uF"
+		(property "Value" "22uF"
 			(at 91.44 151.1299 0)
 			(effects
@@
 			)
 		)
-		(property "Value" "10uF"
+		(property "Value" "22uF"
 			(at 22.86 139.6999 0)
 			(effects
@@
 		(fields_autoplaced yes)
 		(property "Reference" "C130"
-			(at 217.17 156.2101 0)
+			(at 224.79 153.6699 0)
 			(effects
 				(font
 					(size 1.27 1.27)
 				)
-				(justify left)
+				(justify right)
 			)
 		)
-		(property "Value" "10uF"
-			(at 217.17 153.6701 0)
+		(property "Value" "22uF"
+			(at 224.79 156.2099 0)
 			(effects
 				(font
 					(size 1.27 1.27)
 				)
-				(justify left)
+				(justify right)
 			)
 		)
@@
 		(fields_autoplaced yes)
 		(property "Reference" "C135"
-			(at 252.73 142.2401 0)
+			(at 260.35 139.6999 0)
 			(effects
 				(font
 					(size 1.27 1.27)
 				)
-				(justify left)
+				(justify right)
 			)
 		)
-		(property "Value" "10uF"
-			(at 252.73 139.7001 0)
+		(property "Value" "22uF"
+			(at 260.35 142.2399 0)
 			(effects
 				(font
 					(size 1.27 1.27)
 				)
-				(justify left)
+				(justify right)
 			)
 		)

Commit message: .
Parts:
- added R149, R150: 2.2K, Resistor_SMD:R_0402_1005Metric, symbol Device:R
Connections:
- net +3.3V: now also R149.2, R150.2
- net I2C2_SCL: now also R150.1
- net I2C2_SDA: now also R149.1
