File: ESP32.kicad_sch (KiCad schematic)
At the start: 6 parts, among them J2 Conn_01x04_Socket, SW1 TS-1089S-02526, SW2 TS-1089S-02526, U24 ESP32-C3-WROOM-02

Commit message: .
Parts:
- removed J2: Conn_01x04_Socket, Connector_PinSocket_2.54mm:PinSocket_1x04_P2.54mm_Vertical, symbol Connector:Conn_01x04_Socket
- removed U24: ESP32-C3-WROOM-02, RF_Module:ESP32-C3-WROOM-02, symbol RF_Module:ESP32-C3-WROOM-02
- added AE2: Antenna_Shield, RF_Antenna:Texas_SWRA117D_2.4GHz_Right, symbol Device:Antenna_Shield
- added C200, C201: 18pF, Capacitor_SMD:C_0402_1005Metric, symbol Device:C
- added C202, C205, C206, C207, C208: 100nF, Capacitor_SMD:C_0402_1005Metric, symbol Device:C
- added C203, C204: 3p3, Capacitor_SMD:C_0402_1005Metric, symbol Device:C
- added L8: 2n2, Inductor_SMD:L_0402_1005Metric, symbol Device:L
- added R140: 10k, Resistor_SMD:R_0402_1005Metric, symbol Device:R
- added U20: ZX-XH2.54-4PLT, easyeda2kicad:CONN-SMD_4P-P2.54_C9900012758, symbol da:ZX-XH2.54-4PLT
- added U21: ESP32-C3, Package_DFN_QFN:QFN-32-1EP_5x5mm_P0.5mm_EP3.7x3.7mm, symbol MCU_Espressif:ESP32-C3
- added Y5: 25Mhz, Crystal:Crystal_SMD_3225-4Pin_3.2x2.5mm, symbol Device:Crystal_GND24
Connections:
- net +3.3V: now also C202.2, C205.2, C206.2, C207.2, C208.2, R140.1, U21.11 (VDD3P3_RTC), U21.17 (VDD3P3_CPU), U21.18 (VDD_SPI), U21.2 (VDD3P3), U21.3 (VDD3P3), U21.31 (VDDA), U21.32 (VDDA)
- net ESP32_D+: now also U21.26 (GPIO19)
- net ESP32_D-: now also U21.25 (GPIO18)
- net GND: now also SW2.1, AE2.2 (Shield), C200.2, C201.2, C202.1, C203.2, C204.2, C205.1, C206.1, C207.1, C208.1, U20.4, U20.5, U20.6, U21.33 (GND), Y5.2, Y5.4; no longer SW2.2
- net IO3: now also U20.2, U21.8 (GPIO3)
- net at SW1.4: now also U21.7 (CHIP_EN)
- net at SW2.4: now also U21.15 (GPIO9)
- new net: C200.1, U21.30 (XTAL_P), Y5.1
- new net: C201.1, U21.29 (XTAL_N), Y5.3
- new net: C203.1, L8.1, U21.1 (LNA_IN)
- new net: R140.2, U21.6 (GPIO2)
- new net: AE2.1 (A), C204.1, L8.2
- new net +5V: U20.1
- no-connect marks 9 -> 19
Other:
- moved on the sheet: R110, R113, SW1, SW2

Commit message: .
Parts:
- Y5: value 25Mhz -> 40Mhz

Commit message: .
Parts:
- added C219: 100nF, Capacitor_SMD:C_0402_1005Metric, symbol Device:C
- added R158: 10k, Resistor_SMD:R_0402_1005Metric, symbol Device:R
Connections:
- net +3.3V: now also R158.2; no longer C206.2, U21.18 (VDD_SPI)
- net at R110.2, SW1.3: now also C219.2
- net at U21.14 (GPIO8): now also R158.1
- net at SW1.1: now also C219.1
- new net: C206.2, U21.18 (VDD_SPI)
- no-connect marks 19 -> 17
Other:
- note added: "TO ADD bigger caps and to separate from main 3.3v rail maybe"
- moved on the sheet: R110, R113, SW2
