File: HDMI_I2C_LEVEL_SHIFT.kicad_sch (KiCad schematic)
At the start: 12 parts, among them Q10 2N7002-SOT23, Q11 2N7002-SOT23, Q12 2N7002-SOT23, Q13 2N7002-SOT23

Commit message: .
Parts:
- added Q15, Q16: 2N7002-SOT23, easyeda2kicad:SOT-23_L2.9-W1.3-P1.90-LS2.4-BR, symbol da:2N7002-SOT23
- added R152, R153: 1M, Resistor_SMD:R_0402_1005Metric, symbol Device:R
- added R154, R155: 1K, Resistor_SMD:R_0402_1005Metric, symbol Device:R
- added R156, R157: 20K, Resistor_SMD:R_0402_1005Metric, symbol Device:R
Connections:
- net +3.3V: now also Q15.1 (G), Q16.1 (G), R152.2, R153.2
- new net: Q16.3 (D), R155.2, R156.1
- new net: Q15.3 (D), R154.2, R157.1
- new net GND: R156.2, R157.2
- new net HDMI_0_HPD: Q16.2 (S), R153.1
- new net HDMI_0_HPD_5V: R155.1
- new net HDMI_1_HPD: Q15.2 (S), R152.1
- new net HDMI_1_HPD_5V: R154.1
