File: PCIE_WIFI_ETH.kicad_sch (KiCad schematic)
At the start: 49 parts, among them CN1 2199230-4_C2977809, U6 TPS62590DRVT, U7 RTL8125BG-CG, Y3 25Mhz

Commit message: .
Other:
- added sheet ETH_WIFI_PWR (ETH_WIFI_PWR.kicad_sch)
Changed lines of the file:
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@@
+		)
+	)
+	(sheet
+		(at 19.05 54.61)
+		(size 24.13 16.51)
+		(exclude_from_sim no)
+		(in_bom yes)
+		(on_board yes)
+		(dnp no)
+		(fields_autoplaced yes)
+		(stroke
+			(width 0.1524)
+			(type solid)
+		)
+		(fill
+			(color 0 0 0 0.0000)
+		)
+		(property "Sheetname" "ETH_WIFI_PWR"
+			(at 19.05 53.8984 0)
+			(effects
+				(font
+					(size 1.27 1.27)
+				)
+				(justify left bottom)
+			)
+		)
+		(property "Sheetfile" "ETH_WIFI_PWR.kicad_sch"
+			(at 19.05 71.7046 0)
+			(effects
+				(font
+					(size 1.27 1.27)
+				)
+				(justify left top)
+			)
+		)
+		(instances
+			(project "MiniLatte"
+				(path "/ffe475c5-d6e9-41b5-8ca1-322659dd88d8/0b83a0c0-fa35-4171-b0ac-b3d09c000c8e"
+					(page "13")
+				)
+			)
 		)
 	)

Commit message: .
Connections:
- net +3.3V: now also C48.2, C51.2, C53.1, C59.2, C60.2, C61.2, C64.2, C65.2, U6.5 (VIN), U7.15 (AVDD33), U7.19 (AVDD33), U7.29 (DVDD33), U7.33 (AVDD33), U7.34 (AVDD33_XTAL), U7.43 (EVDD33), U7.46 (DVDD33)
- net +3.3VA: no longer C48.2, C51.2, C53.1, C59.2, C60.2, C61.2, C64.2, C65.2, U6.5 (VIN), U7.15 (AVDD33), U7.19 (AVDD33), U7.29 (DVDD33), U7.33 (AVDD33), U7.34 (AVDD33_XTAL), U7.43 (EVDD33), U7.46 (DVDD33)
- net HSIO+: now reaches C69.2, U7.38 (HSOP)
- net HSON-: now reaches C68.2, U7.39 (HSON)
- net HSIN+: now reaches C67.2, U7.41 (HSIP)
- net HSIN-: now reaches C66.2, U7.42 (HSIN)
Other:
- removed sheet ETH_WIFI_PWR
Changed lines of the file:
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@@
 		)
 	)
+	(label "HSIO+"
+		(at 228.6 55.88 0)
+		(effects
+			(font
+				(size 1.27 1.27)
+			)
+			(justify left bottom)
+		)
+	)
+	(label "HSIN+"
+		(at 228.6 48.26 0)
+		(effects
+			(font
+				(size 1.27 1.27)
+			)
+			(justify left bottom)
+		)
+	)
+	(label "HSIN-"
+		(at 228.6 45.72 0)
+		(effects
+			(font
+				(size 1.27 1.27)
+			)
+			(justify left bottom)
+		)
+	)
+	(label "HSON-"
+		(at 228.6 53.34 0)
+		(effects
+			(font
+				(size 1.27 1.27)
+			)
+			(justify left bottom)
+		)
+	)
 	(global_label "MD3+"
 		(shape input)
@@
 			)
 		)
-		(property "Value" "+3.3VA"
+		(property "Value" "+3.3V"
 			(at 218.948 63.6536 0)
 			(effects
@@
 			)
 		)
-		(property "Value" "+3.3VA"
+		(property "Value" "+3.3V"
 			(at 121.92 61.976 0)
 			(effects
@@
 			)
 		)
-		(property "Value" "+3.3VA"
+		(property "Value" "+3.3V"
 			(at 232.41 36.576 0)
 			(effects
@@
 			)
 		)
-		(property "Value" "+3.3VA"
+		(property "Value" "+3.3V"
 			(at 122.682 72.644 0)
 			(effects
@@
 			)
 		)
-		(property "Value" "+3.3VA"
+		(property "Value" "+3.3V"
 			(at 177.292 129.286 0)
 			(effects
@@
 			)
 		)
-		(property "Value" "+3.3VA"
+		(property "Value" "+3.3V"
 			(at 218.948 74.93 0)
 			(effects
@@
 				)
 			)
-		)
-	)
-	(sheet
-		(at 19.05 54.61)
-		(size 24.13 16.51)
-		(exclude_from_sim no)
-		(in_bom yes)
-		(on_board yes)
-		(dnp no)
-		(fields_autoplaced yes)
-		(stroke
-			(width 0.1524)
-			(type solid)
-		)
-		(fill
-			(color 0 0 0 0.0000)
-		)
-		(property "Sheetname" "ETH_WIFI_PWR"
-			(at 19.05 53.8984 0)
-			(effects
-				(font
-					(size 1.27 1.27)
-				)
-				(justify left bottom)
-			)
-		)
-		(property "Sheetfile" "ETH_WIFI_PWR.kicad_sch"
-			(at 19.05 71.7046 0)
-			(effects
-				(font
-					(size 1.27 1.27)
-				)
-				(justify left top)
-			)
-		)
-		(instances
-			(project "MiniLatte"
-				(path "/ffe475c5-d6e9-41b5-8ca1-322659dd88d8/0b83a0c0-fa35-4171-b0ac-b3d09c000c8e"
-					(page "13")
-				)
-			)

Commit message: .
Connections:
- net +3.3VA is gone; now on net +3.3V: R20.1, R21.1
- net PCIE_1_DTX+: now reaches C41.1, CN1.35
- net PCIE_1_DTX-: now reaches C42.1, CN1.37
Other:
- moved on the sheet: C41, C42, CN1, R15, R16

Commit message: .
Connections:
- net HSIN+ renamed HSI+
- net HSIN- renamed HSI-
- net HSIO+ renamed HSO+
- net HSON- renamed HSO-
Changed lines of the file:
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@@
 		)
 	)
-	(label "HSIO+"
+	(label "HSO+"
 		(at 228.6 55.88 0)
 		(effects
@@
 		)
 	)
-	(label "HSIN+"
+	(label "HSI+"
 		(at 228.6 48.26 0)
 		(effects
@@
 		)
 	)
-	(label "HSIN-"
+	(label "HSI-"
 		(at 228.6 45.72 0)
 		(effects
@@
 		)
 	)
-	(label "HSON-"
+	(label "HSO-"
 		(at 228.6 53.34 0)
 		(effects

Commit message: .
Connections:
- net SUSCLK_WIFI: no longer names the net of CN1.50
- no-connect marks 49 -> 50
Changed lines of the file:
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@@
+	)
+	(no_connect
+		(at 72.39 153.67)
 	)
 	(no_connect
@@
 		(pts
 			(xy 85.09 96.52) (xy 85.09 93.98)
-		)
-		(stroke
-			(width 0)
-			(type default)
-		)
-	)
-	(wire
-		(pts
-			(xy 76.2 153.67) (xy 72.39 153.67)
 		)
 		(stroke
@@
 				(hide yes)
 			)
-		)
-	)
-	(global_label "SUSCLK_WIFI"
-		(shape input)
-		(at 76.2 153.67 0)
-		(fields_autoplaced yes)
-		(effects
-			(font
-				(size 1.27 1.27)
-			)
-			(justify left)
-		)
-		(property "Intersheetrefs" "${INTERSHEET_REFS}"
-			(at 91.22 153.67 0)
-			(effects
-				(font
-					(size 1.27 1.27)
-				)
-				(justify left)
-				(hide yes)
-			)

Commit message: .
Parts:
- added TP9: +0.95V, TestPoint:TestPoint_Pad_D1.5mm, symbol Connector:TestPoint
- C45, C53: value 10uF -> 22uF
Connections:
- net +0.95V: now also TP9.1
Changed lines of the file:
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@@
 	)
 	(junction
-		(at 227.33 64.9236)
-		(diameter 0)
-		(color 0 0 0 0)
-	)
-	(junction
 		(at 248.92 81.28)
 		(diameter 0)
@@
 	(wire
 		(pts
-			(xy 227.33 64.9236) (xy 227.33 64.77)
+			(xy 227.33 64.77) (xy 227.33 66.04)
 		)
 		(stroke
@@
 	(wire
 		(pts
-			(xy 227.33 66.04) (xy 227.33 64.9236)
-		)
-		(stroke
-			(width 0)
-			(type default)
-		)
-	)
-	(wire
-		(pts
 			(xy 72.39 184.15) (xy 74.93 184.15)
 		)
@@
 	(symbol
 		(lib_id "power:+3.3VA")
-		(at 227.33 64.9236 0)
+		(at 227.33 64.77 0)
 		(unit 1)
 		(exclude_from_sim no)
@@
 		(dnp no)
 		(property "Reference" "#PWR0148"
-			(at 227.33 68.7336 0)
+			(at 227.33 68.58 0)
 			(effects
 				(font
@@
 		)
 		(property "Value" "+3.3V"
-			(at 218.948 63.6536 0)
+			(at 218.948 63.5 0)
 			(effects
 				(font
@@
 		)
 		(property "Footprint" ""
-			(at 227.33 64.9236 0)
+			(at 227.33 64.77 0)
 			(effects
 				(font
@@
 		)
 		(property "Datasheet" ""
-			(at 227.33 64.9236 0)
+			(at 227.33 64.77 0)
 			(effects
 				(font
@@
 		)
 		(property "Description" ""
-			(at 227.33 64.9236 0)
+			(at 227.33 64.77 0)
 			(effects
 				(font
@@
 	)
 	(symbol
+		(lib_id "Connector:TestPoint")
+		(at 120.65 133.35 0)
+		(unit 1)
+		(exclude_from_sim no)
+		(in_bom yes)
+		(on_board yes)
+		(dnp no)
+		(property "Reference" "TP9"
+			(at 123.19 128.7779 0)
+			(effects
+				(font
+					(size 1.27 1.27)
+				)
+				(justify left)
+			)
+		)
+		(property "Value" "+0.95V"
+			(at 122.936 130.81 0)
+			(effects
+				(font
+					(size 1.27 1.27)
+				)
+				(justify left)
+			)
+		)
+		(property "Footprint" "TestPoint:TestPoint_Pad_D1.5mm"
+			(at 125.73 133.35 0)
+			(effects
+				(font
+					(size 1.27 1.27)
+				)
+				(hide yes)
+			)
+		)
+		(property "Datasheet" "~"
+			(at 125.73 133.35 0)
+			(effects
+				(font
+					(size 1.27 1.27)
+				)
+				(hide yes)
+			)
+		)
+		(property "Description" "test point"
+			(at 120.65 133.35 0)
+			(effects
+				(font
+					(size 1.27 1.27)
+				)
+				(hide yes)
+			)
+		)
+		(pin "1"
+		)
+		(instances
+			(project "MiniLatte"
+				(path "/ffe475c5-d6e9-41b5-8ca1-322659dd88d8/0b83a0c0-fa35-4171-b0ac-b3d09c000c8e"
+					(reference "TP9")
+					(unit 1)
+				)
+			)
+		)
+	)
+	(symbol
 		(lib_id "Device:R")
 		(at 76.2 161.29 90)
@@
 			)
 		)
-		(property "Value" "10uF"
+		(property "Value" "22uF"
 			(at 181.356 144.526 0)
 			(effects
@@
 			)
 		)
-		(property "Value" "10uF"
+		(property "Value" "22uF"
 			(at 113.284 139.7 0)
 			(effects

Commit message: .
Parts:
- added R151: 10k, Resistor_SMD:R_0402_1005Metric, symbol Device:R
Connections:
- net +3.3V: now also R151.2
- net at U7.27 (LED1/EESK/SPISC): now also R151.1
- no-connect marks 50 -> 49
Changed lines of the file:
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@@
 	)
 	(no_connect
-		(at 212.09 83.82)
-	)
-	(no_connect
 		(at 57.15 113.03)
 	)
@@
 	(wire
 		(pts
+			(xy 231.14 85.09) (xy 242.57 85.09)
+		)
+		(stroke
+			(width 0)
+			(type default)
+		)
+	)
+	(wire
+		(pts
 			(xy 74.93 184.15) (xy 96.52 184.15)
 		)
@@
 	(wire
 		(pts
+			(xy 212.09 83.82) (xy 223.52 83.82)
+		)
+		(stroke
+			(width 0)
+			(type default)
+		)
+	)
+	(wire
+		(pts
 			(xy 167.64 135.89) (xy 179.07 135.89)
 		)
@@
 	(wire
 		(pts
+			(xy 223.52 83.82) (xy 223.52 85.09)
+		)
+		(stroke
+			(width 0)
+			(type default)
+		)
+	)
+	(wire
+		(pts
 			(xy 228.6 43.18) (xy 238.76 43.18)
 		)
@@
 	)
 	(symbol
+		(lib_id "Device:R")
+		(at 227.33 85.09 90)
+		(unit 1)
+		(exclude_from_sim no)
+		(in_bom yes)
+		(on_board yes)
+		(dnp no)
+		(property "Reference" "R151"
+			(at 225.298 87.884 90)
+			(effects
+				(font
+					(size 1.27 1.27)
+				)
+			)
+		)
+		(property "Value" "10k"
+			(at 230.378 87.884 90)
+			(effects
+				(font
+					(size 1.27 1.27)
+				)
+			)
+		)
+		(property "Footprint" "Resistor_SMD:R_0402_1005Metric"
+			(at 227.33 86.868 90)
+			(effects
+				(font
+					(size 1.27 1.27)
+				)
+				(hide yes)
+			)
+		)
+		(property "Datasheet" "~"
+			(at 227.33 85.09 0)
+			(effects
+				(font
+					(size 1.27 1.27)
+				)
+				(hide yes)
+			)
+		)
+		(property "Description" "Resistor"
+			(at 227.33 85.09 0)
+			(effects
+				(font
+					(size 1.27 1.27)
+				)
+				(hide yes)
+			)
+		)
+		(pin "1"
+		)
+		(pin "2"
+		)
+		(instances
+			(project "MiniLatte"
+				(path "/ffe475c5-d6e9-41b5-8ca1-322659dd88d8/0b83a0c0-fa35-4171-b0ac-b3d09c000c8e"
+					(reference "R151")
+					(unit 1)
+				)
+			)
+		)
+	)
+	(symbol
 		(lib_id "power:GND")
 		(at 64.77 193.04 0)
@@
 					(unit 1)
 				)
+			)
+		)
+	)
+	(symbol
+		(lib_id "power:+3.3VA")
+		(at 242.57 85.09 0)
+		(unit 1)
+		(exclude_from_sim no)
+		(in_bom yes)
+		(on_board yes)
+		(dnp no)
+		(property "Reference" "#PWR0580"
+			(at 242.57 88.9 0)
+			(effects
+				(font
+					(size 1.27 1.27)
+				)
+				(hide yes)
+			)
+		)
+		(property "Value" "+3.3V"
+			(at 234.188 83.82 0)
+			(effects
+				(font
+					(size 1.27 1.27)
+				)
+				(justify left)
+			)
+		)
+		(property "Footprint" ""
+			(at 242.57 85.09 0)
+			(effects
+				(font
+					(size 1.27 1.27)
+				)
+				(hide yes)
+			)
+		)
+		(property "Datasheet" ""
+			(at 242.57 85.09 0)
+			(effects
+				(font
+					(size 1.27 1.27)
+				)
+				(hide yes)
+			)
+		)
+		(property "Description" ""
+			(at 242.57 85.09 0)
+			(effects
+				(font
+					(size 1.27 1.27)
+				)
+			)
+		)
+		(pin "1"
+		)
+		(instances
+			(project "MiniLatte"
+				(path "/ffe475c5-d6e9-41b5-8ca1-322659dd88d8/0b83a0c0-fa35-4171-b0ac-b3d09c000c8e"
+					(reference "#PWR0580")
+					(unit 1)
+				)
