File: PD_Power.kicad_sch (KiCad schematic)
At the start: 29 parts, among them J1 USB_C_Receptacle_USB2.0_16P, Q3 AON7403, Q5 AON7402, Q6 AON7402, Q7 AON7402, Q8 AON7402, U16 HUSB238_002DD, U17 TPS51275RUKR

Commit message: .
Parts:
- removed C166: ?nF, symbol Device:C_Small
- added C167, C168, C169, C170: 10uF, Capacitor_SMD:C_0805_2012Metric, symbol Device:C
- added C171, C172, C173: 220nF, Capacitor_SMD:C_0402_1005Metric, symbol Device:C_Small
- added R104: 0R, Resistor_SMD:R_0402_1005Metric, symbol Device:R
- added R105: 10K, Resistor_SMD:R_0402_1005Metric, symbol Device:R
- added R106: 3K, Resistor_SMD:R_0402_1005Metric, symbol Device:R
- C163, C164: footprint (none) -> Capacitor_SMD:C_0402_1005Metric
- C165: value ?nF -> 220nF; footprint (none) -> Capacitor_SMD:C_0402_1005Metric
- L6, L7: value L -> 3.3H; footprint (none) -> Inductor_SMD:L_APV_APH1040
- R100, R101, R102, R103, R96, R97, R98, R99: footprint (none) -> Resistor_SMD:R_0402_1005Metric
Connections:
- net +3.3V: now also C171.2
- net +5V: now also C172.1, C173.1
- net GND: now also C167.2, C168.2, C169.2, C170.2, C171.1, C172.2, C173.2, R106.2
- net PD_VBUS: now also R105.1
- net PD_VBUS_GATE: now also C167.1, C168.1, C169.1, C170.1
- net PD_EN: now reaches U17.20 (EN1)
- net PD_EN: now also U17.6 (EN2), R104.2, R105.2, R106.1
- net 3.3LDO: now reaches U17.3 (VREG3)
- net 3.3LDO: now also R104.1
- no-connect marks 11 -> 13
Other:
- moved on the sheet: C163, C164, C165, L6, L7, Q5, Q6, Q7, Q8, R100, R101, R102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

Commit message: .
Connections:
- net PD_VBUS: now also Q3.5 (D), Q3.6 (D), Q3.7 (D), Q3.8 (D), R92.2
- new net: C162.1, R91.2, U16.1 (VIN)
Changed lines of the file:
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@@
+	)
+	(junction
+		(at 95.25 43.18)
+		(diameter 0)
+		(color 0 0 0 0)
 	)
 	(junction
@@
 	(junction
 		(at 68.58 114.3)
-		(diameter 0)
-		(color 0 0 0 0)
-	)
-	(junction
-		(at 129.54 43.18)
 		(diameter 0)
 		(color 0 0 0 0)
@@
 	(wire
 		(pts
-			(xy 81.28 43.18) (xy 105.41 43.18)
+			(xy 81.28 43.18) (xy 95.25 43.18)
 		)
 		(stroke
@@
 	(wire
 		(pts
+			(xy 95.25 35.56) (xy 160.02 35.56)
+		)
+		(stroke
+			(width 0)
+			(type default)
+		)
+	)
+	(wire
+		(pts
 			(xy 104.14 97.79) (xy 104.14 93.98)
 		)
@@
 	(wire
 		(pts
+			(xy 95.25 43.18) (xy 105.41 43.18)
+		)
+		(stroke
+			(width 0)
+			(type default)
+		)
+	)
+	(wire
+		(pts
 			(xy 64.77 116.84) (xy 114.3 116.84)
 		)
@@
 	(wire
 		(pts
+			(xy 95.25 35.56) (xy 95.25 43.18)
+		)
+		(stroke
+			(width 0)
+			(type default)
+		)
+	)
+	(wire
+		(pts
 			(xy 181.61 33.02) (xy 187.96 33.02)
 		)
@@
 	(wire
 		(pts
-			(xy 129.54 35.56) (xy 129.54 43.18)
-		)
-		(stroke
-			(width 0)
-			(type default)
-		)
-	)
-	(wire
-		(pts
 			(xy 73.66 109.22) (xy 68.58 109.22)
 		)
@@
 		)
 		(stroke
-			(width 0)
-			(type default)
-		)
-	)
-	(wire
-		(pts
-			(xy 129.54 35.56) (xy 160.02 35.56)
-		)
-		(stroke

Commit message: .
Parts:
- C165, C171, C172, C173: value 220nF -> 220uF; footprint Capacitor_SMD:C_0402_1005Metric -> Capacitor_SMD:C_Elec_6.3x7.7
Changed lines of the file:
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@@
 			)
 		)
-		(property "Value" "220nF"
+		(property "Value" "220uF"
 			(at 229.616 105.664 0)
 			(effects
@@
 			)
 		)
-		(property "Footprint" "Capacitor_SMD:C_0402_1005Metric"
+		(property "Footprint" "Capacitor_SMD:C_Elec_6.3x7.7"
 			(at 224.79 101.6 0)
 			(effects
@@
 			)
 		)
-		(property "Value" "220nF"
+		(property "Value" "220uF"
 			(at 100.076 96.52 0)
 			(effects
@@
 			)
 		)
-		(property "Footprint" "Capacitor_SMD:C_0402_1005Metric"
+		(property "Footprint" "Capacitor_SMD:C_Elec_6.3x7.7"
 			(at 104.14 100.33 0)
 			(effects
@@
 			)
 		)
-		(property "Value" "220nF"
+		(property "Value" "220uF"
 			(at 238.506 105.664 0)
 			(effects
@@
 			)
 		)
-		(property "Footprint" "Capacitor_SMD:C_0402_1005Metric"
+		(property "Footprint" "Capacitor_SMD:C_Elec_6.3x7.7"
 			(at 233.68 101.6 0)
 			(effects
@@
 			)
 		)
-		(property "Value" "220nF"
+		(property "Value" "220uF"
 			(at 91.186 96.52 0)
 			(effects
@@
 			)
 		)
-		(property "Footprint" "Capacitor_SMD:C_0402_1005Metric"
+		(property "Footprint" "Capacitor_SMD:C_Elec_6.3x7.7"
 			(at 95.25 100.33 0)
 			(effects

Commit message: .
Other:
- added sheet MU_PWR (MU_PWR.kicad_sch)
Changed lines of the file:
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@@
+		)
+	)
+	(sheet
+		(at 100.33 167.64)
+		(size 30.48 26.67)
+		(exclude_from_sim no)
+		(in_bom yes)
+		(on_board yes)
+		(dnp no)
+		(fields_autoplaced yes)
+		(stroke
+			(width 0.1524)
+			(type solid)
+		)
+		(fill
+			(color 0 0 0 0.0000)
+		)
+		(property "Sheetname" "MU_PWR"
+			(at 100.33 166.9284 0)
+			(effects
+				(font
+					(size 1.27 1.27)
+				)
+				(justify left bottom)
+			)
+		)
+		(property "Sheetfile" "MU_PWR.kicad_sch"
+			(at 100.33 194.8946 0)
+			(effects
+				(font
+					(size 1.27 1.27)
+				)
+				(justify left top)
+			)
+		)
+		(instances
+			(project "MiniLatte"
+				(path "/ffe475c5-d6e9-41b5-8ca1-322659dd88d8/3f07c54d-c68c-4501-9d1d-0870eca96d91"
+					(page "18")
+				)
+			)
 		)
 	)

Commit message: .
Parts:
- added TP2: +5V TestPoint, TestPoint:TestPoint_Pad_D1.5mm, symbol Connector:TestPoint
- added TP3: +3.3V TestPoint, TestPoint:TestPoint_Pad_D1.5mm, symbol Connector:TestPoint
- C167, C168, C169, C170: value 10uF -> 22uF
- R94, R95: now not fitted
- TP6: footprint TestPoint:TestPoint_Pad_2.0x2.0mm -> TestPoint:TestPoint_Pad_D1.5mm
Connections:
- net +3.3V: now also TP3.1
- net +5V: now also TP2.1
Other:
- note added: "20V@3A.25 Configuration"
- note removed: "15V@3A Configuration"
Changed lines of the file:
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@@
 	(generator_version "9.0")
 	(paper "A4")
-	(text "15V@3A\nConfiguration"
+	(text "20V@3A.25\nConfiguration"
 		(exclude_from_sim no)
 		(at 183.642 55.88 0)
@@
 	)
 	(junction
+		(at 100.33 93.98)
+		(diameter 0)
+		(color 0 0 0 0)
+	)
+	(junction
 		(at 95.25 43.18)
 		(diameter 0)
@@
 	)
 	(junction
+		(at 233.68 99.06)
+		(diameter 0)
+		(color 0 0 0 0)
+	)
+	(junction
 		(at 81.28 43.18)
 		(diameter 0)
@@
 	)
 	(junction
-		(at 219.71 147.32)
-		(diameter 0)
-		(color 0 0 0 0)
-	)
-	(junction
 		(at 49.53 114.3)
 		(diameter 0)
@@
 	(wire
 		(pts
-			(xy 219.71 147.32) (xy 219.71 146.05)
-		)
-		(stroke
-			(width 0)
-			(type default)
-		)
-	)
-	(wire
-		(pts
 			(xy 236.22 144.78) (xy 236.22 127)
 		)
@@
 	(wire
 		(pts
+			(xy 100.33 93.98) (xy 95.25 93.98)
+		)
+		(stroke
+			(width 0)
+			(type default)
+		)
+	)
+	(wire
+		(pts
 			(xy 220.98 154.94) (xy 119.38 154.94)
 		)
@@
 	(wire
 		(pts
-			(xy 104.14 93.98) (xy 95.25 93.98)
+			(xy 104.14 93.98) (xy 100.33 93.98)
 		)
 		(stroke
@@
 		(in_bom yes)
 		(on_board yes)
-		(dnp no)
+		(dnp yes)
 		(property "Reference" "R95"
 			(at 175.768 59.944 0)
@@
 	)
 	(symbol
+		(lib_id "Connector:TestPoint")
+		(at 233.68 99.06 0)
+		(unit 1)
+		(exclude_from_sim no)
+		(in_bom yes)
+		(on_board yes)
+		(dnp no)
+		(fields_autoplaced yes)
+		(property "Reference" "TP3"
+			(at 236.22 94.4879 0)
+			(effects
+				(font
+					(size 1.27 1.27)
+				)
+				(justify left)
+			)
+		)
+		(property "Value" "+3.3V TestPoint"
+			(at 236.22 97.0279 0)
+			(effects
+				(font
+					(size 1.27 1.27)
+				)
+				(justify left)
+			)
+		)
+		(property "Footprint" "TestPoint:TestPoint_Pad_D1.5mm"
+			(at 238.76 99.06 0)
+			(effects
+				(font
+					(size 1.27 1.27)
+				)
+				(hide yes)
+			)
+		)
+		(property "Datasheet" "~"
+			(at 238.76 99.06 0)
+			(effects
+				(font
+					(size 1.27 1.27)
+				)
+				(hide yes)
+			)
+		)
+		(property "Description" "test point"
+			(at 233.68 99.06 0)
+			(effects
+				(font
+					(size 1.27 1.27)
+				)
+				(hide yes)
+			)
+		)
+		(pin "1"
+		)
+		(instances
+			(project "MiniLatte"
+				(path "/ffe475c5-d6e9-41b5-8ca1-322659dd88d8/3f07c54d-c68c-4501-9d1d-0870eca96d91"
+					(reference "TP3")
+					(unit 1)
+				)
+			)
+		)
+	)
+	(symbol
 		(lib_id "Device:C")
 		(at 278.13 134.62 0)
@@
 		(on_board yes)
 		(dnp no)
-		(fields_autoplaced yes)
 		(property "Reference" "C169"
-			(at 274.32 133.3499 0)
+			(at 270.256 133.35 0)
 			(effects
 				(font
 					(size 1.27 1.27)
 				)
-				(justify left)
+				(justify right)
 			)
 		)
-		(property "Value" "10uF"
-			(at 274.32 135.8899 0)
+		(property "Value" "22uF"
+			(at 270.256 135.89 0)
 			(effects
 				(font
 					(size 1.27 1.27)
 				)
-				(justify left)
+				(justify right)
 			)
 		)
@@
 			)
 		)
-		(property "Value" "10uF"
+		(property "Value" "22uF"
 			(at 41.91 123.1899 0)
 			(effects
@@
 	)
 	(symbol
+		(lib_id "Connector:TestPoint")
+		(at 100.33 93.98 0)
+		(unit 1)
+		(exclude_from_sim no)
+		(in_bom yes)
+		(on_board yes)
+		(dnp no)
+		(fields_autoplaced yes)
+		(property "Reference" "TP2"
+			(at 102.87 89.4079 0)
+			(effects
+				(font
+					(size 1.27 1.27)
+				)
+				(justify left)
+			)
+		)
+		(property "Value" "+5V TestPoint"
+			(at 102.87 91.9479 0)
+			(effects
+				(font
+					(size 1.27 1.27)
+				)
+				(justify left)
+			)
+		)
+		(property "Footprint" "TestPoint:TestPoint_Pad_D1.5mm"
+			(at 105.41 93.98 0)
+			(effects
+				(font
+					(size 1.27 1.27)
+				)
+				(hide yes)
+			)
+		)
+		(property "Datasheet" "~"
+			(at 105.41 93.98 0)
+			(effects
+				(font
+					(size 1.27 1.27)
+				)
+				(hide yes)
+			)
+		)
+		(property "Description" "test point"
+			(at 100.33 93.98 0)
+			(effects
+				(font
+					(size 1.27 1.27)
+				)
+				(hide yes)
+			)
+		)
+		(pin "1"
+		)
+		(instances
+			(project "MiniLatte"
+				(path "/ffe475c5-d6e9-41b5-8ca1-322659dd88d8/3f07c54d-c68c-4501-9d1d-0870eca96d91"
+					(reference "TP2")
+					(unit 1)
+				)
+			)
+		)
+	)
+	(symbol
 		(lib_id "power:GND")
 		(at 26.67 127 0)
@@
 		(in_bom yes)
 		(on_board yes)
-		(dnp no)
+		(dnp yes)
 		(property "Reference" "R94"
 			(at 162.052 59.944 0)
@@
 		(on_board yes)
 		(dnp no)
-		(fields_autoplaced yes)
 		(property "Reference" "C170"
-			(at 262.89 133.3499 0)
+			(at 258.318 133.35 0)
 			(effects
 				(font
 					(size 1.27 1.27)
 				)
-				(justify left)
+				(justify right)
 			)
 		)
-		(property "Value" "10uF"
-			(at 262.89 135.8899 0)
+		(property "Value" "22uF"
+			(at 258.318 135.89 0)
 			(effects
 				(font
 					(size 1.27 1.27)
 				)
-				(justify left)
+				(justify right)
 			)
 		)
@@
 			)
 		)
-		(property "Value" "10uF"
+		(property "Value" "22uF"
 			(at 30.48 123.1899 0)
 			(effects
@@
 			)
 		)
-		(property "Footprint" "TestPoint:TestPoint_Pad_2.0x2.0mm"
+		(property "Footprint" "TestPoint:TestPoint_Pad_D1.5mm"
 			(at 69.85 43.18 0)
 			(effects

Commit message: .
Parts:
- R102: value 13k -> 15k
- R103: value 20k -> 10k
Other:
- note added: "20V@3.25A Configuration"
- note removed: "20V@3A.25 Configuration"
Changed lines of the file:
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@@
 	(generator_version "9.0")
 	(paper "A4")
-	(text "20V@3A.25\nConfiguration"
+	(text "20V@3.25A\nConfiguration"
 		(exclude_from_sim no)
 		(at 183.642 55.88 0)
@@
 			)
 		)
-		(property "Value" "13k"
+		(property "Value" "15k"
 			(at 191.77 95.25 0)
 			(effects
@@
 			)
 		)
-		(property "Value" "20k"
+		(property "Value" "10k"
 			(at 191.77 102.87 0)
 			(effects

Commit message: .
Parts:
- added C217, C218: 1uF, Capacitor_SMD:C_0603_1608Metric, symbol Device:C
Connections:
- net 3.3LDO: now also C218.1
- net GND: now also C217.2, C218.2
- net 5LDO: now reaches U17.13 (VREG5)
- net 5LDO: now also C217.1
- no-connect marks 13 -> 12
