File: PWR_LED.kicad_sch (KiCad schematic)
At the start: 10 parts, among them Q4 2N7002-SOT23, Q9 2N7002-SOT23, SW3 TC-1102N-C-A-B, SW4 TC-1102N-C-A-B

Commit message: .
Parts:
- added R126, R127: R, Resistor_SMD:R_0402_1005Metric, symbol Device:R
Connections:
- net GND: now also R126.1, R127.1
- net S0_PWR_IND: now also R127.2
- net S3_PWR_IND: now also R126.2

Commit message: .
Parts:
- R126, R127: value R -> 10k
- R34: value R -> 65R
- R35: value R -> 40R
- R36: value R -> 10R
Changed lines of the file:
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@@
-	(wire
-		(pts
-			(xy 67.31 60.96) (xy 67.31 66.04)
-		)
-		(stroke
-			(width 0)
-			(type default)
-		)
-	)
 	(wire
 		(pts
@@
 		(dnp no)
 		(property "Reference" "R127"
-			(at 58.674 87.376 90)
-			(effects
-				(font
-					(size 1.27 1.27)
-				)
-			)
-		)
-		(property "Value" "R"
-			(at 58.674 90.932 90)
+			(at 56.388 90.424 0)
+			(effects
+				(font
+					(size 1.27 1.27)
+				)
+			)
+		)
+		(property "Value" "10k"
+			(at 57.15 92.456 0)
 			(effects
 				(font
@@
 			)
 		)
-		(property "Value" "R"
-			(at 124.46 68.834 90)
+		(property "Value" "40R"
+			(at 123.698 69.088 90)
 			(effects
 				(font
@@
 		(dnp no)
 		(property "Reference" "R126"
-			(at 57.404 68.326 90)
-			(effects
-				(font
-					(size 1.27 1.27)
-				)
-			)
-		)
-		(property "Value" "R"
-			(at 57.404 71.882 90)
+			(at 55.118 71.882 0)
+			(effects
+				(font
+					(size 1.27 1.27)
+				)
+			)
+		)
+		(property "Value" "10k"
+			(at 56.134 74.422 0)
 			(effects
 				(font
@@
 			)
 		)
-		(property "Value" "R"
-			(at 124.968 73.914 90)
+		(property "Value" "10R"
+			(at 123.698 73.914 90)
 			(effects
 				(font
@@
 			)
 		)
-		(property "Value" "R"
-			(at 124.46 62.738 90)
-			(effects
-				(font
+		(property "Value" "65R"
+			(at 123.952 62.738 90)
+			(effects
+				(font

Commit message: .
Parts:
- R37, R38: now not fitted
Changed lines of the file:
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@@
 		(in_bom yes)
 		(on_board yes)
-		(dnp no)
+		(dnp yes)
 		(fields_autoplaced yes)
 		(property "Reference" "R38"
@@
 		(in_bom yes)
 		(on_board yes)
-		(dnp no)
+		(dnp yes)
 		(fields_autoplaced yes)
 		(property "Reference" "R37"

Commit message: .
Connections:
- net +3.3V: now also LED1.2 (A), LED1.3 (A); no longer Q4.3 (D), Q9.3 (D)
- net GND: now also Q4.2 (S), Q9.2 (S); no longer R35.2, R36.2
- new net: Q9.3 (D), R36.2
- new net: Q4.3 (D), R35.2
Other:
- moved on the sheet: Q4, Q9, R126, R127
