File: PCB/MiniLatte.kicad_sch (KiCad schematic)
At the start: 21 parts, among them CN5 WAFER-PH2.0-4PLB, CN8 SMTWE2055MTJ, CN9 SMTWE2055MTJ, Q14 2N7002-SOT23, SW6 DSHP01TSGER, U24 W25Q128JVEIQ

Commit message: .
Connections:
- net S0_PWR_IND is gone; now on net S0_PWR: Q14.1 (G), R159.2
Changed lines of the file:
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@@
-	(wire
-		(pts
-			(xy 246.38 109.22) (xy 240.03 109.22)
-		)
-		(stroke
-			(width 0)
-			(type default)
-		)
-	)
 	(wire
 		(pts
@@
 	(wire
 		(pts
+			(xy 229.87 109.22) (xy 246.38 109.22)
+		)
+		(stroke
+			(width 0)
+			(type default)
+		)
+	)
+	(wire
+		(pts
 			(xy 217.17 203.2) (xy 238.76 203.2)
 		)
@@
 			(width 0)
 			(type default)
+		)
+	)
+	(label "S0_PWR"
+		(at 229.87 109.22 0)
+		(effects
+			(font
+				(size 1.27 1.27)
+			)
+			(justify left bottom)
 		)
 	)
@@
 		)
 	)
-	(hierarchical_label "S0_PWR_IND"
-		(shape input)
-		(at 240.03 109.22 180)
-		(effects
-			(font
-				(size 1.27 1.27)
-			)
-			(justify right)
-		)
-	)

Commit message: .
Parts:
- removed Q14: 2N7002-SOT23, easyeda2kicad:SOT-23_L2.9-W1.3-P1.90-LS2.4-BR, symbol da:2N7002-SOT23
- added Q14: AO3400_C2890121, easyeda2kicad:SOT-23-3_L2.9-W1.6-P1.90-LS2.8-BR, symbol da:AO3400_C2890121
Connections:
- net GND: now also Q14.2 (S)
- net S0_PWR: now also Q14.1 (G)
- net at CN5.4: now also Q14.3 (D)
