File: PCB/ESP32.kicad_sch (KiCad schematic)
At the start: 21 parts, among them SW1 TS-1089S-02526, SW2 TS-1089S-02526, U20 ZX-XH2.54-4PLT, U21 ESP32-C3, Y5 40Mhz

Commit message: .
Other:
- note removed: "TO ADD bigger caps and to separate from main 3.3v rail maybe"
Changed lines of the file:
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@@
 	(generator_version "10.0")
 	(paper "A4")
-	(text "TO ADD bigger caps and to separate from main 3.3v rail maybe"
-		(exclude_from_sim no)
-		(at 55.626 75.438 0)
-		(effects
-			(font
-				(size 1.27 1.27)
-			)
-		)
-	)
 	(junction
 		(at 72.39 147.32)
